File: Blade.brd (EAGLE design)
At the start: 160 x 101.6 mm, 100 parts, among them IC1 THN10-2411WIR, IC2 MCP6064-E/SL, IC3 MCP6064-E/SL, IC4 MCP6064-E/SL, Q1 12MHz, U1 ADR366WAUJZ, U2 ADR366WAUJZ, U3 ADS1148QPWRQ1, U4 ADS1148QPWRQ1, U5 ADS1148QPWRQ1, U6 LT1528, U7 S70FL01GS, U8 S70FL01GS, U9 STM32F77XXXLQFP208, X1 D-SUB9-H5M09RA, X2 D-SUB15-H5M15RA, X3 USBPTH

Commit message: opto added
Parts:
- added D5, D6, D7, D8, D9: 3V6, diodes:DMELF
- added IC5: MAX488CSA, maxim:SO08
- added IC6, IC7: MOCD207MSOIC-8, Opto-Electronic:SOIC127P594X363-8N
- added R10: 1k, rcl:R0805
- added RN11, RN12: 56k, resistor-dil:EXBS8V
- moved D4 5.62 mm to (101.0, 49.0), turned to 180 degrees
- moved R9 0.25 mm to (106.7, 25.1)
Connections:
- new net EXP_IN: D5.C, IC5.2, U9.200
- new net EXP_OUT: D6.C, IC5.3, U9.201
- new net LO_OPT: D7.C, IC7.8, RN12.6, U9.208
- new net N$42: IC6.1, RN11.6
- new net N$43: IC6.3, RN11.5
- new net N$45: IC7.6, RN12.5
- new net N$46: IC7.1, RN11.8
- new net N$47: IC7.3, RN11.7
- new net N$48: IC7.4
- new net SODS_OPT: D8.C, IC6.8, RN12.8, U9.206
- new net SOE_OPT: D9.C, IC6.6, RN12.7, U9.207
- net 28V: now also RN11.1, RN11.2, RN11.3, RN11.4
- net 3V3: now also IC5.1, RN12.1, RN12.2, RN12.3, RN12.4
- net EXP_IN_N: now also IC5.7, R10.1
- net EXP_IN_P: now also IC5.8, R10.2
- net EXP_OUT_N: now also IC5.6
- net EXP_OUT_P: now also IC5.5
- net GND: now also D5.A, D6.A, D7.A, D8.A, D9.A, IC5.4, IC6.5, IC6.7, IC7.5, IC7.7
- net LO: now also IC7.2
- net SODS: now also IC6.2
- net SOE: now also IC6.4
Routing:
- net LO_OPT: track 0.00 -> 59.8 mm, vias 0 -> 3
- net SOE_OPT: track 0.00 -> 59.2 mm, vias 0 -> 4
- net SODS_OPT: track 0.00 -> 53.2 mm, vias 0 -> 3
- net EXP_IN: track 0.00 -> 49.8 mm, vias 0 -> 2
- net EXP_OUT: track 0.00 -> 49.4 mm, vias 0 -> 3
- net LO: track 0.00 -> 45.9 mm, vias 0 -> 1
- net EXP_IN_N: track 0.00 -> 41.9 mm
- net EXP_IN_P: track 0.00 -> 33.6 mm
- net EXP_OUT_N: track 0.00 -> 32.0 mm, vias 0 -> 1
- net EXP_OUT_P: track 0.00 -> 30.1 mm, vias 0 -> 1
- net SODS: track 0.00 -> 29.2 mm
- net 3V3: track 671.6 -> 700.1 mm
- net SOE: track 0.00 -> 27.0 mm
- net GND: track 1023.2 -> 1002.7 mm, vias 145 -> 144
- net 28V: track 80.5 -> 100.6 mm
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
Commit message: cleanup
Parts:
- RN11: value 56k -> 3k
- RN12: value 56k -> 1k
Changed lines of the file:
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@@
 <drawing>
 <settings>
-<setting alwaysvectorfont="yes"/>
+<setting alwaysvectorfont="no"/>
 <setting verticaltext="up"/>
 </settings>
@@
 <attribute name="VALUE" x="133.985" y="40.03" size="1.27" layer="27" rot="R180" align="top-center"/>
 </element>
-<element name="RN11" library="resistor-dil" library_urn="urn:adsk.eagle:library:342" package="EXBS8V" package3d_urn="urn:adsk.eagle:package:24925/1" value="56k" x="132.334" y="34.036" smashed="yes" rot="MR90">
+<element name="RN11" library="resistor-dil" library_urn="urn:adsk.eagle:library:342" package="EXBS8V" package3d_urn="urn:adsk.eagle:package:24925/1" value="3k" x="132.334" y="34.036" smashed="yes" rot="MR90">
 <attribute name="MF" value="" x="132.334" y="34.036" size="1.778" layer="28" rot="MR90" display="off"/>
 <attribute name="MPN" value="" x="132.334" y="34.036" size="1.778" layer="28" rot="MR90" display="off"/>
@@
 <attribute name="VALUE" x="133.985" y="34.315" size="1.27" layer="27" rot="R180" align="top-center"/>
 </element>
-<element name="RN12" library="resistor-dil" library_urn="urn:adsk.eagle:library:342" package="EXBS8V" package3d_urn="urn:adsk.eagle:package:24925/1" value="56k" x="114.173" y="24.384" smashed="yes">
+<element name="RN12" library="resistor-dil" library_urn="urn:adsk.eagle:library:342" package="EXBS8V" package3d_urn="urn:adsk.eagle:package:24925/1" value="1k" x="114.173" y="24.384" smashed="yes">
 <attribute name="MF" value="" x="114.173" y="24.384" size="1.778" layer="27" display="off"/>
 <attribute name="MPN" value="" x="114.173" y="24.384" size="1.778" layer="27" display="off"/>

Commit message: RS422 opto galv isolation added
Parts:
- added C42, C43: 100n, rcl:C0805
- added C44: ~0, rcl:C0805
- added D10: 3V6, diodes:DMELF
- added IC8: MOCD207MSOIC-8, Opto-Electronic:SOIC127P594X363-8N
- added R11, R12: 3k, rcl:R0805
- added R13, R14: ~10k, rcl:R0805
- added R15: 500, rcl:R0805
- added R16, R17: 3k3, rcl:R0805
- added U$1: LM78L05ACMX/NOPB, m-pad-2.1:SOIC8
- D5, D6: value 3V6 -> ~5V2
- R10: value 1k -> 500
Connections:
- new net 5V-28V: C43.1, IC5.1, R14.2, R16.1, U$1.1
- new net EXP_IN_OPT: D10.C, IC8.8, R13.1
- new net EXP_OUT_OPT: IC8.3
- new net N$44: IC8.4, R12.2
- new net N$49: IC8.2, R11.2
- new net N$50: C44.1, R10.1, R15.2
- net 28V: now also C42.2, U$1.8
- net 28VGND: now also C42.1, C43.2, C44.2, D5.A, D6.A, IC5.4, IC8.5, R11.1, R17.1, U$1.2, U$1.3, U$1.6, U$1.7
- net 3V3: now also R13.2; no longer IC5.1
- net EXP_IN: now also IC8.1
- net EXP_IN_N: now also R15.1, R17.2; no longer R10.1
- net EXP_IN_P: now also R16.2
- net EXP_OUT: now also IC8.6, R14.1
- net GND: now also D10.A, IC8.7, R12.1; no longer D5.A, D6.A, IC5.4
Routing:
- net GND: track 1002.7 -> 997.7 mm
- net 3V3: track 700.1 -> 695.8 mm
- net EXP_IN_N: track 41.9 -> 38.8 mm

Commit message: rerouting
Parts:
- moved R17 198.6 mm to (123.8, 45.7)
- moved R16 193.4 mm to (123.8, 43.2)
- moved R15 193.2 mm to (130.2, 45.7), turned to 90 degrees
- moved C44 192.7 mm to (123.8, 48.3), turned to 180 degrees
- moved R14 173.0 mm to (117.5, 39.4), turned to 90 degrees
- moved R13 163.8 mm to (116.8, 25.4), turned to 270 degrees
- moved C42 163.6 mm to (130.2, 50.2), turned to 90 degrees
- moved R12 161.7 mm to (118.1, 22.2), flipped to the bottom, turned to 270 degrees
- moved R11 157.8 mm to (116.8, 19.7), turned to 270 degrees
- moved IC8 156.4 mm to (123.8, 19.7), turned to 90 degrees
- moved C43 156.1 mm to (118.4, 51.9), turned to 270 degrees
- moved U$1 153.8 mm to (123.8, 52.1), turned to 270 degrees
- moved D10 147.8 mm to (74.9, 52.1), flipped to the bottom, turned to 180 degrees
- moved SV1 47.1 mm to (87.6, 21.0), turned to 225 degrees
- moved D5 29.9 mm to (116.2, 35.6), turned to 90 degrees
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Connections:
- net 28V: no longer X1.8
- net 28VGND: now also X1.8
- net EXP_IN: no longer U9.200
- net EXP_IN_OPT: now also U9.200
- net EXP_OUT: no longer U9.201
- net EXP_OUT_OPT: now also U9.201
- net LED_1: now also U9.24
- net LED_2: now also U9.23
- net LED_3: now also U9.22
- net LED_4: now also U9.21
Routing:
- net GND: track 997.7 -> 1147.5 mm, vias 144 -> 59
- net 28VGND: track 47.0 -> 192.7 mm, vias 2 -> 5
- net 3V3: track 695.8 -> 567.1 mm, vias 20 -> 18
- net 5V: track 265.2 -> 177.5 mm, vias 4 -> 5
- net EXP_IN_OPT: track 0.00 -> 72.7 mm, vias 0 -> 2
- net LED_1: track 0.00 -> 69.0 mm, vias 0 -> 4
- net LED_2: track 0.00 -> 68.2 mm, vias 0 -> 4
- net LED_3: track 0.00 -> 67.4 mm, vias 0 -> 4
- net LED_4: track 0.00 -> 66.5 mm, vias 0 -> 4
- net EXP_OUT_OPT: track 0.00 -> 52.6 mm
- net ADC3_RES: track 66.9 -> 30.6 mm, vias 4 -> 2
- net EXP_IN_N: track 38.8 -> 70.9 mm, vias 0 -> 1
- net EXP_IN_P: track 33.6 -> 63.2 mm, vias 0 -> 3
- net OUT_PT_2: track 113.7 -> 87.4 mm, vias 2 -> 4
- net SPI5_CS: track 51.5 -> 25.6 mm
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- added copper zone on layer 1, net 28VGND
- added copper zone on layer 16, net 28VGND

Commit message: ground vias
Parts:
- added LED5, LED6, LED7, LED8: (no value), adafruit:CHIP-LED0603
- added R18, R19, R20, R21: ?, rcl:R0805
- moved LED1 2.54 mm to (152.4, 81.3)
- moved LED2 1.91 mm to (154.3, 81.3)
- moved LED3 1.27 mm to (156.2, 81.3)
- moved LED4 0.64 mm to (158.1, 81.3)
Connections:
- new net N$51: LED5.A, R18.1
- new net N$52: LED6.A, R19.1
- new net N$55: LED7.A, R20.1
- new net N$56: LED8.A, R21.1
- net 28V: now also R20.2
- net 28VGND: now also LED7.C, LED8.C
- net 3V3: now also R19.2
- net 5V: now also R18.2
- net 5V-28V: now also R21.2
- net GND: now also LED5.C, LED6.C
Routing:
- net 5V: track 177.5 -> 341.1 mm, vias 5 -> 17
- net 3V3: track 567.1 -> 692.4 mm, vias 18 -> 26
- net GND: track 1147.5 -> 1194.8 mm, vias 59 -> 141
- net 5V-28V: track 22.4 -> 58.9 mm, vias 2 -> 3
- net N$32: track 23.4 -> 29.9 mm, vias 0 -> 2
- net N$55: track 0.00 -> 5.97 mm, vias 0 -> 1
- net N$56: track 0.00 -> 5.27 mm, vias 0 -> 1
- net 28VGND: track 192.7 -> 197.3 mm, vias 5 -> 35
- net N$52: track 0.00 -> 4.52 mm, vias 0 -> 1
- net N$51: track 0.00 -> 4.52 mm, vias 0 -> 1
- net N$30: track 16.8 -> 20.3 mm
- net N$33: track 29.8 -> 31.9 mm
- net N$31: track 20.3 -> 22.3 mm
- net 28V: track 97.8 -> 99.7 mm, vias 2 -> 3
- net TCK: track 95.7 -> 97.2 mm
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