File: Blade.sch (EAGLE design)
At the start: 132 parts, among them IC1 THN10-2411WIR, IC2 MCP6064-E/SL, IC3 MCP6064-E/SL, IC4 MCP6064-E/SL, IC5 MAX488CSA, IC6 MOCD207MSOIC-8, IC7 MOCD207MSOIC-8, IC8 MOCD207MSOIC-8, Q1 12MHz, U1 ADR366WAUJZ, U2 ADR366WAUJZ, U3 ADS1148QPWRQ1, U4 ADS1148QPWRQ1, U5 ADS1148QPWRQ1, U6 LT1528, U7 S70FL01GS, U8 S70FL01GS, U9 STM32F77XXXLQFP208, X1 D-SUB9-H5M09RA, X2 D-SUB15-H5M15RA, X3 USBPTH

Commit message: ads added
Parts:
- added C45, C46, C48, C49: 100n, rcl:C-EUC0805
- added C47, C50, C53: 1u, rcl:C-EUC0805
- added C54, C57: 10n, rcl:C-EUC0805
- added C55, C58: 10u, rcl:C-EUC0805
- added IC10, IC9: MCP6064-E/SL, linear:MCP604SL
- added L4, L5: 1m, rcl:L-EUL5650M
- added RN13, RN14, RN15, RN16, RN17, RN18: ?, resistor-dil:4R-NEXBS8V
- added U10, U11, U12: ADS1148QPWRQ1, ads11xx:ADS1148QPWRQ1
- added X_IN_10, X_IN_11, X_IN_12, X_IN_13, X_IN_14, X_IN_15: (no value), adafruit:SMACONNECTOR_EDGE
- RN1, RN4: value 56k -> ?
- RN2, RN5: value 5k6 -> ?
- RN3, RN6: value 330 -> ?
Connections:
- new net IN_DMS_10: IC9D.-IN, RN15A.1, X_IN_13.ANT
- new net IN_DMS_11: IC10A.-IN, RN18D.1, X_IN_14.ANT
- new net IN_DMS_12: IC10B.-IN, RN18C.1, X_IN_15.ANT
- new net IN_DMS_7: IC9A.-IN, RN15D.1, X_IN_10.ANT
- new net IN_DMS_8: IC9B.-IN, RN15C.1, X_IN_11.ANT
- new net IN_DMS_9: IC9C.-IN, RN15B.1, X_IN_12.ANT
- new net N$53: C47.1, U10.VREFOUT
- new net N$54: C50.1, U11.VREFOUT
- new net N$57: C53.1, U12.VREFOUT
- new net N$58: IC9A.+IN, RN13D.2, RN14D.1
- new net N$59: IC9B.+IN, RN13C.2, RN14C.1
- new net N$60: IC9C.+IN, RN13B.2, RN14B.1
- new net N$61: IC9D.+IN, RN13A.2, RN14A.1
- new net N$62: C54.2, IC9P.V+, L4.2
- new net N$63: IC10A.+IN, RN16D.2, RN17D.1
- new net N$64: IC10B.+IN, RN16C.2, RN17C.1
- new net N$65: RN16B.2, RN17B.1
- new net N$66: RN16A.2, RN17A.1
- new net N$67: C57.2, IC10P.V+, L5.2
- new net OUT_DMS_10: IC9D.OUT, RN15A.2, U10.AIN2/IEXC/GPIO2
- new net OUT_DMS_11: IC10A.OUT, RN18D.2, U12.AIN0/IEXC
- new net OUT_DMS_12: IC10B.OUT, RN18C.2, U12.AIN2/IEXC/GPIO2
- new net OUT_DMS_7: IC9A.OUT, RN15D.2, U11.AIN0/IEXC
- new net OUT_DMS_8: IC9B.OUT, RN15C.2, U11.AIN2/IEXC/GPIO2
- new net OUT_DMS_9: IC9C.OUT, RN15B.2, U10.AIN0/IEXC
- new net SPI3_CS2: U11.!CS
- new net SPI4_CS2: U10.!CS
- new net SPI5_CS2: U12.!CS
- net 3V3: now also C45.1, C46.1, C48.1, C49.1, L4.1, L5.1, U10.AVDD, U10.DVDD, U11.AVDD, U11.DVDD, U12.AVDD, U12.DVDD
- net 3V3REF: now also C55.2, RN13A.1, RN13B.1, RN13C.1, RN13D.1
- net 3V3REF2: now also C58.2, RN16A.1, RN16B.1, RN16C.1, RN16D.1
- net ADC1_DRDY: now also U11.!DRDY
- net ADC1_RES: now also U11.!RESET
- net ADC1_START: now also U11.START
- net ADC2_DRDY: now also U10.!DRDY
- net ADC2_RES: now also U10.!RESET
- net ADC2_START: now also U10.START
- net ADC3_DRDY: now also U12.!DRDY
- net ADC3_RES: now also U12.!RESET
- net ADC3_START: now also U12.START
- net GND: now also C45.2, C46.2, C47.2, C48.2, C49.2, C50.2, C53.2, C54.1, C55.1, C57.1, C58.1, IC10P.V-, IC9P.V-, RN14A.2, RN14B.2, RN14C.2, RN14D.2, RN17A.2, RN17B.2, RN17C.2, RN17D.2, U10.AVSS, U10.CLK, U10.DGND/DSS, U10.VREFCOM, U11.AVSS, U11.CLK, U11.DGND/DSS, U11.VREFCOM, U12.AVSS, U12.CLK, U12.DGND/DSS, U12.VREFCOM, X_IN_10.GND1, X_IN_10.GND2, X_IN_10.GND3, X_IN_10.GND4, X_IN_11.GND1, X_IN_11.GND2, X_IN_11.GND3, X_IN_11.GND4, X_IN_12.GND1, X_IN_12.GND2, X_IN_12.GND3, X_IN_12.GND4, X_IN_13.GND1, X_IN_13.GND2, X_IN_13.GND3, X_IN_13.GND4, X_IN_14.GND1, X_IN_14.GND2, X_IN_14.GND3, X_IN_14.GND4, X_IN_15.GND1, X_IN_15.GND2, X_IN_15.GND3, X_IN_15.GND4
- net SPI3_MISO: now also U11.DOUT/!DRDY
- net SPI3_MOSI: now also U11.DIN
- net SPI3_SCK: now also U11.SCLK
- net SPI4_MISO: now also U10.DOUT/!DRDY
- net SPI4_MOSI: now also U10.DIN
- net SPI4_SCK: now also U10.SCLK
- net SPI5_MISO: now also U12.DOUT/!DRDY
- net SPI5_MOSI: now also U12.DIN
- net SPI5_SCK: now also U12.SCLK

Commit message: Foo
Connections:
- removed net 3V3REF3: U9.VREF+
- net 3V3REF2: now also U9.VREF+
- net SPI3_CS2: now also U9.PF2
- net SPI4_CS2: now also U9.PI12
- net SPI5_CS2: now also U9.PI13
Changed lines of the file:
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@@
 </segment>
 </net>
-<net name="3V3REF3" class="0">
+<net name="3V3REF2" class="0">
 <segment>
 <pinref part="U9" gate="G$1" pin="VREF+"/>
@@
 </segment>
 </net>
+<net name="SPI3_CS2" class="0">
+<segment>
+<pinref part="U9" gate="G$1" pin="PF2"/>
+<wire x1="292.1" y1="142.24" x2="292.1" y2="137.16" width="0.1524" layer="91"/>
+<label x="292.1" y="137.16" size="1.27" layer="95" rot="R270" xref="yes"/>
+</segment>
+</net>
+<net name="SPI4_CS2" class="0">
+<segment>
+<pinref part="U9" gate="G$1" pin="PI12"/>
+<wire x1="210.82" y1="391.16" x2="205.74" y2="391.16" width="0.1524" layer="91"/>
+<label x="205.74" y="391.16" size="1.27" layer="95" rot="R180" xref="yes"/>
+</segment>
+</net>
+<net name="SPI5_CS2" class="0">
+<segment>
+<pinref part="U9" gate="G$1" pin="PI13"/>
+<wire x1="210.82" y1="396.24" x2="205.74" y2="396.24" width="0.1524" layer="91"/>
+<label x="205.74" y="396.24" size="1.27" layer="95" rot="R180" xref="yes"/>
+</segment>
+</net>
