File: SPU_Rev_2.0.sch (EAGLE design)
At the start: 140 parts, among them Q1 12MHz, X2 D-SUB15-H5M15RA

Commit message: NOP
Changed lines of the file:
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@@
 <grid distance="0.1" unitdist="inch" unit="inch" style="lines" multiple="1" display="yes" altdistance="0.01" altunitdist="inch" altunit="inch"/>
 <layers>
-<layer number="1" name="Top" color="4" fill="1" visible="yes" active="no"/>
-<layer number="2" name="Route2" color="16" fill="1" visible="yes" active="no"/>
-<layer number="3" name="Route3" color="17" fill="1" visible="yes" active="no"/>
-<layer number="4" name="Route4" color="18" fill="1" visible="yes" active="no"/>
-<layer number="5" name="Route5" color="19" fill="1" visible="yes" active="no"/>
-<layer number="6" name="Route6" color="25" fill="1" visible="yes" active="no"/>
-<layer number="7" name="Route7" color="26" fill="1" visible="yes" active="no"/>
-<layer number="8" name="Route8" color="27" fill="1" visible="yes" active="no"/>
-<layer number="9" name="Route9" color="28" fill="1" visible="yes" active="no"/>
-<layer number="10" name="Route10" color="29" fill="1" visible="yes" active="no"/>
-<layer number="11" name="Route11" color="30" fill="1" visible="yes" active="no"/>
-<layer number="12" name="Route12" color="20" fill="1" visible="yes" active="no"/>
-<layer number="13" name="Route13" color="21" fill="1" visible="yes" active="no"/>
-<layer number="14" name="Route14" color="22" fill="1" visible="yes" active="no"/>
-<layer number="15" name="Route15" color="23" fill="1" visible="yes" active="no"/>
-<layer number="16" name="Bottom" color="1" fill="1" visible="yes" active="no"/>
-<layer number="17" name="Pads" color="2" fill="1" visible="yes" active="no"/>
-<layer number="18" name="Vias" color="2" fill="1" visible="yes" active="no"/>
-<layer number="19" name="Unrouted" color="6" fill="1" visible="yes" active="no"/>
-<layer number="20" name="Dimension" color="24" fill="1" visible="yes" active="no"/>
-<layer number="21" name="tPlace" color="7" fill="1" visible="yes" active="no"/>
-<layer number="22" name="bPlace" color="7" fill="1" visible="yes" active="no"/>
-<layer number="23" name="tOrigins" color="15" fill="1" visible="yes" active="no"/>
-<layer number="24" name="bOrigins" color="15" fill="1" visible="yes" active="no"/>
-<layer number="25" name="tNames" color="7" fill="1" visible="yes" active="no"/>
-<layer number="26" name="bNames" color="7" fill="1" visible="yes" active="no"/>
-<layer number="27" name="tValues" color="7" fill="1" visible="yes" active="no"/>
-<layer number="28" name="bValues" color="7" fill="1" visible="yes" active="no"/>
+<layer number="1" name="Top" color="4" fill="1" visible="no" active="no"/>
+<layer number="2" name="Route2" color="16" fill="1" visible="no" active="no"/>
+<layer number="3" name="Route3" color="17" fill="1" visible="no" active="no"/>
+<layer number="4" name="Route4" color="18" fill="1" visible="no" active="no"/>
+<layer number="5" name="Route5" color="19" fill="1" visible="no" active="no"/>
+<layer number="6" name="Route6" color="25" fill="1" visible="no" active="no"/>
+<layer number="7" name="Route7" color="26" fill="1" visible="no" active="no"/>
+<layer number="8" name="Route8" color="27" fill="1" visible="no" active="no"/>
+<layer number="9" name="Route9" color="28" fill="1" visible="no" active="no"/>
+<layer number="10" name="Route10" color="29" fill="1" visible="no" active="no"/>
+<layer number="11" name="Route11" color="30" fill="1" visible="no" active="no"/>
+<layer number="12" name="Route12" color="20" fill="1" visible="no" active="no"/>
+<layer number="13" name="Route13" color="21" fill="1" visible="no" active="no"/>
+<layer number="14" name="Route14" color="22" fill="1" visible="no" active="no"/>
+<layer number="15" name="Route15" color="23" fill="1" visible="no" active="no"/>
+<layer number="16" name="Bottom" color="1" fill="1" visible="no" active="no"/>
+<layer number="17" name="Pads" color="2" fill="1" visible="no" active="no"/>
+<layer number="18" name="Vias" color="2" fill="1" visible="no" active="no"/>
+<layer number="19" name="Unrouted" color="6" fill="1" visible="no" active="no"/>
+<layer number="20" name="Dimension" color="24" fill="1" visible="no" active="no"/>
+<layer number="21" name="tPlace" color="7" fill="1" visible="no" active="no"/>
+<layer number="22" name="bPlace" color="7" fill="1" visible="no" active="no"/>
+<layer number="23" name="tOrigins" color="15" fill="1" visible="no" active="no"/>
+<layer number="24" name="bOrigins" color="15" fill="1" visible="no" active="no"/>
+<layer number="25" name="tNames" color="7" fill="1" visible="no" active="no"/>
+<layer number="26" name="bNames" color="7" fill="1" visible="no" active="no"/>
+<layer number="27" name="tValues" color="7" fill="1" visible="no" active="no"/>
+<layer number="28" name="bValues" color="7" fill="1" visible="no" active="no"/>
 <layer number="29" name="tStop" color="7" fill="3" visible="no" active="no"/>
 <layer number="30" name="bStop" color="7" fill="6" visible="no" active="no"/>
@@
 <layer number="35" name="tGlue" color="7" fill="4" visible="no" active="no"/>
 <layer number="36" name="bGlue" color="7" fill="5" visible="no" active="no"/>
-<layer number="37" name="tTest" color="7" fill="1" visible="yes" active="no"/>
-<layer number="38" name="bTest" color="7" fill="1" visible="yes" active="no"/>
+<layer number="37" name="tTest" color="7" fill="1" visible="no" active="no"/>
+<layer number="38" name="bTest" color="7" fill="1" visible="no" active="no"/>
 <layer number="39" name="tKeepout" color="4" fill="11" visible="no" active="no"/>
 <layer number="40" name="bKeepout" color="1" fill="11" visible="no" active="no"/>
@@
 <layer number="44" name="Drills" color="7" fill="1" visible="no" active="no"/>
 <layer number="45" name="Holes" color="7" fill="1" visible="no" active="no"/>
-<layer number="46" name="Milling" color="3" fill="1" visible="yes" active="no"/>
-<layer number="47" name="Measures" color="7" fill="1" visible="yes" active="no"/>
-<layer number="48" name="Document" color="7" fill="1" visible="yes" active="no"/>
-<layer number="49" name="Reference" color="7" fill="1" visible="yes" active="no"/>
-<layer number="50" name="dxf" color="7" fill="1" visible="yes" active="no"/>
-<layer number="51" name="tDocu" color="7" fill="1" visible="yes" active="no"/>
-<layer number="52" name="bDocu" color="7" fill="1" visible="yes" active="no"/>
-<layer number="53" name="tGND_GNDA" color="7" fill="9" visible="yes" active="no"/>
-<layer number="54" name="bGND_GNDA" color="1" fill="9" visible="yes" active="no"/>
-<layer number="56" name="wert" color="7" fill="1" visible="yes" active="no"/>
-<layer number="57" name="tCAD" color="7" fill="1" visible="yes" active="no"/>
-<layer number="58" name="bCAD" color="7" fill="1" visible="yes" active="no"/>
-<layer number="59" name="tCarbon" color="7" fill="1" visible="yes" active="no"/>
-<layer number="60" name="bCarbon" color="7" fill="1" visible="yes" active="no"/>
+<layer number="46" name="Milling" color="3" fill="1" visible="no" active="no"/>
+<layer number="47" name="Measures" color="7" fill="1" visible="no" active="no"/>
+<layer number="48" name="Document" color="7" fill="1" visible="no" active="no"/>
+<layer number="49" name="Reference" color="7" fill="1" visible="no" active="no"/>
+<layer number="50" name="dxf" color="7" fill="1" visible="no" active="no"/>
+<layer number="51" name="tDocu" color="7" fill="1" visible="no" active="no"/>
+<layer number="52" name="bDocu" color="7" fill="1" visible="no" active="no"/>
+<layer number="53" name="tGND_GNDA" color="7" fill="9" visible="no" active="no"/>
+<layer number="54" name="bGND_GNDA" color="1" fill="9" visible="no" active="no"/>
+<layer number="56" name="wert" color="7" fill="1" visible="no" active="no"/>
+<layer number="57" name="tCAD" color="7" fill="1" visible="no" active="no"/>
+<layer number="58" name="bCAD" color="7" fill="1" visible="no" active="no"/>
+<layer number="59" name="tCarbon" color="7" fill="1" visible="no" active="no"/>
+<layer number="60" name="bCarbon" color="7" fill="1" visible="no" active="no"/>
 <layer number="88" name="SimResults" color="9" fill="1" visible="yes" active="yes"/>
 <layer number="89" name="SimProbes" color="9" fill="1" visible="yes" active="yes"/>
@@
 <wire x1="25.4" y1="96.52" x2="25.4" y2="132.08" width="0.1524" layer="94" style="shortdash"/>
 <wire x1="25.4" y1="132.08" x2="96.52" y2="132.08" width="0.1524" layer="94" style="shortdash"/>
-<text x="116.84" y="-99.568" size="7.62" layer="94">all logic sided on this page</text>
+<text x="200.66" y="-99.568" size="7.62" layer="94">all logic sided on this page</text>
 <text x="523.24" y="254" size="5.08" layer="94">TODO for Rev 2.1
    12 DMS-Paare (ergo 24 DMS), pro SPU 6 DMS-Paare

Commit message: NOT final
Connections:
- net 3V3REF3 renamed 3V3REF
Changed lines of the file:
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@@
 <?xml version="1.0" encoding="utf-8"?>
 <!DOCTYPE eagle SYSTEM "eagle.dtd">
-<eagle version="9.3.1">
+<eagle version="9.6.2">
 <drawing>
 <settings>
-<setting alwaysvectorfont="yes"/>
+<setting alwaysvectorfont="no"/>
 <setting verticaltext="up"/>
 </settings>
@@
 </segment>
 </net>
-<net name="3V3REF3" class="0">
+<net name="3V3REF" class="0">
 <segment>
 <pinref part="U_STM32F779" gate="G$1" pin="VREF+"/>
@@
 </segment>
 </net>
-<net name="3V3REF3" class="0">
+<net name="3V3REF" class="0">
 <segment>
 <pinref part="U_ADR366_3" gate="G$1" pin="VOUT"/>

Commit message: foo
bar
Parts:
- removed X2: D-SUB15-H5M15RA, con-thomas-betts:D-SUB15-H5M15RA
- removed X_DAPI: USBPTH, aSparkFun:USBPTH
- added X_RXSM-DAPI: 403-5X020-5X, con-ept-One27:403-5X020-5X
Connections:
- removed net N$10: X2-10.F
- removed net N$11: X2-11.F
- removed net N$12: X2-12.F
- removed net N$2: X2-2.F
- net 28V: now also X_RXSM-DAPI.B1, X_RXSM-DAPI.B2; no longer X2-1.F, X2-9.F
- net 28VGND: now also X_RXSM-DAPI.A1, X_RXSM-DAPI.A2, X_RXSM-DAPI.A6; no longer X2-15.F, X2-8.F
- net 5V: now also X_RXSM-DAPI.A9; no longer X_DAPI.VBUS
- net DAPI_N: now also X_RXSM-DAPI.B9; no longer X_DAPI.D-
- net DAPI_P: now also X_RXSM-DAPI.B10; no longer X_DAPI.D+
- net EXP_IN_N: now also X_RXSM-DAPI.B3; no longer X2-14.F
- net EXP_IN_P: now also X_RXSM-DAPI.B4; no longer X2-13.F
- net EXP_OUT_N: now also X_RXSM-DAPI.A3; no longer X2-7.F
- net EXP_OUT_P: now also X_RXSM-DAPI.A4; no longer X2-6.F
- net GND: now also X_RXSM-DAPI.A10; no longer X_DAPI.GND
- net LO: now also X_RXSM-DAPI.A5; no longer X2-5.F
- net SODS: now also X_RXSM-DAPI.B6; no longer X2-3.F
- net SOE: now also X_RXSM-DAPI.B5; no longer X2-4.F
Other:
- moved on the sheet: X_PROG

Commit message: rev 2.1
Parts:
- added C10, C12, C13, C14, C15, C19, C21, C22, C23, C24, C25, C27, C3, C45, C46, C47, C48, C5, C50, C51, C53, C54, C55, C57, C58, C59, C6, C7, C8, C9: 100n, rcl:C-EUC0603
- added C11, C20, C26, C4, C49, C56: 1u, rcl:C-EUC1206
- added R1, R2, R30, R36, R37, R43, R44, R50, R51, R57, R58, R8: 4k7, ++Bedrahtet:R-EU_R0603
- added R3, R31, R38, R45, R52, R59: 47, ++Bedrahtet:R-EU_R0603
- added R32, R33, R39, R4, R40, R46, R47, R5, R53, R54, R60, R61: 40 1%, ++Bedrahtet:R-EU_R0805
- added R34, R35, R41, R42, R48, R49, R55, R56, R6, R62, R63, R7: 1k 0.1%, ++Bedrahtet:R-EU_R0805
- added RN_DMS1, RN_DMS2, RN_DMS3, RN_DMS4, RN_DMS5, RN_DMS6: 47, resistor-dil:4R-N0603-ARC
- added U$1, U$2, U$3, U$4, U$5, U$6: COMMON_MODE_CHOKE, selfmade:COMMON_MODE_CHOKE
- added U_ADC_DMS1, U_ADC_DMS2, U_ADC_DMS3, U_ADC_DMS4, U_ADC_DMS5, U_ADC_DMS6: ADS1147TSSOP20, ads11xx:ADS1147TSSOP20
- added X1: 403-5X020-5X, con-ept-One27:403-5X020-5X
- renumbered S70FL01GS_2 to U_S70FL01GS_2
Connections:
- net PT1_DIN renamed PT_DIN
- net PT1_DOUT renamed PT_DOUT
- net PT1_SCLK renamed PT_SCLK
- removed net PT1_!CS: RN_B_PT1B.2, RN_B_PT2B.2, RN_B_PT3B.2
- removed net PT1_!DRDY: RN_B_PT1A.2, RN_B_PT2A.2, RN_B_PT3A.2
- removed net PT1_!RESET: RN_A_PT1A.2, RN_A_PT2A.2, RN_A_PT3A.2
- removed net PT1_START: RN_B_PT1C.2, RN_B_PT2C.2, RN_B_PT3C.2
- new net !CS!_DMS1: R3.2
- new net !CS!_DMS2: R31.2
- new net !CS!_DMS3: R38.2
- new net !CS!_DMS4: R45.2
- new net !CS!_DMS5: R52.2
- new net !CS!_DMS6: R59.2
- new net !CS!_PT1: RN_B_PT1B.2
- new net !CS!_PT2: RN_B_PT2B.2
- new net !CS!_PT3: RN_B_PT3B.2
- new net !DRDY!_DMS1: RN_DMS1D.2
- new net !DRDY!_DMS2: RN_DMS2D.2
- new net !DRDY!_DMS3: RN_DMS3D.2
- new net !DRDY!_DMS4: RN_DMS4D.2
- new net !DRDY!_DMS5: RN_DMS5D.2
- new net !DRDY!_DMS6: RN_DMS6D.2
- new net !DRDY!_PT1: RN_B_PT1A.2
- new net !DRDY!_PT2: RN_B_PT2A.2
- new net !DRDY!_PT3: RN_B_PT3A.2
- new net DMS11: U$2.1, X1.B3
- new net DMS12: U$2.3, X1.B2
- new net DMS13: U$2.5, X1.B1
- new net DMS21: U$1.1, X1.B6
- new net DMS22: U$1.3, X1.B5
- new net DMS23: U$1.5, X1.B4
- new net DMS31: U$3.1, X1.B9
- new net DMS32: U$3.3, X1.B8
- new net DMS33: U$3.5, X1.B7
- new net DMS41: U$4.1, X1.A1
- new net DMS42: U$4.3, X1.A2
- new net DMS43: U$4.5, X1.A3
- new net DMS51: U$5.1, X1.A4
- new net DMS52: U$5.3, X1.A5
- new net DMS53: U$5.5, X1.A6
- new net DMS61: U$6.1, X1.A7
- new net DMS62: U$6.3, X1.A8
- new net DMS63: U$6.5, X1.A9
- new net DMS_DIN: RN_DMS1B.2, RN_DMS2B.2, RN_DMS3B.2, RN_DMS4B.2, RN_DMS5B.2, RN_DMS6B.2
- new net DMS_DOUT: RN_DMS1C.2, RN_DMS2C.2, RN_DMS3C.2, RN_DMS4C.2, RN_DMS5C.2, RN_DMS6C.2
- new net DMS_SCLK: RN_DMS1A.2, RN_DMS2A.2, RN_DMS3A.2, RN_DMS4A.2, RN_DMS5A.2, RN_DMS6A.2
- new net N$10: RN_DMS1A.1, U_ADC_DMS1.SCLK
- new net N$100: RN_DMS3D.1, U_ADC_DMS3.!DRDY
- new net N$101: R38.1, U_ADC_DMS3.!CS
- new net N$102: C27.2, C45.1, R46.1, U_ADC_DMS4.AIN0/IEXC
- new net N$103: C45.2, C46.1, R47.1, U_ADC_DMS4.AIN1/IEXC
- new net N$104: R47.2, R48.1, R49.1
- new net N$105: C26.1, U_ADC_DMS4.VREFOUT
- new net N$106: R46.2, U$4.4
- new net N$107: R43.2, U_ADC_DMS4.!RESET
- new net N$108: R44.1, U_ADC_DMS4.START
- new net N$109: RN_DMS4A.1, U_ADC_DMS4.SCLK
- new net N$11: C13.2, C14.1, R33.1, U_ADC_DMS2.AIN1/IEXC
- new net N$110: RN_DMS4B.1, U_ADC_DMS4.DIN
- new net N$111: RN_DMS4C.1, U_ADC_DMS4.DOUT/!DRDY
- new net N$112: RN_DMS4D.1, U_ADC_DMS4.!DRDY
- new net N$113: R45.1, U_ADC_DMS4.!CS
- new net N$114: C50.2, C51.1, R53.1, U_ADC_DMS5.AIN0/IEXC
- new net N$115: C51.2, C53.1, R54.1, U_ADC_DMS5.AIN1/IEXC
- new net N$116: R54.2, R55.1, R56.1
- new net N$117: C49.1, U_ADC_DMS5.VREFOUT
- new net N$118: R53.2, U$5.4
- new net N$119: R50.2, U_ADC_DMS5.!RESET
- new net N$12: R33.2, R34.1, R35.1
- new net N$120: R51.1, U_ADC_DMS5.START
- new net N$121: RN_DMS5A.1, U_ADC_DMS5.SCLK
- new net N$122: RN_DMS5B.1, U_ADC_DMS5.DIN
- new net N$123: RN_DMS5C.1, U_ADC_DMS5.DOUT/!DRDY
- new net N$124: RN_DMS5D.1, U_ADC_DMS5.!DRDY
- new net N$125: R52.1, U_ADC_DMS5.!CS
- new net N$127: C47.1, R50.1, U_ADC_DMS5.DVDD
- new net N$128: C57.2, C58.1, R60.1, U_ADC_DMS6.AIN0/IEXC
- new net N$129: C58.2, C59.1, R61.1, U_ADC_DMS6.AIN1/IEXC
- new net N$130: R61.2, R62.1, R63.1
- new net N$131: C56.1, U_ADC_DMS6.VREFOUT
- new net N$132: R60.2, U$6.4
- new net N$133: R57.2, U_ADC_DMS6.!RESET
- new net N$134: R58.1, U_ADC_DMS6.START
- new net N$135: RN_DMS6A.1, U_ADC_DMS6.SCLK
- new net N$136: RN_DMS6B.1, U_ADC_DMS6.DIN
- new net N$137: RN_DMS6C.1, U_ADC_DMS6.DOUT/!DRDY
- new net N$138: RN_DMS6D.1, U_ADC_DMS6.!DRDY
- new net N$139: R59.1, U_ADC_DMS6.!CS
- new net N$141: C54.1, R57.1, U_ADC_DMS6.DVDD
- new net N$148: X1.B10
- new net N$157: X1.A10
- new net N$2: R2.1, U_ADC_DMS1.START
- new net N$67: C11.1, U_ADC_DMS2.VREFOUT
- new net N$7: C12.2, C13.1, R32.1, U_ADC_DMS2.AIN0/IEXC
- new net N$72: R32.2, U$1.4
- new net N$73: R1.2, U_ADC_DMS1.!RESET
- new net N$74: RN_DMS1B.1, U_ADC_DMS1.DIN
- new net N$75: RN_DMS1C.1, U_ADC_DMS1.DOUT/!DRDY
- new net N$76: RN_DMS1D.1, U_ADC_DMS1.!DRDY
- new net N$77: R3.1, U_ADC_DMS1.!CS
- new net N$78: R8.2, U_ADC_DMS2.!RESET
- new net N$79: R30.1, U_ADC_DMS2.START
- new net N$80: C6.2, C7.1, R4.1, U_ADC_DMS1.AIN0/IEXC
- new net N$81: C7.2, C8.1, R5.1, U_ADC_DMS1.AIN1/IEXC
- new net N$82: R5.2, R6.1, R7.1
- new net N$83: C4.1, U_ADC_DMS1.VREFOUT
- new net N$84: R4.2, U$2.4
- new net N$85: RN_DMS2A.1, U_ADC_DMS2.SCLK
- new net N$86: RN_DMS2B.1, U_ADC_DMS2.DIN
- new net N$87: RN_DMS2C.1, U_ADC_DMS2.DOUT/!DRDY
- new net N$88: RN_DMS2D.1, U_ADC_DMS2.!DRDY
- new net N$89: R31.1, U_ADC_DMS2.!CS
- new net N$90: C21.2, C22.1, R39.1, U_ADC_DMS3.AIN0/IEXC
- new net N$91: C22.2, C23.1, R40.1, U_ADC_DMS3.AIN1/IEXC
- new net N$92: R40.2, R41.1, R42.1
- new net N$93: C20.1, U_ADC_DMS3.VREFOUT
- new net N$94: R39.2, U$3.4
- new net N$95: R36.2, U_ADC_DMS3.!RESET
- new net N$96: R37.1, U_ADC_DMS3.START
- new net N$97: RN_DMS3A.1, U_ADC_DMS3.SCLK
- new net N$98: RN_DMS3B.1, U_ADC_DMS3.DIN
- new net N$99: RN_DMS3C.1, U_ADC_DMS3.DOUT/!DRDY
- net 3V3: now also C10.1, C15.1, C19.1, C24.1, C25.1, C3.1, C48.1, C5.1, C55.1, C9.1, R1.1, R2.2, R30.2, R34.2, R36.1, R37.2, R41.2, R43.1, R44.2, R48.2, R51.2, R55.2, R58.2, R6.2, R62.2, R8.1, RN_A_PT1A.2, RN_A_PT2A.2, RN_A_PT3A.2, RN_B_PT1C.2, RN_B_PT2C.2, RN_B_PT3C.2, U$1.2, U$2.2, U$3.2, U$4.2, U$5.2, U$6.2, U_ADC_DMS1.AVDD, U_ADC_DMS1.DVDD, U_ADC_DMS2.AVDD, U_ADC_DMS2.DVDD, U_ADC_DMS3.AVDD, U_ADC_DMS3.DVDD, U_ADC_DMS4.AVDD, U_ADC_DMS4.DVDD, U_ADC_DMS5.AVDD, U_ADC_DMS6.AVDD
- net GND: now also C10.2, C11.2, C12.1, C14.2, C15.2, C19.2, C20.2, C21.1, C23.2, C24.2, C25.2, C26.2, C27.1, C3.2, C4.2, C46.2, C47.2, C48.2, C49.2, C5.2, C50.1, C53.2, C54.2, C55.2, C56.2, C57.1, C59.2, C6.1, C8.2, C9.2, R35.2, R42.2, R49.2, R56.2, R63.2, R7.2, U$1.6, U$2.6, U$3.6, U$4.6, U$5.6, U$6.6, U_ADC_DMS1.AVSS, U_ADC_DMS1.CLK, U_ADC_DMS1.DGND/DSS, U_ADC_DMS1.VREFCOM, U_ADC_DMS2.AVSS, U_ADC_DMS2.CLK, U_ADC_DMS2.DGND/DSS, U_ADC_DMS2.VREFCOM, U_ADC_DMS3.AVSS, U_ADC_DMS3.CLK, U_ADC_DMS3.DGND/DSS, U_ADC_DMS3.VREFCOM, U_ADC_DMS4.AVSS, U_ADC_DMS4.CLK, U_ADC_DMS4.DGND/DSS, U_ADC_DMS4.VREFCOM, U_ADC_DMS5.AVSS, U_ADC_DMS5.CLK, U_ADC_DMS5.DGND/DSS, U_ADC_DMS5.VREFCOM, U_ADC_DMS6.AVSS, U_ADC_DMS6.CLK, U_ADC_DMS6.DGND/DSS, U_ADC_DMS6.VREFCOM
Other:
- note added: "3dB attenuation @ 1989Hz"
- note added: "WE-SL3 SMT COMMON MODE LINE FILT"
- moved on the sheet: C_AVDD_PT1, C_AVDD_PT2, C_AVDD_PT3, C_DVDD_PT1, C_DVDD_PT2, C_DVDD_PT3, C_ICM1_PT1, C_ICM1_PT2, C_ICM1_PT3, C_ICM2_PT1, C_ICM2_PT2, C_ICM2_PT3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
