File: SPU_Rev_2.1.sch (EAGLE design)
At the start: 236 parts, among them Q1 12MHz, X1 403-5X020-5X

Commit message: renamed to 2.1
Parts:
- added C60, C61, C62, C63, C64, C65, C66, C67: 10u, rcl:CPOL-EUE/7260-38W
- added D13: (no value), special:7SEG-CA
- added RN_SEG1, RN_SEG2: 220, resistor-dil:4R-N0603-ARC
Connections:
- new net N$126: D13.A, RN_SEG1A.2
- new net N$140: D13.B, RN_SEG1B.2
- new net N$142: D13.C, RN_SEG1C.2
- new net N$143: D13.D, RN_SEG1D.2
- new net N$144: D13.E, RN_SEG2A.2
- new net N$145: D13.F, RN_SEG2B.2
- new net N$146: D13.G, RN_SEG2C.2
- new net N$147: D13.DP, RN_SEG2D.2
- new net N$149: RN_SEG2A.1
- new net N$150: RN_SEG1D.1
- new net N$151: RN_SEG1C.1
- new net N$152: RN_SEG1B.1
- new net N$153: RN_SEG1A.1
- new net N$154: RN_SEG2B.1
- new net N$155: RN_SEG2C.1
- new net N$156: RN_SEG2D.1
- net 28V: now also C60.+, C61.+, C62.+
- net 28VGND: now also C60.-, C61.-, C62.-
- net 3V3: now also C67.+, D13.CA1, D13.CA2
- net 5V: now also C63.+, C64.+, C65.+, C66.+
- net GND: now also C63.-, C64.-, C65.-, C66.-, C67.-

Commit message: foo
Parts:
- removed D13: (no value), special:7SEG-CA
- removed RN_SEG1, RN_SEG2: 220, resistor-dil:4R-N0603-ARC
- added C68, C69, C70, C71: 10u, rcl:CPOL-EUE/7260-38W
- added X_GPIO: 403-5X020-5X, con-ept-One27:403-5X020-5X
- renumbered X1 to X_DMS
Connections:
- removed net N$126: D13.A, RN_SEG1A.2
- removed net N$140: D13.B, RN_SEG1B.2
- removed net N$142: D13.C, RN_SEG1C.2
- removed net N$143: D13.D, RN_SEG1D.2
- removed net N$144: D13.E, RN_SEG2A.2
- removed net N$145: D13.F, RN_SEG2B.2
- removed net N$146: D13.G, RN_SEG2C.2
- removed net N$147: D13.DP, RN_SEG2D.2
- removed net N$149: RN_SEG2A.1
- removed net N$150: RN_SEG1D.1
- removed net N$151: RN_SEG1C.1
- removed net N$152: RN_SEG1B.1
- removed net N$153: RN_SEG1A.1
- removed net N$154: RN_SEG2B.1
- removed net N$155: RN_SEG2C.1
- removed net N$156: RN_SEG2D.1
- net 3V3: now also C68.+, C69.+, C70.+, C71.+, X_GPIO.B1, X_GPIO.B2; no longer D13.CA1, D13.CA2
- net GND: now also C68.-, C69.-, C70.-, C71.-, X_GPIO.A1, X_GPIO.A2
Other:
- note added: "GPIO"

Commit message: foo
Parts:
- added C72, C73: 10u, rcl:CPOL-EUE/7260-38W
Connections:
- net 3V3: now also C72.+, C73.+, U_CH340G.V3
- net GND: now also C72.-, C73.-
Changed lines of the file:
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@@
 <part name="C70" library="rcl" library_urn="urn:adsk.eagle:library:334" deviceset="CPOL-EU" device="E/7260-38W" package3d_urn="urn:adsk.eagle:package:23423/1" value="10u"/>
 <part name="C71" library="rcl" library_urn="urn:adsk.eagle:library:334" deviceset="CPOL-EU" device="E/7260-38W" package3d_urn="urn:adsk.eagle:package:23423/1" value="10u"/>
+<part name="C72" library="rcl" library_urn="urn:adsk.eagle:library:334" deviceset="CPOL-EU" device="E/7260-38W" package3d_urn="urn:adsk.eagle:package:23423/1" value="10u"/>
+<part name="C73" library="rcl" library_urn="urn:adsk.eagle:library:334" deviceset="CPOL-EU" device="E/7260-38W" package3d_urn="urn:adsk.eagle:package:23423/1" value="10u"/>
 </parts>
 <sheets>
@@
 <wire x1="254" y1="279.4" x2="198.12" y2="279.4" width="0.1524" layer="94" style="shortdash"/>
 <wire x1="198.12" y1="279.4" x2="198.12" y2="220.98" width="0.1524" layer="94" style="shortdash"/>
-<wire x1="287.02" y1="182.88" x2="317.5" y2="182.88" width="0.1524" layer="94" style="shortdash"/>
-<wire x1="317.5" y1="182.88" x2="317.5" y2="279.4" width="0.1524" layer="94" style="shortdash"/>
+<wire x1="287.02" y1="167.64" x2="317.5" y2="167.64" width="0.1524" layer="94" style="shortdash"/>
+<wire x1="317.5" y1="167.64" x2="317.5" y2="279.4" width="0.1524" layer="94" style="shortdash"/>
 <wire x1="317.5" y1="279.4" x2="287.02" y2="279.4" width="0.1524" layer="94" style="shortdash"/>
-<wire x1="287.02" y1="279.4" x2="287.02" y2="182.88" width="0.1524" layer="94" style="shortdash"/>
+<wire x1="287.02" y1="279.4" x2="287.02" y2="167.64" width="0.1524" layer="94" style="shortdash"/>
 <wire x1="203.2" y1="142.24" x2="353.06" y2="142.24" width="0.1524" layer="94" style="shortdash"/>
 <wire x1="353.06" y1="142.24" x2="353.06" y2="45.72" width="0.1524" layer="94" style="shortdash"/>
@@
 <attribute name="VALUE" x="297.4086" y="191.643" size="1.778" layer="96" rot="R270"/>
 </instance>
+<instance part="C72" gate="G$1" x="299.72" y="185.928" smashed="yes" rot="R90">
+<attribute name="NAME" x="302.9966" y="184.023" size="1.778" layer="95" rot="R270"/>
+<attribute name="VALUE" x="297.4086" y="184.023" size="1.778" layer="96" rot="R270"/>
+</instance>
+<instance part="C73" gate="G$1" x="299.72" y="178.308" smashed="yes" rot="R90">
+<attribute name="NAME" x="302.9966" y="176.403" size="1.778" layer="95" rot="R270"/>
+<attribute name="VALUE" x="297.4086" y="176.403" size="1.778" layer="96" rot="R270"/>
+</instance>
 </instances>
 <busses>
@@
 <junction x="307.086" y="208.28"/>
 <junction x="307.086" y="201.168"/>
+<pinref part="C72" gate="G$1" pin="-"/>
+<wire x1="307.086" y1="193.548" x2="307.086" y2="185.928" width="0.1524" layer="91"/>
+<wire x1="307.086" y1="185.928" x2="304.8" y2="185.928" width="0.1524" layer="91"/>
+<junction x="307.086" y="193.548"/>
+<pinref part="C73" gate="G$1" pin="-"/>
+<wire x1="307.086" y1="185.928" x2="307.086" y2="178.308" width="0.1524" layer="91"/>
+<wire x1="307.086" y1="178.308" x2="304.8" y2="178.308" width="0.1524" layer="91"/>
+<junction x="307.086" y="185.928"/>
 </segment>
 <segment>
@@
 <junction x="294.386" y="215.9"/>
 <pinref part="C70" gate="G$1" pin="+"/>
-<wire x1="294.64" y1="208.28" x2="297.18" y2="208.28" width="0.1524" layer="91"/>
+<wire x1="294.386" y1="208.28" x2="297.18" y2="208.28" width="0.1524" layer="91"/>
 <wire x1="297.18" y1="201.168" x2="294.386" y2="201.168" width="0.1524" layer="91"/>
 <pinref part="C71" gate="G$1" pin="+"/>
 <wire x1="294.386" y1="201.168" x2="294.386" y2="193.548" width="0.1524" layer="91"/>
 <wire x1="294.386" y1="193.548" x2="297.18" y2="193.548" width="0.1524" layer="91"/>
-<wire x1="294.64" y1="208.28" x2="294.386" y2="208.28" width="0.1524" layer="91"/>
 <wire x1="294.386" y1="208.28" x2="294.386" y2="201.168" width="0.1524" layer="91"/>
 <junction x="294.386" y="201.168"/>
+<pinref part="C72" gate="G$1" pin="+"/>
+<wire x1="294.386" y1="193.548" x2="294.386" y2="185.928" width="0.1524" layer="91"/>
+<wire x1="294.386" y1="185.928" x2="297.18" y2="185.928" width="0.1524" layer="91"/>
+<junction x="294.386" y="193.548"/>
+<pinref part="C73" gate="G$1" pin="+"/>
+<wire x1="294.386" y1="185.928" x2="294.386" y2="178.308" width="0.1524" layer="91"/>
+<wire x1="294.386" y1="178.308" x2="297.18" y2="178.308" width="0.1524" layer="91"/>
+<junction x="294.386" y="185.928"/>
 </segment>
 <segment>
@@
 <pinref part="R58" gate="G$1" pin="2"/>
 </segment>
+<segment>
+<pinref part="U_CH340G" gate="G$1" pin="V3"/>
+<wire x1="160.02" y1="96.52" x2="157.48" y2="96.52" width="0.1524" layer="91"/>
+<label x="157.48" y="96.52" size="1.27" layer="95" rot="R180" xref="yes"/>
+</segment>
 </net>

Commit message: some routing
Connections:
- removed net ADC1_DRDY: U_STM32F779.PJ0
- removed net ADC1_RES: U_STM32F779.PJ3
- removed net ADC1_START: U_STM32F779.PJ2
- removed net ADC2_DRDY: U_STM32F779.PH3
- removed net ADC2_RES: U_STM32F779.PA3
- removed net ADC2_START: U_STM32F779.PH5
- removed net ADC3_DRDY: U_STM32F779.PF12
- removed net ADC3_RES: U_STM32F779.PF15
- removed net ADC3_START: U_STM32F779.PF14
- removed net ADC4_DRDY: U_STM32F779.PH0
- removed net ADC4_RES: U_STM32F779.PF10
- removed net ADC4_START: U_STM32F779.PF9
- removed net ADC5_DRDY: U_STM32F779.PA1
- removed net ADC5_RES: U_STM32F779.PC2
- removed net ADC5_START: U_STM32F779.PC0
- removed net ADC6_DRDY: U_STM32F779.PA2
- removed net ADC6_RES: U_STM32F779.PH1
- removed net ADC6_START: U_STM32F779.PC3
- removed net OUT_PT_1: U_STM32F779.PB1
- removed net OUT_PT_2: U_STM32F779.PA4
- removed net OUT_PT_3: U_STM32F779.PB0
- removed net SPI3_CS: U_STM32F779.PJ1
- removed net SPI3_CS2: U_STM32F779.PF2
- removed net SPI3_MISO: U_STM32F779.PC11
- removed net SPI3_MOSI: U_STM32F779.PB2
- removed net SPI3_SCK: U_STM32F779.PC10
- removed net SPI4_CS: U_STM32F779.PH4
- removed net SPI4_CS2: U_STM32F779.PI12
- removed net SPI4_MISO: U_STM32F779.PE5
- removed net SPI4_MOSI: U_STM32F779.PE6
- removed net SPI4_SCK: U_STM32F779.PE2
- removed net SPI5_CS: U_STM32F779.PF13
- removed net SPI5_CS2: U_STM32F779.PI13
- removed net SPI5_MISO: U_STM32F779.PF8
- removed net SPI5_MOSI: U_STM32F779.PF11
- removed net SPI5_SCK: U_STM32F779.PF7

Commit message: Pins matched to Cube
next step, autoroute (if possible)
Connections:
- removed net DMS_DIN: RN_DMS1B.2, RN_DMS2B.2, RN_DMS3B.2, RN_DMS4B.2, RN_DMS5B.2, RN_DMS6B.2
- removed net DMS_DOUT: RN_DMS1C.2, RN_DMS2C.2, RN_DMS3C.2, RN_DMS4C.2, RN_DMS5C.2, RN_DMS6C.2
- removed net DMS_SCLK: RN_DMS1A.2, RN_DMS2A.2, RN_DMS3A.2, RN_DMS4A.2, RN_DMS5A.2, RN_DMS6A.2
- removed net N$148: X_DMS.B10
- removed net N$157: X_DMS.A10
- removed net N$17: X_PT.A6
- removed net N$18: X_PT.A5
- removed net N$19: X_PT.A4
- removed net PT_DIN: RN_A_PT1C.2, RN_A_PT2C.2, RN_A_PT3C.2
- removed net PT_DOUT: RN_A_PT1D.2, RN_A_PT2D.2, RN_A_PT3D.2
- removed net PT_SCLK: RN_A_PT1B.2, RN_A_PT2B.2, RN_A_PT3B.2
- new net SPI3_MISO: RN_A_PT1D.2, RN_A_PT2D.2, RN_A_PT3D.2, U_STM32F779.PC11
- new net SPI3_MOSI: RN_A_PT1C.2, RN_A_PT2C.2, RN_A_PT3C.2, U_STM32F779.PB2
- new net SPI3_SCK: RN_A_PT1B.2, RN_A_PT2B.2, RN_A_PT3B.2, U_STM32F779.PC10
- new net SPI4_MISO: RN_DMS1C.2, RN_DMS2C.2, RN_DMS3C.2, RN_DMS4C.2, RN_DMS5C.2, RN_DMS6C.2, U_STM32F779.PE5
- new net SPI4_MOSI: RN_DMS1B.2, RN_DMS2B.2, RN_DMS3B.2, RN_DMS4B.2, RN_DMS5B.2, RN_DMS6B.2, U_STM32F779.PE6
- new net SPI4_SCK: RN_DMS1A.2, RN_DMS2A.2, RN_DMS3A.2, RN_DMS4A.2, RN_DMS5A.2, RN_DMS6A.2, U_STM32F779.PE2
- net !CS!_DMS1: now also U_STM32F779.PF13
- net !CS!_DMS2: now also U_STM32F779.PF14
- net !CS!_DMS3: now also U_STM32F779.PF15
- net !CS!_DMS4: now also U_STM32F779.PG0
- net !CS!_DMS5: now also U_STM32F779.PG1
- net !CS!_DMS6: now also U_STM32F779.PE7
- net !CS!_PT1: now also U_STM32F779.PD15
- net !CS!_PT2: now also U_STM32F779.PD14
- net !CS!_PT3: now also U_STM32F779.PD8
- net !DRDY!_DMS1: now also U_STM32F779.PG4
- net !DRDY!_DMS2: now also U_STM32F779.PA8
- net !DRDY!_DMS3: now also U_STM32F779.PA9
- net !DRDY!_DMS4: now also U_STM32F779.PA10
- net !DRDY!_DMS5: now also U_STM32F779.PA11
- net !DRDY!_DMS6: now also U_STM32F779.PA12
- net !DRDY!_PT1: now also U_STM32F779.PJ15
- net !DRDY!_PT2: now also U_STM32F779.PJ14
- net !DRDY!_PT3: now also U_STM32F779.PJ13
- net FL_2_WP: now also U_STM32F779.PD13; no longer U_STM32F779.PD8
- net GND: now also X_DMS.A10, X_DMS.B10, X_PT.A4, X_PT.A5, X_PT.A6

Commit message: finalized silkscreen
Parts:
- renumbered U_S70FL01GS_1 to U_FLASH1, U_S70FL01GS_2 to U_FLASH2
Changed lines of the file:
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@@
 <part name="C18" library="aSparkFun" deviceset="CAP" device="0603-CAP" value="100n"/>
 <part name="JP1" library="SparkFun-Jumpers" deviceset="JUMPER-SMT_2_NC_PASTE" device="_SILK"/>
-<part name="U_S70FL01GS_1" library="S70FL01GS" deviceset="S70FL01GS" device="" package3d_urn="urn:adsk.eagle:package:16378380/2"/>
-<part name="U_S70FL01GS_2" library="S70FL01GS" deviceset="S70FL01GS" device="" package3d_urn="urn:adsk.eagle:package:16378380/2"/>
+<part name="U_FLASH1" library="S70FL01GS" deviceset="S70FL01GS" device="" package3d_urn="urn:adsk.eagle:package:16378380/2"/>
+<part name="U_FLASH2" library="S70FL01GS" deviceset="S70FL01GS" device="" package3d_urn="urn:adsk.eagle:package:16378380/2"/>
 <part name="C28" library="rcl" library_urn="urn:adsk.eagle:library:334" deviceset="C-EU" device="C0805" package3d_urn="urn:adsk.eagle:package:23617/2" value="100n"/>
 <part name="C29" library="rcl" library_urn="urn:adsk.eagle:library:334" deviceset="C-EU" device="C0805" package3d_urn="urn:adsk.eagle:package:23617/2" value="100n"/>
@@
 <attribute name="VALUE" x="50.8" y="139.7" size="1.4224" layer="96" font="vector"/>
 </instance>
-<instance part="U_S70FL01GS_1" gate="G$1" x="231.14" y="71.12" smashed="yes"/>
-<instance part="U_S70FL01GS_2" gate="G$1" x="302.26" y="71.12" smashed="yes"/>
+<instance part="U_FLASH1" gate="G$1" x="231.14" y="71.12" smashed="yes"/>
+<instance part="U_FLASH2" gate="G$1" x="302.26" y="71.12" smashed="yes"/>
 <instance part="C28" gate="G$1" x="299.466" y="261.112" smashed="yes" rot="R90">
 <attribute name="NAME" x="299.085" y="262.636" size="1.778" layer="95" rot="R90"/>
@@
 </segment>
 <segment>
-<pinref part="U_S70FL01GS_1" gate="G$1" pin="VSS"/>
+<pinref part="U_FLASH1" gate="G$1" pin="VSS"/>
 <wire x1="264.16" y1="71.12" x2="264.16" y2="76.2" width="0.1524" layer="91"/>
 <label x="264.16" y="76.2" size="1.27" layer="95" rot="R90" xref="yes"/>
 </segment>
 <segment>
-<pinref part="U_S70FL01GS_2" gate="G$1" pin="VSS"/>
+<pinref part="U_FLASH2" gate="G$1" pin="VSS"/>
 <wire x1="335.28" y1="71.12" x2="335.28" y2="76.2" width="0.1524" layer="91"/>
 <label x="335.28" y="76.2" size="1.27" layer="95" rot="R90" xref="yes"/>
@@
 </segment>
 <segment>
-<pinref part="U_S70FL01GS_1" gate="G$1" pin="VCC"/>
+<pinref part="U_FLASH1" gate="G$1" pin="VCC"/>
 <wire x1="223.52" y1="96.52" x2="220.98" y2="96.52" width="0.1524" layer="91"/>
 <label x="220.98" y="96.52" size="1.27" layer="95" rot="R270" xref="yes"/>
 </segment>
 <segment>
-<pinref part="U_S70FL01GS_2" gate="G$1" pin="VCC"/>
+<pinref part="U_FLASH2" gate="G$1" pin="VCC"/>
 <wire x1="294.64" y1="96.52" x2="292.1" y2="96.52" width="0.1524" layer="91"/>
 <label x="292.1" y="96.52" size="1.27" layer="95" rot="R270" xref="yes"/>
@@
 <net name="FL_1_HLD" class="0">
 <segment>
-<pinref part="U_S70FL01GS_1" gate="G$1" pin="HOLD"/>
+<pinref part="U_FLASH1" gate="G$1" pin="HOLD"/>
 <wire x1="223.52" y1="101.6" x2="220.98" y2="101.6" width="0.1524" layer="91"/>
 <wire x1="220.98" y1="101.6" x2="220.98" y2="114.3" width="0.1524" layer="91"/>
@@
 <net name="FL_1_RES" class="0">
 <segment>
-<pinref part="U_S70FL01GS_1" gate="G$1" pin="RESET"/>
+<pinref part="U_FLASH1" gate="G$1" pin="RESET"/>
 <wire x1="223.52" y1="91.44" x2="218.44" y2="91.44" width="0.1524" layer="91"/>
 <wire x1="218.44" y1="91.44" x2="218.44" y2="114.3" width="0.1524" layer="91"/>
@@
 <net name="FL_1_CS2" class="0">
 <segment>
-<pinref part="U_S70FL01GS_1" gate="G$1" pin="CS2"/>
+<pinref part="U_FLASH1" gate="G$1" pin="CS2"/>
 <wire x1="223.52" y1="76.2" x2="215.9" y2="76.2" width="0.1524" layer="91"/>
 <wire x1="215.9" y1="76.2" x2="215.9" y2="114.3" width="0.1524" layer="91"/>
@@
 <net name="FL_1_CS1" class="0">
 <segment>
-<pinref part="U_S70FL01GS_1" gate="G$1" pin="CS1"/>
+<pinref part="U_FLASH1" gate="G$1" pin="CS1"/>
 <wire x1="223.52" y1="71.12" x2="213.36" y2="71.12" width="0.1524" layer="91"/>
 <wire x1="213.36" y1="71.12" x2="213.36" y2="114.3" width="0.1524" layer="91"/>
@@
 <net name="SPI6_MISO" class="0">
 <segment>
-<pinref part="U_S70FL01GS_1" gate="G$1" pin="SO"/>
+<pinref part="U_FLASH1" gate="G$1" pin="SO"/>
 <wire x1="223.52" y1="66.04" x2="210.82" y2="66.04" width="0.1524" layer="91"/>
 <wire x1="210.82" y1="66.04" x2="210.82" y2="114.3" width="0.1524" layer="91"/>
@@
 <net name="SPI6_SCK" class="0">
 <segment>
-<pinref part="U_S70FL01GS_1" gate="G$1" pin="SCK"/>
+<pinref part="U_FLASH1" gate="G$1" pin="SCK"/>
 <wire x1="264.16" y1="101.6" x2="264.16" y2="106.68" width="0.1524" layer="91"/>
 <wire x1="264.16" y1="106.68" x2="223.52" y2="106.68" width="0.1524" layer="91"/>
@@
 <wire x1="226.06" y1="109.22" x2="266.7" y2="109.22" width="0.1524" layer="91"/>
 <wire x1="266.7" y1="109.22" x2="266.7" y2="96.52" width="0.1524" layer="91"/>
-<pinref part="U_S70FL01GS_1" gate="G$1" pin="SI"/>
+<pinref part="U_FLASH1" gate="G$1" pin="SI"/>
 <wire x1="266.7" y1="96.52" x2="264.16" y2="96.52" width="0.1524" layer="91"/>
 <wire x1="226.06" y1="109.22" x2="226.06" y2="114.3" width="0.1524" layer="91"/>
@@
 <net name="FL_1_WP" class="0">
 <segment>
-<pinref part="U_S70FL01GS_1" gate="G$1" pin="WP"/>
+<pinref part="U_FLASH1" gate="G$1" pin="WP"/>
 <wire x1="264.16" y1="66.04" x2="269.24" y2="66.04" width="0.1524" layer="91"/>
 <wire x1="269.24" y1="66.04" x2="269.24" y2="111.76" width="0.1524" layer="91"/>
@@
 <net name="SPI2_MISO" class="0">
 <segment>
-<pinref part="U_S70FL01GS_2" gate="G$1" pin="SO"/>
+<pinref part="U_FLASH2" gate="G$1" pin="SO"/>
 <wire x1="294.64" y1="66.04" x2="281.94" y2="66.04" width="0.1524" layer="91"/>
 <wire x1="281.94" y1="66.04" x2="281.94" y2="114.3" width="0.1524" layer="91"/>
@@
 <net name="FL_2_CS1" class="0">
 <segment>
-<pinref part="U_S70FL01GS_2" gate="G$1" pin="CS1"/>
+<pinref part="U_FLASH2" gate="G$1" pin="CS1"/>
 <wire x1="294.64" y1="71.12" x2="284.48" y2="71.12" width="0.1524" layer="91"/>
 <wire x1="284.48" y1="71.12" x2="284.48" y2="114.3" width="0.1524" layer="91"/>
@@
 <net name="FL_2_CS2" class="0">
 <segment>
-<pinref part="U_S70FL01GS_2" gate="G$1" pin="CS2"/>
+<pinref part="U_FLASH2" gate="G$1" pin="CS2"/>
 <wire x1="294.64" y1="76.2" x2="287.02" y2="76.2" width="0.1524" layer="91"/>
 <wire x1="287.02" y1="76.2" x2="287.02" y2="114.3" width="0.1524" layer="91"/>
@@
 <net name="FL_2_RES" class="0">
 <segment>
-<pinref part="U_S70FL01GS_2" gate="G$1" pin="RESET"/>
+<pinref part="U_FLASH2" gate="G$1" pin="RESET"/>
 <wire x1="294.64" y1="91.44" x2="289.56" y2="91.44" width="0.1524" layer="91"/>
 <wire x1="289.56" y1="91.44" x2="289.56" y2="114.3" width="0.1524" layer="91"/>
@@
 <net name="FL_2_HLD" class="0">
 <segment>
-<pinref part="U_S70FL01GS_2" gate="G$1" pin="HOLD"/>
+<pinref part="U_FLASH2" gate="G$1" pin="HOLD"/>
 <wire x1="294.64" y1="101.6" x2="292.1" y2="101.6" width="0.1524" layer="91"/>
 <wire x1="292.1" y1="101.6" x2="292.1" y2="114.3" width="0.1524" layer="91"/>
@@
 <net name="SPI2_SCK" class="0">
 <segment>
-<pinref part="U_S70FL01GS_2" gate="G$1" pin="SCK"/>
+<pinref part="U_FLASH2" gate="G$1" pin="SCK"/>
 <wire x1="335.28" y1="101.6" x2="335.28" y2="106.68" width="0.1524" layer="91"/>
 <wire x1="335.28" y1="106.68" x2="294.64" y2="106.68" width="0.1524" layer="91"/>
@@
 <wire x1="297.18" y1="109.22" x2="337.82" y2="109.22" width="0.1524" layer="91"/>
 <wire x1="337.82" y1="109.22" x2="337.82" y2="96.52" width="0.1524" layer="91"/>
-<pinref part="U_S70FL01GS_2" gate="G$1" pin="SI"/>
+<pinref part="U_FLASH2" gate="G$1" pin="SI"/>
 <wire x1="337.82" y1="96.52" x2="335.28" y2="96.52" width="0.1524" layer="91"/>
 <wire x1="297.18" y1="109.22" x2="297.18" y2="114.3" width="0.1524" layer="91"/>
@@
 <net name="FL_2_WP" class="0">
 <segment>
-<pinref part="U_S70FL01GS_2" gate="G$1" pin="WP"/>
+<pinref part="U_FLASH2" gate="G$1" pin="WP"/>
 <wire x1="335.28" y1="66.04" x2="340.36" y2="66.04" width="0.1524" layer="91"/>
 <wire x1="340.36" y1="66.04" x2="340.36" y2="111.76" width="0.1524" layer="91"/>
