File: SPU.sch (EAGLE design)
At the start: 88 parts, among them Q1 12MHz

Commit message: Adds smf2 lib
Parts:
- added R1: 10k, rcl:R-EU_R0805
- added SF2_M2S010TQ1: SF2_M2S010TQ144, smf2:SF2_M2S010TQ144
Connections:
- new net 3.3V: R1.1, SF2_M2S010TQ1G$7.VDD, SF2_M2S010TQ1G$7.VDDI0, SF2_M2S010TQ1G$7.VDDI2, SF2_M2S010TQ1G$7.VDDI3, SF2_M2S010TQ1G$7.VDDI4, SF2_M2S010TQ1G$7.VDDI6, SF2_M2S010TQ1G$7.VDDI7, SF2_M2S010TQ1G$7.VPP, SF2_M2S010TQ1G$7.VPPNVM
- new net N$2: R1.2, SF2_M2S010TQ1G$7.DEVRST_N
- net GND: now also SF2_M2S010TQ1G$7.VSS, SF2_M2S010TQ1G$7.VSSNVM
Changed lines of the file:
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@@
 <part name="FRAME2" library="frames" library_urn="urn:adsk.eagle:library:229" deviceset="A3L-LOC" device=""/>
 <part name="FRAME3" library="frames" library_urn="urn:adsk.eagle:library:229" deviceset="A3L-LOC" device=""/>
+<part name="SF2_M2S010TQ1" library="smf2" deviceset="SF2_M2S010TQ144" device=""/>
+<part name="R1" library="rcl" library_urn="urn:adsk.eagle:library:334" deviceset="R-EU_" device="R0805" package3d_urn="urn:adsk.eagle:package:23553/2" value="10k"/>
 </parts>
 <sheets>
@@
 <attribute name="SHEET" x="357.505" y="5.08" size="2.54" layer="94"/>
 </instance>
+<instance part="SF2_M2S010TQ1" gate="G$1" x="33.02" y="208.28" smashed="yes">
+<attribute name="NAME" x="33.02" y="244.348" size="1.27" layer="95"/>
+</instance>
+<instance part="SF2_M2S010TQ1" gate="G$2" x="30.48" y="175.26" smashed="yes">
+<attribute name="NAME" x="30.48" y="201.168" size="1.27" layer="95"/>
+</instance>
+<instance part="SF2_M2S010TQ1" gate="G$3" x="30.48" y="147.32" smashed="yes">
+<attribute name="NAME" x="30.48" y="168.148" size="1.27" layer="95"/>
+</instance>
+<instance part="SF2_M2S010TQ1" gate="G$4" x="27.94" y="106.68" smashed="yes">
+<attribute name="NAME" x="27.94" y="135.128" size="1.27" layer="95"/>
+</instance>
+<instance part="SF2_M2S010TQ1" gate="G$5" x="25.4" y="71.12" smashed="yes">
+<attribute name="NAME" x="25.4" y="91.948" size="1.27" layer="95"/>
+</instance>
+<instance part="SF2_M2S010TQ1" gate="G$6" x="22.86" y="22.86" smashed="yes">
+<attribute name="NAME" x="22.86" y="48.768" size="1.27" layer="95"/>
+</instance>
+<instance part="SF2_M2S010TQ1" gate="G$7" x="175.26" y="205.74" smashed="yes">
+<attribute name="NAME" x="175.26" y="244.348" size="1.27" layer="95"/>
+</instance>
+<instance part="R1" gate="G$1" x="167.64" y="236.22" smashed="yes" rot="R270">
+<attribute name="NAME" x="169.1386" y="240.03" size="1.778" layer="95" rot="R270"/>
+<attribute name="VALUE" x="164.338" y="240.03" size="1.778" layer="96" rot="R270"/>
+</instance>
 </instances>
 <busses>
 </busses>
 <nets>
+<net name="3.3V" class="0">
+<segment>
+<pinref part="SF2_M2S010TQ1" gate="G$7" pin="VDD"/>
+<wire x1="170.18" y1="228.6" x2="162.56" y2="228.6" width="0.1524" layer="91"/>
+<label x="160.02" y="228.6" size="1.27" layer="95" rot="R180" xref="yes"/>
+<pinref part="R1" gate="G$1" pin="1"/>
+<wire x1="162.56" y1="228.6" x2="160.02" y2="228.6" width="0.1524" layer="91"/>
+<wire x1="167.64" y1="241.3" x2="162.56" y2="241.3" width="0.1524" layer="91"/>
+<wire x1="162.56" y1="241.3" x2="162.56" y2="228.6" width="0.1524" layer="91"/>
+<junction x="162.56" y="228.6"/>
+</segment>
+<segment>
+<pinref part="SF2_M2S010TQ1" gate="G$7" pin="VDDI0"/>
+<wire x1="170.18" y1="220.98" x2="165.1" y2="220.98" width="0.1524" layer="91"/>
+<pinref part="SF2_M2S010TQ1" gate="G$7" pin="VDDI7"/>
+<wire x1="165.1" y1="220.98" x2="160.02" y2="220.98" width="0.1524" layer="91"/>
+<wire x1="170.18" y1="208.28" x2="165.1" y2="208.28" width="0.1524" layer="91"/>
+<wire x1="165.1" y1="208.28" x2="165.1" y2="210.82" width="0.1524" layer="91"/>
+<junction x="165.1" y="220.98"/>
+<pinref part="SF2_M2S010TQ1" gate="G$7" pin="VDDI2"/>
+<wire x1="165.1" y1="210.82" x2="165.1" y2="213.36" width="0.1524" layer="91"/>
+<wire x1="165.1" y1="213.36" x2="165.1" y2="215.9" width="0.1524" layer="91"/>
+<wire x1="165.1" y1="215.9" x2="165.1" y2="218.44" width="0.1524" layer="91"/>
+<wire x1="165.1" y1="218.44" x2="165.1" y2="220.98" width="0.1524" layer="91"/>
+<wire x1="170.18" y1="218.44" x2="165.1" y2="218.44" width="0.1524" layer="91"/>
+<junction x="165.1" y="218.44"/>
+<pinref part="SF2_M2S010TQ1" gate="G$7" pin="VDDI3"/>
+<wire x1="170.18" y1="215.9" x2="165.1" y2="215.9" width="0.1524" layer="91"/>
+<junction x="165.1" y="215.9"/>
+<pinref part="SF2_M2S010TQ1" gate="G$7" pin="VDDI4"/>
+<wire x1="170.18" y1="213.36" x2="165.1" y2="213.36" width="0.1524" layer="91"/>
+<junction x="165.1" y="213.36"/>
+<pinref part="SF2_M2S010TQ1" gate="G$7" pin="VDDI6"/>
+<wire x1="170.18" y1="210.82" x2="165.1" y2="210.82" width="0.1524" layer="91"/>
+<junction x="165.1" y="210.82"/>
+<label x="160.02" y="220.98" size="1.27" layer="95" rot="R180" xref="yes"/>
+</segment>
+<segment>
+<pinref part="SF2_M2S010TQ1" gate="G$7" pin="VPPNVM"/>
+<wire x1="215.9" y1="236.22" x2="220.98" y2="236.22" width="0.1524" layer="91"/>
+<pinref part="SF2_M2S010TQ1" gate="G$7" pin="VPP"/>
+<wire x1="215.9" y1="238.76" x2="220.98" y2="238.76" width="0.1524" layer="91"/>
+<wire x1="220.98" y1="238.76" x2="223.52" y2="238.76" width="0.1524" layer="91"/>
+<wire x1="220.98" y1="236.22" x2="220.98" y2="238.76" width="0.1524" layer="91"/>
+<junction x="220.98" y="238.76"/>
+<label x="223.52" y="238.76" size="1.27" layer="95" xref="yes"/>
+</segment>
+</net>
+<net name="GND" class="0">
+<segment>
+<pinref part="SF2_M2S010TQ1" gate="G$7" pin="VSS"/>
+<wire x1="170.18" y1="226.06" x2="160.02" y2="226.06" width="0.1524" layer="91"/>
+<label x="160.02" y="226.06" size="1.27" layer="95" rot="R180" xref="yes"/>
+</segment>
+<segment>
+<pinref part="SF2_M2S010TQ1" gate="G$7" pin="VSSNVM"/>
+<wire x1="215.9" y1="233.68" x2="223.52" y2="233.68" width="0.1524" layer="91"/>
+<label x="223.52" y="233.68" size="1.27" layer="95" xref="yes"/>
+</segment>
+</net>
+<net name="N$2" class="0">
+<segment>
+<pinref part="SF2_M2S010TQ1" gate="G$7" pin="DEVRST_N"/>
+<pinref part="R1" gate="G$1" pin="2"/>
+<wire x1="170.18" y1="231.14" x2="167.64" y2="231.14" width="0.1524" layer="91"/>
+</segment>
+</net>
 </nets>
 </sheet>

Commit message: Adds STAMPs
Parts:
- removed C28, C29, C30, C31, C32, C33, C75: 100n, rcl:C-EUC0805
- removed C52, C74: 10n, rcl:C-EUC0805
- removed C68, C69, C70, C71, C72, C73: 10u, rcl:CPOL-EUE/7260-38W
- removed D10, D11, D12, D3, D4, D7, D8, D9: 3V6, diodes:DZMELF
- removed D2, D6: 5V6, diodes:DZMELF
- removed Q1: 12MHz, adafruit:CRYSTALSM49
- removed R24: ?, rcl:R-EU_R0805
- removed RN11: 3k, resistor-dil:4R-NEXBS8V
- removed RN12: 1k, resistor-dil:4R-NEXBS8V
- removed U_ADR366_3: ADR366WAUJZ, ADR360:ADR36_UJZ
- removed U_CH340G: CH340G, ch340g:CH340G
- removed U_FLASH1: S70FL01GS, S70FL01GS:S70FL01GS
- removed U_OPTO_1, U_OPTO_2: MOCD207MSOIC-8, Opto-Electronic:MOCD207MSOIC-8
- added C10, C11, C12, C13, C14, C15, C16, C17, C18, C19, C20, C21, C22, C23, C24, C25, C26, C27, C7, C8, C9: 100n, rcl:C-EUC0805
- added C3, C5: 4.7u, rcl:C-EUC0805
- added C4, C6: 470n, rcl:C-EUC0805
- added PROBES: (no value), selfmade:PSS254_G3
- added Q2: CSTCR6M00G53Z, murata-filter:CSTCR6M00G53Z
- added R2, R3: 2, rcl:R-EU_R0805
- added R26, R27, R4: 10k, rcl:R-EU_R0805
- added R34, R35, R36, R37, R38, R39, R40, R41, R42, R43, R44, R45, R46, R47, R48, R49, R50, R51, R52, R53, R54, R55, R56, R57, R58, R59, R60, R61, R62, R63, R67: 47, rcl:R-EU_R0805
- added R5: 4k7, rcl:R-EU_R0805
- added R6, R8: 27, rcl:R-EU_R0805
- added R7: 1k5, rcl:R-EU_R0805
- added R9: 470, rcl:R-EU_R0805
- added U$1: FT2232D, smf2:FT2232D
- added U$2: USB_B_STANDING, selfmade:USB_B_STANDING
- added U$3: M93C46-WDW6TP, smf2:M93C46-WDW6TP
- added U$4: S70FL01GSAGM, smf2:S70FL01GSAGM
- added U$5: DSC1001CI1-004.0960T, selfmade:DSC1001CI1-004.0960T
- added U_OPTO_4, U_OPTO_5: MOCD207M, Opto-Electronic:MOCD207M_SOIC8
- added WP: (no value), selfmade:PSS254_G2
- C1: value 22p -> 100n; device rcl:C-EUC0603 -> rcl:C-EUC0805
- C2: value 22p -> 10n; device rcl:C-EUC0603 -> rcl:C-EUC0805
- R12: value 2k -> 3k
- R13: value 4k7 -> 3k
- R14: value 7k5 -> 47
- R22: value 100k -> 2k
- R23: value 1k -> 3k
- R25: value ? -> 7k5
- U_OPTO_3: value MOCD207MSOIC-8 -> MOCD207M; device Opto-Electronic:MOCD207MSOIC-8 -> Opto-Electronic:MOCD207M_SOIC8
Connections:
- removed net 3.3V: R1.1, SF2_M2S010TQ1G$7.VDD, SF2_M2S010TQ1G$7.VDDI0, SF2_M2S010TQ1G$7.VDDI2, SF2_M2S010TQ1G$7.VDDI3, SF2_M2S010TQ1G$7.VDDI4, SF2_M2S010TQ1G$7.VDDI6, SF2_M2S010TQ1G$7.VDDI7, SF2_M2S010TQ1G$7.VPP, SF2_M2S010TQ1G$7.VPPNVM
- removed net 3V3REF: C74.2, C75.2, R24.2, U_ADR366_3.VOUT
- removed net DAPI_N: D1.C, U_CH340G.D-
- removed net DAPI_P: D2.C, U_CH340G.D+
- removed net DAPI_RX: D4.C, U_CH340G.TX
- removed net DAPI_TX: D3.C, U_CH340G.RX
- removed net EXP_IN_OPT: D10.C, R13.1, U_OPTO_3.COL1
- removed net EXP_OUT_OPT: U_OPTO_3.A2
- removed net FL_1_CS1: U_FLASH1.CS1
- removed net FL_1_CS2: U_FLASH1.CS2
- removed net FL_1_HLD: U_FLASH1.HOLD
- removed net FL_1_RES: U_FLASH1.RESET
- removed net FL_1_WP: U_FLASH1.WP
- removed net INTERSPU_RX: D11.C
- removed net INTERSPU_TX: D12.C
- removed net LO_OPT: D7.C, RN12C.2, U_OPTO_2.COL1
- removed net N$1 (its old number): C2.1, Q1.2, U_CH340G.XO
- removed net N$42: RN11C.2, U_OPTO_1.A1
- removed net N$43: RN11D.2, U_OPTO_1.A2
- removed net SODS_OPT: D8.C, RN12A.2, U_OPTO_1.COL1
- removed net SOE_OPT: D9.C, RN12B.2, U_OPTO_1.COL2
- removed net SPI6_MISO: U_FLASH1.SO
- removed net SPI6_MOSI: U_FLASH1.SI
- removed net SPI6_SCK: U_FLASH1.SCK
- new net ADC_START: R34.2
- new net DAPI_CTS: SF2_M2S010TQ1G$1.DDRIO30NB0, U$1.BDBUS2
- new net DAPI_DSR: SF2_M2S010TQ1G$1.DDRIO35PB0, U$1.BDBUS4
- new net DAPI_DTR: SF2_M2S010TQ1G$1.DDRIO37NB0, U$1.BDBUS5
- new net DAPI_RTS: SF2_M2S010TQ1G$1.DDRIO35NB0, U$1.BDBUS3
- new net DAPI_RXD: SF2_M2S010TQ1G$1.DDRIO29PB0, U$1.BDBUS0
- new net DAPI_TXD: SF2_M2S010TQ1G$1.DDRIO30PB0, U$1.BDBUS1
- new net EECLK: U$1.EESK, U$3.CLK
- new net EECS: U$1.EECS, U$3.CS
- new net EED: R27.2, U$1.EEDATA, U$3.DIN
- new net F_CLK: SF2_M2S010TQ1G$2.MSIO12PB2/SPI_0_CLK, U$4.SCLK
- new net F_CS1: SF2_M2S010TQ1G$2.MSIO13NB2/SPI_0_SS0/GPIO_7_A, U$4.CS1#
- new net F_CS2: SF2_M2S010TQ1G$2.MSIO6PB2/USB_DATA6_B, U$4.CS2#
- new net F_MISO: SF2_M2S010TQ1G$2.MSIO12NB2/SPI_0_SDI/GPIO_5_A, U$4.SO/O1
- new net F_MOSI: SF2_M2S010TQ1G$2.MSIO13PB2/SPI_0_SDO/GPIO_6_A, U$4.SI/O0
- new net N$10: R26.2, SF2_M2S010TQ1G$3.JTAGSEL
- new net N$11: R8.1, U$1.USBDM
- new net N$12: Q2.1, U$1.XTIN
- new net N$13: C21.2, U$1.3V3OUT
- new net N$14: C22.2, R9.2, U$1.AVCC
- new net N$15: R4.2, R5.1, U$1.RESET#
- new net N$16: R5.2, U$2.V+
- new net N$18: SF2_M2S010TQ1G$3.JTAG_TCK/M3_TCK, U$1.ADBUS0
- new net N$19: SF2_M2S010TQ1G$3.JTAG_TDI/M3_TDI, U$1.ADBUS1
- new net N$20: SF2_M2S010TQ1G$3.JTAG_TDO/M3_TDO/M3_SWO, U$1.ADBUS2
- new net N$21: SF2_M2S010TQ1G$3.JTAG_TMS/M3_TMS/M3_SWDIO, U$1.ADBUS3
- new net N$22: Q2.3, U$1.XTOUT
- new net N$23: R27.1, U$3.DOUT
- new net N$24: R13.2, U_OPTO_3.A1
- new net N$25: R12.2, U_OPTO_5.A2
- new net N$26: R11.2, U_OPTO_5.A1
- new net N$27: R22.1, U_OPTO_4.C1
- new net N$28: U$4.WP#/IO2, WP.2
- new net N$29: R14.1, U$5.OUT
- new net N$4: C3.1, C4.1, SF2_M2S010TQ1G$7.CCC_NE1_PLL_VSSA
- new net N$5: C3.2, C4.2, R2.2, SF2_M2S010TQ1G$7.CCC_NE1_PLL_VDDA
- new net N$50: R45.2, SF2_M2S010TQ1G$2.MSIO4NB2/USB_DATA3_B
- new net N$53: R37.2, SF2_M2S010TQ1G$1.DDRIO55PB0/CCC_NE0_CLKI3
- new net N$54: R38.2, SF2_M2S010TQ1G$1.DDRIO59NB0/GB4
- new net N$57: R39.2, SF2_M2S010TQ1G$1.DDRIO60NB0/CCC_NE1_CLKI3
- new net N$58: R42.1, SF2_M2S010TQ1G$2.MSIO2NB2/USB_NXT_B
- new net N$59: R43.1, SF2_M2S010TQ1G$2.MSIO3PB2/USB_DATA0_B
- new net N$6: C5.2, C6.2, R3.2, SF2_M2S010TQ1G$7.CCC_NE0_PLL_VDDA
- new net N$60: R44.1, SF2_M2S010TQ1G$2.MSIO4PB2/USB_DATA2_B
- new net N$61: R47.1, SF2_M2S010TQ1G$4.MSIO104NB4/GB7
- new net N$62: R48.1, SF2_M2S010TQ1G$4.MSIO104PB4/GB3
- new net N$63: R49.1, SF2_M2S010TQ1G$4.MSIO105PB4/CCC_NE0_CLKI0
- new net N$64: R50.1, SF2_M2S010TQ1G$4.MSIO105NB4
- new net N$65: R51.1, SF2_M2S010TQ1G$4.MSIO106PB4
- new net N$66: R54.2, SF2_M2S010TQ1G$4.MSIO109NB4
- new net N$67: R53.2, SF2_M2S010TQ1G$4.MSIO109PB4
- new net N$7: C5.1, C6.1, SF2_M2S010TQ1G$7.CCC_NE0_PLL_VSSA
- new net N$71: R57.1, SF2_M2S010TQ1G$5.MSIOD93NB6
- new net N$72: R58.1, SF2_M2S010TQ1G$5.MSIOD93PB6
- new net N$73: R59.2, SF2_M2S010TQ1G$5.MSIOD96PB6
- new net N$74: R60.2, SF2_M2S010TQ1G$5.MSIOD96NB6
- new net N$75: R61.2, SF2_M2S010TQ1G$5.MSIOD98NB6
- new net N$76: R62.1, SF2_M2S010TQ1G$6.MSIO67NB7
- new net N$77: R63.1, SF2_M2S010TQ1G$6.MSIO67PB7
- new net N$78: R67.1, SF2_M2S010TQ1G$6.MSIO71NB7
- new net N$8: R7.1, U$1.RSTOUT#
- new net N$9: R6.1, R7.2, U$1.USBDP
- new net PROBE_A: PROBES.1, SF2_M2S010TQ1G$4.MSIO103PB4/PROBE_A
- new net PROBE_B: PROBES.3, SF2_M2S010TQ1G$4.MSIO103NB4/PROBE_B
- new net RXSM_LO: U_OPTO_5.C1
- new net RXSM_SODS: U_OPTO_5.C2
- new net RXSM_SOE: U_OPTO_3.C1
- new net SG_CLK: R14.2
- new net STAMP1_CS_SG1: R37.1
- new net STAMP1_CS_SG2: R38.1
- new net STAMP1_CS_TEMP: R39.1
- new net STAMP1_DRDY_SG1: SF2_M2S010TQ1G$1.DDRIO53NB0
- new net STAMP1_DRDY_SG2: SF2_M2S010TQ1G$1.DDRIO53PB0
- new net STAMP1_DRDY_TEMP: SF2_M2S010TQ1G$1.DDRIO55NB0
- new net STAMP1_MISO: SF2_M2S010TQ1G$1.DDRIO48PB0
- new net STAMP1_MOSI: R35.1
- new net STAMP1_SCLK: R36.1
- new net STAMP2_CS_SG1: R42.2
- new net STAMP2_CS_SG2: R43.2
- new net STAMP2_CS_TEMP: R44.2
- new net STAMP2_DRDY_SG1: SF2_M2S010TQ1G$2.MSIO1PB2/USB_XCLK_B
- new net STAMP2_DRDY_SG2: SF2_M2S010TQ1G$2.MSIO1NB2/USB_DIR_B
- new net STAMP2_DRDY_TEMP: SF2_M2S010TQ1G$2.MSIO2PB2/USB_STP_B
- new net STAMP2_MISO: SF2_M2S010TQ1G$2.MSIO0NB2/USB_DATA7_B
- new net STAMP2_MOSI: R41.1
- new net STAMP2_SCLK: R40.1
- new net STAMP3_CS_SG1: R47.2
- new net STAMP3_CS_SG2: R48.2
- new net STAMP3_CS_TEMP: R49.2
- new net STAMP3_DRDY_SG1: SF2_M2S010TQ1G$2.MSIO5NB2/USB_DATA5_B
- new net STAMP3_DRDY_SG2: SF2_M2S010TQ1G$4.MSIO102PB4
- new net STAMP3_DRDY_TEMP: SF2_M2S010TQ1G$4.MSIO102NB4/CCC_NE1_CLKI0
- new net STAMP3_MISO: SF2_M2S010TQ1G$2.MSIO5PB2/USB_DATA4_B
- new net STAMP3_MOSI: R45.1
- new net STAMP3_SCLK: R46.2
- new net STAMP4_CS_SG1: R54.1
- new net STAMP4_CS_SG2: R53.1
- new net STAMP4_CS_TEMP: R52.1
- new net STAMP4_DRDY_SG1: SF2_M2S010TQ1G$4.MSIO114PB4
- new net STAMP4_DRDY_SG2: SF2_M2S010TQ1G$4.MSIO113NB4
- new net STAMP4_DRDY_TEMP: SF2_M2S010TQ1G$4.MSIO113PB4
- new net STAMP4_MISO: SF2_M2S010TQ1G$4.MSIO114NB4
- new net STAMP4_MOSI: R51.2
- new net STAMP4_SCLK: R50.2
- new net STAMP5_CS_SG1: R57.2
- new net STAMP5_CS_SG2: R58.2
- new net STAMP5_CS_TEMP: R59.1
- new net STAMP5_DRDY_SG1: SF2_M2S010TQ1G$5.MSIOD85PB6/CCC_NE1_CLKI1
- new net STAMP5_DRDY_SG2: SF2_M2S010TQ1G$5.MSIOD90NB6
- new net STAMP5_DRDY_TEMP: SF2_M2S010TQ1G$5.MSIOD90PB6
- new net STAMP5_MISO: SF2_M2S010TQ1G$5.MSIOD84PB6/CCC_NE1_CLKI2
- new net STAMP5_MOSI: R55.1
- new net STAMP5_SCLK: R56.1
- new net STAMP6_CS_SG1: R62.2
- new net STAMP6_CS_SG2: R63.2
- new net STAMP6_CS_TEMP: R67.2
- new net STAMP6_DRDY_SG1: SF2_M2S010TQ1G$5.MSIOD99NB6
- new net STAMP6_DRDY_SG2: SF2_M2S010TQ1G$6.MSIO64NB7
- new net STAMP6_DRDY_TEMP: SF2_M2S010TQ1G$6.MSIO64PB7
- new net STAMP6_MISO: SF2_M2S010TQ1G$5.MSIOD99PB6
- new net STAMP6_MOSI: R61.1
- new net STAMP6_SCLK: R60.1
- new net TM_RX: SF2_M2S010TQ1G$1.DDRIO37PB0, U_OPTO_4.COL2
- new net TM_TX: SF2_M2S010TQ1G$1.DDRIO43NB0, U_OPTO_4.A1
- new net USB_N: R8.2, U$2.D-
- new net USB_P: R6.2, U$2.D+
- new net VCCINT: C10.1, C11.1, C12.1, C13.1, C14.1, C7.1, C8.1, C9.1, SF2_M2S010TQ1G$7.VDD
- net 28V: now also R11.1, R12.1, R13.1; no longer RN11A.1, RN11B.1, RN11C.1, RN11D.1
- net 28VGND: now also D1.A, R23.2, U_OPTO_4.EMT1; no longer D6.A, R11.1, U_OPTO_3.EMT2
- net 3V3: now also C1.1, C15.1, C16.1, C17.1, C18.1, C19.1, C2.1, C20.1, C23.1, C24.2, C25.2, C26.2, C27.2, R1.1, R2.1, R26.1, R3.1, R9.1, SF2_M2S010TQ1G$3.JTAG_TRSTB/M3_TRSTB, SF2_M2S010TQ1G$7.VDDI0, SF2_M2S010TQ1G$7.VDDI2, SF2_M2S010TQ1G$7.VDDI3, SF2_M2S010TQ1G$7.VDDI4, SF2_M2S010TQ1G$7.VDDI6, SF2_M2S010TQ1G$7.VDDI7, SF2_M2S010TQ1G$7.VPP, SF2_M2S010TQ1G$7.VPPNVM, U$1.VCC, U$1.VCC1, U$1.VCCIOB, U$1.VVCIOA, U$3.ORG, U$3.VCC, U$4.VCC, U$5.VDD; no longer C28.1, C29.1, C30.1, C31.1, C32.1, C33.1, C68.+, C69.+, C70.+, C71.+, C72.+, C73.+, R13.2, RN12A.1, RN12B.1, RN12C.1, RN12D.1, U_CH340G.V3, U_CH340G.VCC, U_FLASH1.VCC
- net 5V: no longer C52.2, U_ADR366_3.VIN
- net 5V-28V: now also R25.2; no longer R14.2
- net EXP_IN: now also U_OPTO_4.A2; no longer U_OPTO_3.A1
- net EXP_OUT: now also D1.C, R25.1, U_OPTO_4.COL1; no longer D6.C, R14.1, U_OPTO_3.COL2
- net GND: now also C10.2, C11.2, C12.2, C13.2, C14.2, C15.2, C16.2, C17.2, C18.2, C19.2, C20.2, C21.1, C22.1, C23.2, C24.1, C25.1, C26.1, C27.1, C7.2, C8.2, C9.2, PROBES.2, Q2.2, R22.2, R4.1, U$1.AGND, U$1.GND1, U$1.GND2, U$1.GND3, U$1.GND4, U$1.TEST, U$2.S, U$2.V-, U$3.VSS, U$4.VSS, U$5.GND, U_OPTO_3.A2, U_OPTO_3.C2, U_OPTO_3.COL2, U_OPTO_3.EMT2, U_OPTO_4.EMT2, U_OPTO_5.EMT1, U_OPTO_5.EMT2, WP.1; no longer C28.2, C29.2, C30.2, C31.2, C32.2, C33.2, C52.1, C68.-, C69.-, C70.-, C71.-, C72.-, C73.-, C74.1, C75.1, D1.A, D10.A, D11.A, D12.A, D2.A, D3.A, D4.A, D7.A, D8.A, D9.A, R12.1, R23.1, U_ADR366_3.GND, U_CH340G.GND, U_FLASH1.VSS, U_OPTO_1.EMT1, U_OPTO_1.EMT2, U_OPTO_2.EMT1, U_OPTO_2.EMT2
- net LO: now also SF2_M2S010TQ1G$1.DDRIO43PB0, U_OPTO_5.COL1; no longer U_OPTO_2.C1
- net N$3: now also R23.1, U_OPTO_4.C2; no longer C1.1, Q1.1, U_CH340G.XI
- net N$44: now also R34.1, SF2_M2S010TQ1G$1.DDRIO47NB0; no longer R12.2, U_OPTO_3.C2
- net N$45: now also R35.2, SF2_M2S010TQ1G$1.DDRIO48NB0; no longer RN12D.2, U_OPTO_2.COL2
- net N$46: now also R40.2, SF2_M2S010TQ1G$1.DDRIO59PB0/GB0; no longer RN11A.2, U_OPTO_2.A1
- net N$47: now also R36.2, SF2_M2S010TQ1G$1.DDRIO47PB0; no longer RN11B.2, U_OPTO_2.A2
- net N$48: now also R41.2, SF2_M2S010TQ1G$1.DDRIO63PB0; no longer U_OPTO_2.C2
- net N$49: now also R46.1, SF2_M2S010TQ1G$2.MSIO3NB2/USB_DATA1_B; no longer R11.2, U_OPTO_3.C1
- net N$68: now also R52.2, SF2_M2S010TQ1G$4.MSIO108NB4; no longer R22.1, U_ADR366_3.TRIM
- net N$69: now also R55.2, SF2_M2S010TQ1G$4.MSIO108PB4; no longer R22.2, R24.1, R25.2
- net N$70: now also R56.2, SF2_M2S010TQ1G$4.MSIO106NB4; no longer R23.2, R25.1
- net SODS: now also SF2_M2S010TQ1G$1.DDRIO44NB0, U_OPTO_5.COL2; no longer U_OPTO_1.C1
- net SOE: now also SF2_M2S010TQ1G$1.DDRIO44PB0, U_OPTO_3.COL1; no longer U_OPTO_1.C2
Other:
- note added: "3dB attenuation @ 1989Hz"
- note removed: "FL1"
- note removed: "FLASH mem"
- note removed: "Feinabgleich"
- note removed: "Filter/Buffer caps."
- note removed: "Opto. isolation"
- note removed: "RS422 driver"
- note removed: "Ref voltage"
- note removed: "Spike/ESD protection"
- note removed: "USB- UART"
- note removed: "logic side <-> RXSM side"
- moved on the sheet: C44, D1, D5, R1, R10, R11, R12, R13, R15, R16, R17, R22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

Commit message: Almost final sch
Connections:
- removed net LED_1: RN10A.1
- removed net LED_2: RN10B.1
- removed net LED_3: RN10C.1
- removed net N$28: U$4.WP#/IO2, WP.2
- new net HB_MSS: RN10C.1, SF2_M2S010TQ1G$6.MSIO77NB7
- new net HB_STAMPS: RN10A.1, SF2_M2S010TQ1G$6.MSIO76NB7
- new net HB_STORAGE: RN10B.1, SF2_M2S010TQ1G$6.MSIO76PB7
- new net LED4: SF2_M2S010TQ1G$6.MSIO77PB7
- new net WP: SF2_M2S010TQ1G$6.MSIO71PB7, U$4.WP#/IO2, WP.2
Other:
- note removed: "(5V-)28V rail 3V3 5V User LED 1 - 4"
- note removed: "V. Reg"
- moved on the sheet: C34, C35, C36, C37, C38, C39, C40, C41, C42, C43, C60, C61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

Commit message: Minor changes
Parts:
- removed U$2: USB_B_STANDING, selfmade:USB_B_STANDING
- added CN1: (no value), adafruit:USBMINIB
- added X1: (no value), con-subd:F15HP
Connections:
- net 28V: now also X1.1, X1.9
- net 28VGND: now also X1.15, X1.8
- net EXP_IN_N: now also X1.14
- net EXP_IN_P: now also X1.13
- net EXP_OUT_N: now also X1.7
- net EXP_OUT_P: now also X1.6
- net GND: now also CN1.GND; no longer U$2.S, U$2.V-
- net N$16: now also CN1.VBUS; no longer U$2.V+
- net RXSM_LO: now also X1.5
- net RXSM_SODS: now also X1.3
- net RXSM_SOE: now also X1.4
- net USB_N: now also CN1.D-; no longer U$2.D-
- net USB_P: now also CN1.D+; no longer U$2.D+
Other:
- moved on the sheet: C10, C11, C12, C13, C14, C15, C16, C17, C18, C19, C20, C21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

Commit message: Adds changes as of Grimsmann
Parts:
- added C28, C29: 100n, rcl:C-EUC0805
- added C30, C31, C32: 10u, rcl:CPOL-EUE/7260-38W
- added R24: 2k2, rcl:R-EU_R0805
- added U_LT1: LT1528, aSparkFun:LT1528
Connections:
- removed net LED_4: RN10D.1
- new net N$34: C29.1
- new net N$37: R24.1
- new net N$39: C31.2, C32.1
- new net N$40: C32.2
- net 3V3: now also C28.1, C30.1, R24.2, R27.2, U$5.STDBY
- net 5V: now also C28.2, C30.+, U_LT1.IN, U_LT1.SHDN
- net EED: now also R24.2; no longer R27.2
- net GND: now also C28.1, C28.2, C29.1, C29.2, C30.-, C30.2, C31.-, C31.1, C32.-, U_LT1.GND
- net LED4: now also RN10D.1
- net N$23: now also R24.1
- net VCCINT: now also C29.2, C31.+, C32.+, U_LT1.OUT, U_LT1.SENSE
Other:
- moved on the sheet: C42, C43, R27

Commit message: First STAMP layout
Parts:
- removed C34: 100n, rcl:C-EUC0805
- removed R34, R37, R38, R39, R42, R43, R44, R47, R48, R49, R52, R53, R54, R57, R58, R59, R62, R63, R67: 47, rcl:R-EU_R0805
- C42: device rcl:C-EUC0805 -> rcl:C-EUC1206
Connections:
- removed net N$44: R34.1, SF2_M2S010TQ1G$1.DDRIO47NB0
- removed net N$53: R37.2, SF2_M2S010TQ1G$1.DDRIO55PB0/CCC_NE0_CLKI3
- removed net N$54: R38.2, SF2_M2S010TQ1G$1.DDRIO59NB0/GB4
- removed net N$57: R39.2, SF2_M2S010TQ1G$1.DDRIO60NB0/CCC_NE1_CLKI3
- removed net N$58: R42.1, SF2_M2S010TQ1G$2.MSIO2NB2/USB_NXT_B
- removed net N$59: R43.1, SF2_M2S010TQ1G$2.MSIO3PB2/USB_DATA0_B
- removed net N$60: R44.1, SF2_M2S010TQ1G$2.MSIO4PB2/USB_DATA2_B
- removed net N$61: R47.1, SF2_M2S010TQ1G$4.MSIO104NB4/GB7
- removed net N$62: R48.1, SF2_M2S010TQ1G$4.MSIO104PB4/GB3
- removed net N$63: R49.1, SF2_M2S010TQ1G$4.MSIO105PB4/CCC_NE0_CLKI0
- removed net N$66: R54.2, SF2_M2S010TQ1G$4.MSIO109NB4
- removed net N$67: R53.2, SF2_M2S010TQ1G$4.MSIO109PB4
- removed net N$68: R52.2, SF2_M2S010TQ1G$4.MSIO108NB4
- removed net N$71: R57.1, SF2_M2S010TQ1G$5.MSIOD93NB6
- removed net N$72: R58.1, SF2_M2S010TQ1G$5.MSIOD93PB6
- removed net N$73: R59.2, SF2_M2S010TQ1G$5.MSIOD96PB6
- removed net N$76: R62.1, SF2_M2S010TQ1G$6.MSIO67NB7
- removed net N$77: R63.1, SF2_M2S010TQ1G$6.MSIO67PB7
- removed net N$78: R67.1, SF2_M2S010TQ1G$6.MSIO71NB7
- net 28V: no longer C34.2
- net 28VGND: no longer C34.1
- net ADC_START: now also SF2_M2S010TQ1G$1.DDRIO47NB0; no longer R34.2
- net HB_MSS: now also SF2_M2S010TQ1G$6.MSIO76PB7; no longer SF2_M2S010TQ1G$6.MSIO77NB7
- net HB_STAMPS: now also SF2_M2S010TQ1G$6.MSIO77PB7; no longer SF2_M2S010TQ1G$6.MSIO76NB7
- net HB_STORAGE: now also SF2_M2S010TQ1G$6.MSIO77NB7; no longer SF2_M2S010TQ1G$6.MSIO76PB7
- net LED4: now also SF2_M2S010TQ1G$6.MSIO76NB7; no longer SF2_M2S010TQ1G$6.MSIO77PB7
- net STAMP1_CS_SG1: now also SF2_M2S010TQ1G$1.DDRIO55PB0/CCC_NE0_CLKI3; no longer R37.1
- net STAMP1_CS_SG2: now also SF2_M2S010TQ1G$1.DDRIO59NB0/GB4; no longer R38.1
- net STAMP1_CS_TEMP: now also SF2_M2S010TQ1G$1.DDRIO60NB0/CCC_NE1_CLKI3; no longer R39.1
- net STAMP2_CS_SG1: now also SF2_M2S010TQ1G$2.MSIO2NB2/USB_NXT_B; no longer R42.2
- net STAMP2_CS_SG2: now also SF2_M2S010TQ1G$2.MSIO3PB2/USB_DATA0_B; no longer R43.2
- net STAMP2_CS_TEMP: now also SF2_M2S010TQ1G$2.MSIO4PB2/USB_DATA2_B; no longer R44.2
- net STAMP3_CS_SG1: now also SF2_M2S010TQ1G$4.MSIO104NB4/GB7; no longer R47.2
- net STAMP3_CS_SG2: now also SF2_M2S010TQ1G$4.MSIO104PB4/GB3; no longer R48.2
- net STAMP3_CS_TEMP: now also SF2_M2S010TQ1G$4.MSIO105PB4/CCC_NE0_CLKI0; no longer R49.2
- net STAMP4_CS_SG1: now also SF2_M2S010TQ1G$4.MSIO109NB4; no longer R54.1
- net STAMP4_CS_SG2: now also SF2_M2S010TQ1G$4.MSIO109PB4; no longer R53.1
- net STAMP4_CS_TEMP: now also SF2_M2S010TQ1G$4.MSIO108NB4; no longer R52.1
- net STAMP5_CS_SG1: now also SF2_M2S010TQ1G$5.MSIOD93NB6; no longer R57.2
- net STAMP5_CS_SG2: now also SF2_M2S010TQ1G$5.MSIOD93PB6; no longer R58.2
- net STAMP5_CS_TEMP: now also SF2_M2S010TQ1G$5.MSIOD96PB6; no longer R59.1
- net STAMP6_CS_SG1: now also SF2_M2S010TQ1G$6.MSIO67NB7; no longer R62.2
- net STAMP6_CS_SG2: now also SF2_M2S010TQ1G$6.MSIO67PB7; no longer R63.2
- net STAMP6_CS_TEMP: now also SF2_M2S010TQ1G$6.MSIO71NB7; no longer R67.2
