File: SPU.sch (EAGLE design)
At the start: 120 parts, among them Q2 CSTCR6M00G53Z

Commit message: Before autoroute
Parts:
- removed U$1: FT2232D, smf2:FT2232D
- removed U$3: M93C46-WDW6TP, smf2:M93C46-WDW6TP
- removed U$4: S70FL01GSAGM, smf2:S70FL01GSAGM
- added C100, C101, C102, C103, C104, C105, C113, C115, C116, C117, C118, C119, C121, C122, C123, C124, C125, C126, C134, C136, C137, C138, C139, C140, C142, C143, C144, C145, C146, C147, C155, C157, C158, C159, C160, C161, C163, C164, C165, C166, C167, C168, C197, C199, C200, C201, C202, C203, C205, C206, C207, C208, C209, C210, C33, C45, C46, C47, C48, C49, C51, C52, C53, C54, C55, C56, C92, C94, C95, C96, C97, C98: 100n, rcl:C-EUC0805
- added C106, C108, C127, C129, C148, C150, C169, C171, C211, C213, C57, C59: 6n8, rcl:C-EUC0805
- added C107, C128, C149, C170, C212, C58: 68n, rcl:C-EUC0805
- added C109, C114, C120, C130, C135, C141, C151, C156, C162, C172, C198, C204, C214, C34, C50, C63, C93, C99: 1u, rcl:C-EUC0805
- added C110, C131, C152, C173, C215, C68: 33n, rcl:C-EUC0805
- added C111, C112, C132, C133, C153, C154, C174, C175, C216, C217, C69, C70: 3n3, rcl:C-EUC0805
- added CON_STAMP1, CON_STAMP3, CON_STAMP4, CON_STAMP5, CON_STAMP6, CON_STAMP8: IL-AG5-10P-S3T2, con-jae:IL-AG5-10P-S3T2
- added FTDI: FT2232D, smf2:FT2232D
- added FT_EEPROM: M93C46-WDW6TP, smf2:M93C46-WDW6TP
- added R100, R106, R113, R119, R125, R132, R138, R144, R151, R176, R182, R189, R28, R68, R71, R77, R87, R94: 4k7, rcl:R-EU_R0805
- added R101, R105, R107, R111, R120, R124, R126, R130, R139, R143, R145, R149, R177, R181, R183, R187, R30, R33, R69, R74, R76, R86, R88, R92: 1k 0.1%, rcl:R-EU_R0805
- added R102, R108, R112, R121, R127, R131, R140, R146, R150, R178, R184, R188, R31, R70, R75, R83, R89, R93: 47, rcl:R-EU_R0805
- added R103, R104, R109, R110, R122, R123, R128, R129, R141, R142, R147, R148, R179, R180, R185, R186, R29, R32, R72, R73, R84, R85, R90, R91: 40 1%, rcl:R-EU_R0805
- added R114, R115, R133, R134, R152, R153, R190, R191, R78, R79, R95, R96: 4k7 1%, rcl:R-EU_R0805
- added R116, R117, R135, R136, R154, R155, R192, R193, R80, R81, R97, R98: 9k09 1%, rcl:R-EU_R0805
- added R118, R137, R156, R194, R82, R99: 820 0.1%, rcl:R-EU_R0805
- added S70FL: S70FL01GSAGM, smf2:S70FL01GSAGM
- added STAMP1_ADC_SG1, STAMP1_ADC_SG10, STAMP1_ADC_SG11, STAMP1_ADC_SG12, STAMP1_ADC_SG15, STAMP1_ADC_SG16, STAMP1_ADC_SG2, STAMP1_ADC_SG5, STAMP1_ADC_SG6, STAMP1_ADC_SG7, STAMP1_ADC_SG8, STAMP1_ADC_SG9, STAMP1_ADC_TEMP, STAMP1_ADC_TEMP2, STAMP1_ADC_TEMP3, STAMP1_ADC_TEMP4, STAMP1_ADC_TEMP5, STAMP1_ADC_TEMP7: ADS1148QPWRQ1, ads11xx:ADS1148QPWRQ1
- added U$10, U$11, U$12, U$13, U$14, U$15, U$16, U$19, U$20, U$6, U$7, U$9: COMMON_MODE_CHOKE, selfmade:COMMON_MODE_CHOKE
Connections:
- new net N$100: R89.2, STAMP1_ADC_SG6.DOUT/!DRDY
- new net N$101: C101.2, C102.1, R90.1, STAMP1_ADC_SG6.AIN0/IEXC
- new net N$102: C102.2, C103.1, R91.1, STAMP1_ADC_SG6.AIN1/IEXC
- new net N$103: R88.1, R91.2, R92.1
- new net N$104: R90.2, U$10.3
- new net N$105: R93.2, STAMP1_ADC_TEMP2.DOUT/!DRDY
- new net N$106: R94.1, STAMP1_ADC_TEMP2.!RESET
- new net N$107: C106.2, C107.1, R95.1, STAMP1_ADC_TEMP2.AIN1/IEXC
- new net N$108: C107.2, C108.1, R96.1, STAMP1_ADC_TEMP2.AIN2/IEXC/GPIO2
- new net N$109: C109.1, STAMP1_ADC_TEMP2.VREFOUT
- new net N$110: C110.2, C111.1, R98.1, STAMP1_ADC_TEMP2.REFN0/GPIO1
- new net N$111: C110.1, C112.2, R97.1, STAMP1_ADC_TEMP2.REFP0/GPIO0
- new net N$112: R100.1, STAMP1_ADC_SG7.!RESET
- new net N$113: C114.1, STAMP1_ADC_SG7.VREFOUT
- new net N$114: R102.2, STAMP1_ADC_SG7.DOUT/!DRDY
- new net N$115: C116.2, C117.1, R103.1, STAMP1_ADC_SG7.AIN0/IEXC
- new net N$116: C117.2, C118.1, R104.1, STAMP1_ADC_SG7.AIN1/IEXC
- new net N$117: R101.1, R104.2, R105.1
- new net N$118: R103.2, U$11.3
- new net N$119: R106.1, STAMP1_ADC_SG8.!RESET
- new net N$120: C120.1, STAMP1_ADC_SG8.VREFOUT
- new net N$121: R108.2, STAMP1_ADC_SG8.DOUT/!DRDY
- new net N$122: C122.2, C123.1, R109.1, STAMP1_ADC_SG8.AIN0/IEXC
- new net N$123: C123.2, C124.1, R110.1, STAMP1_ADC_SG8.AIN1/IEXC
- new net N$124: R107.1, R110.2, R111.1
- new net N$125: R109.2, U$12.3
- new net N$126: R112.2, STAMP1_ADC_TEMP3.DOUT/!DRDY
- new net N$127: R113.1, STAMP1_ADC_TEMP3.!RESET
- new net N$128: C127.2, C128.1, R114.1, STAMP1_ADC_TEMP3.AIN1/IEXC
- new net N$129: C128.2, C129.1, R115.1, STAMP1_ADC_TEMP3.AIN2/IEXC/GPIO2
- new net N$130: C130.1, STAMP1_ADC_TEMP3.VREFOUT
- new net N$131: C131.2, C132.1, R117.1, STAMP1_ADC_TEMP3.REFN0/GPIO1
- new net N$132: C131.1, C133.2, R116.1, STAMP1_ADC_TEMP3.REFP0/GPIO0
- new net N$133: R119.1, STAMP1_ADC_SG9.!RESET
- new net N$134: C135.1, STAMP1_ADC_SG9.VREFOUT
- new net N$135: R121.2, STAMP1_ADC_SG9.DOUT/!DRDY
- new net N$136: C137.2, C138.1, R122.1, STAMP1_ADC_SG9.AIN0/IEXC
- new net N$137: C138.2, C139.1, R123.1, STAMP1_ADC_SG9.AIN1/IEXC
- new net N$138: R120.1, R123.2, R124.1
- new net N$139: R122.2, U$13.3
- new net N$140: R125.1, STAMP1_ADC_SG10.!RESET
- new net N$141: C141.1, STAMP1_ADC_SG10.VREFOUT
- new net N$142: R127.2, STAMP1_ADC_SG10.DOUT/!DRDY
- new net N$143: C143.2, C144.1, R128.1, STAMP1_ADC_SG10.AIN0/IEXC
- new net N$144: C144.2, C145.1, R129.1, STAMP1_ADC_SG10.AIN1/IEXC
- new net N$145: R126.1, R129.2, R130.1
- new net N$146: R128.2, U$14.3
- new net N$147: R131.2, STAMP1_ADC_TEMP4.DOUT/!DRDY
- new net N$148: R132.1, STAMP1_ADC_TEMP4.!RESET
- new net N$149: C148.2, C149.1, R133.1, STAMP1_ADC_TEMP4.AIN1/IEXC
- new net N$150: C149.2, C150.1, R134.1, STAMP1_ADC_TEMP4.AIN2/IEXC/GPIO2
- new net N$151: C151.1, STAMP1_ADC_TEMP4.VREFOUT
- new net N$152: C152.2, C153.1, R136.1, STAMP1_ADC_TEMP4.REFN0/GPIO1
- new net N$153: C152.1, C154.2, R135.1, STAMP1_ADC_TEMP4.REFP0/GPIO0
- new net N$154: R138.1, STAMP1_ADC_SG11.!RESET
- new net N$155: C156.1, STAMP1_ADC_SG11.VREFOUT
- new net N$156: R140.2, STAMP1_ADC_SG11.DOUT/!DRDY
- new net N$157: C158.2, C159.1, R141.1, STAMP1_ADC_SG11.AIN0/IEXC
- new net N$158: C159.2, C160.1, R142.1, STAMP1_ADC_SG11.AIN1/IEXC
- new net N$159: R139.1, R142.2, R143.1
- new net N$160: R141.2, U$15.3
- new net N$161: R144.1, STAMP1_ADC_SG12.!RESET
- new net N$162: C162.1, STAMP1_ADC_SG12.VREFOUT
- new net N$163: R146.2, STAMP1_ADC_SG12.DOUT/!DRDY
- new net N$164: C164.2, C165.1, R147.1, STAMP1_ADC_SG12.AIN0/IEXC
- new net N$165: C165.2, C166.1, R148.1, STAMP1_ADC_SG12.AIN1/IEXC
- new net N$166: R145.1, R148.2, R149.1
- new net N$167: R147.2, U$16.3
- new net N$168: R150.2, STAMP1_ADC_TEMP5.DOUT/!DRDY
- new net N$169: R151.1, STAMP1_ADC_TEMP5.!RESET
- new net N$170: C169.2, C170.1, R152.1, STAMP1_ADC_TEMP5.AIN1/IEXC
- new net N$171: C170.2, C171.1, R153.1, STAMP1_ADC_TEMP5.AIN2/IEXC/GPIO2
- new net N$172: C172.1, STAMP1_ADC_TEMP5.VREFOUT
- new net N$173: C173.2, C174.1, R155.1, STAMP1_ADC_TEMP5.REFN0/GPIO1
- new net N$174: C173.1, C175.2, R154.1, STAMP1_ADC_TEMP5.REFP0/GPIO0
- new net N$196: R176.1, STAMP1_ADC_SG15.!RESET
- new net N$197: C198.1, STAMP1_ADC_SG15.VREFOUT
- new net N$198: R178.2, STAMP1_ADC_SG15.DOUT/!DRDY
- new net N$199: C200.2, C201.1, R179.1, STAMP1_ADC_SG15.AIN0/IEXC
- new net N$200: C201.2, C202.1, R180.1, STAMP1_ADC_SG15.AIN1/IEXC
- new net N$201: R177.1, R180.2, R181.1
- new net N$202: R179.2, U$19.3
- new net N$203: R182.1, STAMP1_ADC_SG16.!RESET
- new net N$204: C204.1, STAMP1_ADC_SG16.VREFOUT
- new net N$205: R184.2, STAMP1_ADC_SG16.DOUT/!DRDY
- new net N$206: C206.2, C207.1, R185.1, STAMP1_ADC_SG16.AIN0/IEXC
- new net N$207: C207.2, C208.1, R186.1, STAMP1_ADC_SG16.AIN1/IEXC
- new net N$208: R183.1, R186.2, R187.1
- new net N$209: R185.2, U$20.3
- new net N$210: R188.2, STAMP1_ADC_TEMP7.DOUT/!DRDY
- new net N$211: R189.1, STAMP1_ADC_TEMP7.!RESET
- new net N$212: C211.2, C212.1, R190.1, STAMP1_ADC_TEMP7.AIN1/IEXC
- new net N$213: C212.2, C213.1, R191.1, STAMP1_ADC_TEMP7.AIN2/IEXC/GPIO2
- new net N$214: C214.1, STAMP1_ADC_TEMP7.VREFOUT
- new net N$215: C215.2, C216.1, R193.1, STAMP1_ADC_TEMP7.REFN0/GPIO1
- new net N$216: C215.1, C217.2, R192.1, STAMP1_ADC_TEMP7.REFP0/GPIO0
- new net N$35: R68.1, STAMP1_ADC_SG2.!RESET
- new net N$38: R31.2, STAMP1_ADC_SG1.DOUT/!DRDY
- new net N$41: C50.1, STAMP1_ADC_SG2.VREFOUT
- new net N$43: R70.2, STAMP1_ADC_SG2.DOUT/!DRDY
- new net N$78: R71.1, STAMP1_ADC_SG5.!RESET
- new net N$79: C52.2, C53.1, R72.1, STAMP1_ADC_SG2.AIN0/IEXC
- new net N$80: C53.2, C54.1, R73.1, STAMP1_ADC_SG2.AIN1/IEXC
- new net N$81: R30.1, R32.2, R33.1
- new net N$82: R69.1, R73.2, R74.1
- new net N$83: R29.2, U$6.3
- new net N$84: R72.2, U$7.3
- new net N$85: C93.1, STAMP1_ADC_SG5.VREFOUT
- new net N$86: R75.2, STAMP1_ADC_TEMP.DOUT/!DRDY
- new net N$87: R77.1, STAMP1_ADC_TEMP.!RESET
- new net N$88: C57.2, C58.1, R78.1, STAMP1_ADC_TEMP.AIN1/IEXC
- new net N$89: C58.2, C59.1, R79.1, STAMP1_ADC_TEMP.AIN2/IEXC/GPIO2
- new net N$90: C63.1, STAMP1_ADC_TEMP.VREFOUT
- new net N$91: C68.2, C69.1, R81.1, STAMP1_ADC_TEMP.REFN0/GPIO1
- new net N$92: C68.1, C70.2, R80.1, STAMP1_ADC_TEMP.REFP0/GPIO0
- new net N$93: R83.2, STAMP1_ADC_SG5.DOUT/!DRDY
- new net N$94: C95.2, C96.1, R84.1, STAMP1_ADC_SG5.AIN0/IEXC
- new net N$95: C96.2, C97.1, R85.1, STAMP1_ADC_SG5.AIN1/IEXC
- new net N$96: R76.1, R85.2, R86.1
- new net N$97: R84.2, U$9.3
- new net N$98: R87.1, STAMP1_ADC_SG6.!RESET
- new net N$99: C99.1, STAMP1_ADC_SG6.VREFOUT
- new net STAMP1_SG1_AIN1: CON_STAMP1.P$1, U$6.6
- new net STAMP1_SG1_AIN2: CON_STAMP1.P$2, U$6.4
- new net STAMP1_SG1_AIN3: CON_STAMP1.P$3, U$6.2
- new net STAMP1_SG2_AIN1: CON_STAMP1.P$10, U$7.6
- new net STAMP1_SG2_AIN2: CON_STAMP1.P$9, U$7.4
- new net STAMP1_SG2_AIN3: CON_STAMP1.P$8, U$7.2
- new net STAMP1_TEMP_AIN1: CON_STAMP1.P$4, R78.2, STAMP1_ADC_TEMP.AIN0/IEXC
- new net STAMP1_TEMP_AIN2: CON_STAMP1.P$5, R79.2, STAMP1_ADC_TEMP.AIN3/IEXC/GPIO3
- new net STAMP1_TEMP_AIN3: CON_STAMP1.P$6, R80.2, R82.2
- new net STAMP2_SG1_AIN1: CON_STAMP3.P$1, U$9.6
- new net STAMP2_SG1_AIN2: CON_STAMP3.P$2, U$9.4
- new net STAMP2_SG1_AIN3: CON_STAMP3.P$3, U$9.2
- new net STAMP2_SG2_AIN1: CON_STAMP3.P$10, U$10.6
- new net STAMP2_SG2_AIN2: CON_STAMP3.P$9, U$10.4
- new net STAMP2_SG2_AIN3: CON_STAMP3.P$8, U$10.2
- new net STAMP2_TEMP_AIN1: CON_STAMP3.P$4, R95.2, STAMP1_ADC_TEMP2.AIN0/IEXC
- new net STAMP2_TEMP_AIN2: CON_STAMP3.P$5, R96.2, STAMP1_ADC_TEMP2.AIN3/IEXC/GPIO3
- new net STAMP2_TEMP_AIN3: CON_STAMP3.P$6, R97.2, R99.2
- new net STAMP3_SG1_AIN1: CON_STAMP5.P$1, U$13.6
- new net STAMP3_SG1_AIN2: CON_STAMP5.P$2, U$13.4
- new net STAMP3_SG1_AIN3: CON_STAMP5.P$3, U$13.2
- new net STAMP3_SG2_AIN1: CON_STAMP5.P$10, U$14.6
- new net STAMP3_SG2_AIN2: CON_STAMP5.P$9, U$14.4
- new net STAMP3_SG2_AIN3: CON_STAMP5.P$8, U$14.2
- new net STAMP3_TEMP_AIN1: CON_STAMP5.P$4, R133.2, STAMP1_ADC_TEMP4.AIN0/IEXC
- new net STAMP3_TEMP_AIN2: CON_STAMP5.P$5, R134.2, STAMP1_ADC_TEMP4.AIN3/IEXC/GPIO3
- new net STAMP3_TEMP_AIN3: CON_STAMP5.P$6, R135.2, R137.2
- new net STAMP4_SG1_AIN1: CON_STAMP6.P$1, U$15.6
- new net STAMP4_SG1_AIN2: CON_STAMP6.P$2, U$15.4
- new net STAMP4_SG1_AIN3: CON_STAMP6.P$3, U$15.2
- new net STAMP4_SG2_AIN1: CON_STAMP6.P$10, U$16.6
- new net STAMP4_SG2_AIN2: CON_STAMP6.P$9, U$16.4
- new net STAMP4_SG2_AIN3: CON_STAMP6.P$8, U$16.2
- new net STAMP4_TEMP_AIN1: CON_STAMP6.P$4, R152.2, STAMP1_ADC_TEMP5.AIN0/IEXC
- new net STAMP4_TEMP_AIN2: CON_STAMP6.P$5, R153.2, STAMP1_ADC_TEMP5.AIN3/IEXC/GPIO3
- new net STAMP4_TEMP_AIN3: CON_STAMP6.P$6, R154.2, R156.2
- new net STAMP5_SG1_AIN1: CON_STAMP4.P$1, U$11.6
- new net STAMP5_SG1_AIN2: CON_STAMP4.P$2, U$11.4
- new net STAMP5_SG1_AIN3: CON_STAMP4.P$3, U$11.2
- new net STAMP5_SG2_AIN1: CON_STAMP4.P$10, U$12.6
- new net STAMP5_SG2_AIN2: CON_STAMP4.P$9, U$12.4
- new net STAMP5_SG2_AIN3: CON_STAMP4.P$8, U$12.2
- new net STAMP5_TEMP_AIN1: CON_STAMP4.P$4, R114.2, STAMP1_ADC_TEMP3.AIN0/IEXC
- new net STAMP5_TEMP_AIN2: CON_STAMP4.P$5, R115.2, STAMP1_ADC_TEMP3.AIN3/IEXC/GPIO3
- new net STAMP5_TEMP_AIN3: CON_STAMP4.P$6, R116.2, R118.2
- new net STAMP6_SG1_AIN1: CON_STAMP8.P$1, U$19.6
- new net STAMP6_SG1_AIN2: CON_STAMP8.P$2, U$19.4
- new net STAMP6_SG1_AIN3: CON_STAMP8.P$3, U$19.2
- new net STAMP6_SG2_AIN1: CON_STAMP8.P$10, U$20.6
- new net STAMP6_SG2_AIN2: CON_STAMP8.P$9, U$20.4
- new net STAMP6_SG2_AIN3: CON_STAMP8.P$8, U$20.2
- new net STAMP6_TEMP_AIN1: CON_STAMP8.P$4, R190.2, STAMP1_ADC_TEMP7.AIN0/IEXC
- new net STAMP6_TEMP_AIN2: CON_STAMP8.P$5, R191.2, STAMP1_ADC_TEMP7.AIN3/IEXC/GPIO3
- new net STAMP6_TEMP_AIN3: CON_STAMP8.P$6, R192.2, R194.2
- net 3V3: now also C100.1, C104.1, C105.1, C113.1, C115.1, C119.1, C121.1, C125.1, C126.1, C134.1, C136.1, C140.1, C142.1, C146.1, C147.1, C155.1, C157.1, C161.1, C163.1, C167.1, C168.1, C197.1, C199.1, C203.1, C205.1, C209.1, C210.1, C33.1, C45.1, C49.1, C51.1, C55.1, C56.1, C92.1, C94.1, C98.1, FTDI.VCC, FTDI.VCC1, FTDI.VCCIOB, FTDI.VVCIOA, FT_EEPROM.ORG, FT_EEPROM.VCC, R100.2, R105.2, R106.2, R111.2, R113.2, R119.2, R124.2, R125.2, R130.2, R132.2, R138.2, R143.2, R144.2, R149.2, R151.2, R176.2, R181.2, R182.2, R187.2, R189.2, R28.2, R33.2, R68.2, R71.2, R74.2, R77.2, R86.2, R87.2, R92.2, R94.2, S70FL.VCC, STAMP1_ADC_SG1.AVDD, STAMP1_ADC_SG1.DVDD, STAMP1_ADC_SG10.AVDD, STAMP1_ADC_SG10.DVDD, STAMP1_ADC_SG11.AVDD, STAMP1_ADC_SG11.DVDD, STAMP1_ADC_SG12.AVDD, STAMP1_ADC_SG12.DVDD, STAMP1_ADC_SG15.AVDD, STAMP1_ADC_SG15.DVDD, STAMP1_ADC_SG16.AVDD, STAMP1_ADC_SG16.DVDD, STAMP1_ADC_SG2.AVDD, STAMP1_ADC_SG2.DVDD, STAMP1_ADC_SG5.AVDD, STAMP1_ADC_SG5.DVDD, STAMP1_ADC_SG6.AVDD, STAMP1_ADC_SG6.DVDD, STAMP1_ADC_SG7.AVDD, STAMP1_ADC_SG7.DVDD, STAMP1_ADC_SG8.AVDD, STAMP1_ADC_SG8.DVDD, STAMP1_ADC_SG9.AVDD, STAMP1_ADC_SG9.DVDD, STAMP1_ADC_TEMP.AVDD, STAMP1_ADC_TEMP.DVDD, STAMP1_ADC_TEMP2.AVDD, STAMP1_ADC_TEMP2.DVDD, STAMP1_ADC_TEMP3.AVDD, STAMP1_ADC_TEMP3.DVDD, STAMP1_ADC_TEMP4.AVDD, STAMP1_ADC_TEMP4.DVDD, STAMP1_ADC_TEMP5.AVDD, STAMP1_ADC_TEMP5.DVDD, STAMP1_ADC_TEMP7.AVDD, STAMP1_ADC_TEMP7.DVDD, U$10.5, U$11.5, U$12.5, U$13.5, U$14.5, U$15.5, U$16.5, U$19.5, U$20.5, U$6.5, U$7.5, U$9.5; no longer C28.1, C30.1, R24.2, U$1.VCC, U$1.VCC1, U$1.VCCIOB, U$1.VVCIOA, U$3.ORG, U$3.VCC, U$4.VCC
- net ADC_START: now also STAMP1_ADC_SG1.START, STAMP1_ADC_SG10.START, STAMP1_ADC_SG11.START, STAMP1_ADC_SG12.START, STAMP1_ADC_SG15.START, STAMP1_ADC_SG16.START, STAMP1_ADC_SG2.START, STAMP1_ADC_SG5.START, STAMP1_ADC_SG6.START, STAMP1_ADC_SG7.START, STAMP1_ADC_SG8.START, STAMP1_ADC_SG9.START, STAMP1_ADC_TEMP.START, STAMP1_ADC_TEMP2.START, STAMP1_ADC_TEMP3.START, STAMP1_ADC_TEMP4.START, STAMP1_ADC_TEMP5.START, STAMP1_ADC_TEMP7.START
- net DAPI_CTS: now also FTDI.BDBUS2; no longer U$1.BDBUS2
- net DAPI_DSR: now also FTDI.BDBUS4; no longer U$1.BDBUS4
- net DAPI_DTR: now also FTDI.BDBUS5; no longer U$1.BDBUS5
- net DAPI_RTS: now also FTDI.BDBUS3; no longer U$1.BDBUS3
- net DAPI_RXD: now also FTDI.BDBUS0; no longer U$1.BDBUS0
- net DAPI_TXD: now also FTDI.BDBUS1; no longer U$1.BDBUS1
- net EECLK: now also FTDI.EESK, FT_EEPROM.CLK; no longer U$1.EESK, U$3.CLK
- net EECS: now also FTDI.EECS, FT_EEPROM.CS; no longer U$1.EECS, U$3.CS
- net EED: now also FTDI.EEDATA, FT_EEPROM.DIN; no longer U$1.EEDATA, U$3.DIN
- net F_CLK: now also S70FL.SCLK; no longer U$4.SCLK
- net F_CS1: now also S70FL.CS1#; no longer U$4.CS1#
- net F_CS2: now also S70FL.CS2#; no longer U$4.CS2#
- net F_MISO: now also S70FL.SO/O1; no longer U$4.SO/O1
- net F_MOSI: now also S70FL.SI/O0; no longer U$4.SI/O0
- net GND: now also C100.2, C101.1, C103.2, C104.2, C105.2, C106.1, C108.2, C109.2, C111.2, C112.1, C113.2, C114.2, C115.2, C116.1, C118.2, C119.2, C120.2, C121.2, C122.1, C124.2, C125.2, C126.2, C127.1, C129.2, C130.2, C132.2, C133.1, C134.2, C135.2, C136.2, C137.1, C139.2, C140.2, C141.2, C142.2, C143.1, C145.2, C146.2, C147.2, C148.1, C150.2, C151.2, C153.2, C154.1, C155.2, C156.2, C157.2, C158.1, C160.2, C161.2, C162.2, C163.2, C164.1, C166.2, C167.2, C168.2, C169.1, C171.2, C172.2, C174.2, C175.1, C197.2, C198.2, C199.2, C200.1, C202.2, C203.2, C204.2, C205.2, C206.1, C208.2, C209.2, C210.2, C211.1, C213.2, C214.2, C216.2, C217.1, C33.2, C34.2, C45.2, C46.1, C48.2, C49.2, C50.2, C51.2, C52.1, C54.2, C55.2, C56.2, C57.1, C59.2, C63.2, C69.2, C70.1, C92.2, C93.2, C94.2, C95.1, C97.2, C98.2, C99.2, CON_STAMP1.P$7, CON_STAMP3.P$7, CON_STAMP4.P$7, CON_STAMP5.P$7, CON_STAMP6.P$7, CON_STAMP8.P$7, FTDI.AGND, FTDI.GND1, FTDI.GND2, FTDI.GND3, FTDI.GND4, FTDI.TEST, FT_EEPROM.VSS, R101.2, R107.2, R117.2, R118.1, R120.2, R126.2, R136.2, R137.1, R139.2, R145.2, R155.2, R156.1, R177.2, R183.2, R193.2, R194.1, R30.2, R69.2, R76.2, R81.2, R82.1, R88.2, R98.2, R99.1, S70FL.VSS, STAMP1_ADC_SG1.AVSS, STAMP1_ADC_SG1.DGND/DSS, STAMP1_ADC_SG1.VREFCOM, STAMP1_ADC_SG10.AVSS, STAMP1_ADC_SG10.DGND/DSS, STAMP1_ADC_SG10.VREFCOM, STAMP1_ADC_SG11.AVSS, STAMP1_ADC_SG11.DGND/DSS, STAMP1_ADC_SG11.VREFCOM, STAMP1_ADC_SG12.AVSS, STAMP1_ADC_SG12.DGND/DSS, STAMP1_ADC_SG12.VREFCOM, STAMP1_ADC_SG15.AVSS, STAMP1_ADC_SG15.DGND/DSS, STAMP1_ADC_SG15.VREFCOM, STAMP1_ADC_SG16.AVSS, STAMP1_ADC_SG16.DGND/DSS, STAMP1_ADC_SG16.VREFCOM, STAMP1_ADC_SG2.AVSS, STAMP1_ADC_SG2.DGND/DSS, STAMP1_ADC_SG2.VREFCOM, STAMP1_ADC_SG5.AVSS, STAMP1_ADC_SG5.DGND/DSS, STAMP1_ADC_SG5.VREFCOM, STAMP1_ADC_SG6.AVSS, STAMP1_ADC_SG6.DGND/DSS, STAMP1_ADC_SG6.VREFCOM, STAMP1_ADC_SG7.AVSS, STAMP1_ADC_SG7.DGND/DSS, STAMP1_ADC_SG7.VREFCOM, STAMP1_ADC_SG8.AVSS, STAMP1_ADC_SG8.DGND/DSS, STAMP1_ADC_SG8.VREFCOM, STAMP1_ADC_SG9.AVSS, STAMP1_ADC_SG9.DGND/DSS, STAMP1_ADC_SG9.VREFCOM, STAMP1_ADC_TEMP.AVSS, STAMP1_ADC_TEMP.CLK, STAMP1_ADC_TEMP.DGND/DSS, STAMP1_ADC_TEMP.VREFCOM, STAMP1_ADC_TEMP2.AVSS, STAMP1_ADC_TEMP2.CLK, STAMP1_ADC_TEMP2.DGND/DSS, STAMP1_ADC_TEMP2.VREFCOM, STAMP1_ADC_TEMP3.AVSS, STAMP1_ADC_TEMP3.CLK, STAMP1_ADC_TEMP3.DGND/DSS, STAMP1_ADC_TEMP3.VREFCOM, STAMP1_ADC_TEMP4.AVSS, STAMP1_ADC_TEMP4.CLK, STAMP1_ADC_TEMP4.DGND/DSS, STAMP1_ADC_TEMP4.VREFCOM, STAMP1_ADC_TEMP5.AVSS, STAMP1_ADC_TEMP5.CLK, STAMP1_ADC_TEMP5.DGND/DSS, STAMP1_ADC_TEMP5.VREFCOM, STAMP1_ADC_TEMP7.AVSS, STAMP1_ADC_TEMP7.CLK, STAMP1_ADC_TEMP7.DGND/DSS, STAMP1_ADC_TEMP7.VREFCOM, U$10.1, U$11.1, U$12.1, U$13.1, U$14.1, U$15.1, U$16.1, U$19.1, U$20.1, U$6.1, U$7.1, U$9.1; no longer C28.2, C29.2, C30.2, C31.1, U$1.AGND, U$1.GND1, U$1.GND2, U$1.GND3, U$1.GND4, U$1.TEST, U$3.VSS, U$4.VSS
- net N$11: now also FTDI.USBDM; no longer U$1.USBDM
- net N$12: now also FTDI.XTIN; no longer U$1.XTIN
- net N$13: now also FTDI.3V3OUT; no longer U$1.3V3OUT
- net N$14: now also FTDI.AVCC; no longer U$1.AVCC
- net N$15: now also FTDI.RESET#; no longer U$1.RESET#
- net N$18: now also FTDI.ADBUS0; no longer U$1.ADBUS0
- net N$19: now also FTDI.ADBUS1; no longer U$1.ADBUS1
- net N$20: now also FTDI.ADBUS2; no longer U$1.ADBUS2
- net N$21: now also FTDI.ADBUS3; no longer U$1.ADBUS3
- net N$22: now also FTDI.XTOUT; no longer U$1.XTOUT
- net N$23: now also FT_EEPROM.DOUT; no longer U$3.DOUT
- net N$34: now also C34.1, STAMP1_ADC_SG1.VREFOUT; no longer C29.1
- net N$37: now also R28.1, STAMP1_ADC_SG1.!RESET; no longer R24.1
- net N$39: now also C46.2, C47.1, R29.1, STAMP1_ADC_SG1.AIN0/IEXC; no longer C31.2, C32.1
- net N$40: now also C47.2, C48.1, R32.1, STAMP1_ADC_SG1.AIN1/IEXC; no longer C32.2
- net N$8: now also FTDI.RSTOUT#; no longer U$1.RSTOUT#
- net N$9: now also FTDI.USBDP; no longer U$1.USBDP
- net SG_CLK: now also STAMP1_ADC_SG1.CLK, STAMP1_ADC_SG10.CLK, STAMP1_ADC_SG11.CLK, STAMP1_ADC_SG12.CLK, STAMP1_ADC_SG15.CLK, STAMP1_ADC_SG16.CLK, STAMP1_ADC_SG2.CLK, STAMP1_ADC_SG5.CLK, STAMP1_ADC_SG6.CLK, STAMP1_ADC_SG7.CLK, STAMP1_ADC_SG8.CLK, STAMP1_ADC_SG9.CLK
- net STAMP1_CS_SG1: now also STAMP1_ADC_SG1.!CS
- net STAMP1_CS_SG2: now also STAMP1_ADC_SG2.!CS
- net STAMP1_CS_TEMP: now also STAMP1_ADC_TEMP.!CS
- net STAMP1_DRDY_SG1: now also STAMP1_ADC_SG1.!DRDY
- net STAMP1_DRDY_SG2: now also STAMP1_ADC_SG2.!DRDY
- net STAMP1_DRDY_TEMP: now also STAMP1_ADC_TEMP.!DRDY
- net STAMP1_MISO: now also R31.1, R70.1, R75.1
- net STAMP1_MOSI: now also STAMP1_ADC_SG1.DIN, STAMP1_ADC_SG2.DIN, STAMP1_ADC_TEMP.DIN
- net STAMP1_SCLK: now also STAMP1_ADC_SG1.SCLK, STAMP1_ADC_SG2.SCLK, STAMP1_ADC_TEMP.SCLK
- net STAMP2_CS_SG1: now also STAMP1_ADC_SG5.!CS
- net STAMP2_CS_SG2: now also STAMP1_ADC_SG6.!CS
- net STAMP2_CS_TEMP: now also STAMP1_ADC_TEMP2.!CS
- net STAMP2_DRDY_SG1: now also STAMP1_ADC_SG5.!DRDY
- net STAMP2_DRDY_SG2: now also STAMP1_ADC_SG6.!DRDY
- net STAMP2_DRDY_TEMP: now also STAMP1_ADC_TEMP2.!DRDY
- net STAMP2_MISO: now also R83.1, R89.1, R93.1
- net STAMP2_MOSI: now also STAMP1_ADC_SG5.DIN, STAMP1_ADC_SG6.DIN, STAMP1_ADC_TEMP2.DIN
- net STAMP2_SCLK: now also STAMP1_ADC_SG5.SCLK, STAMP1_ADC_SG6.SCLK, STAMP1_ADC_TEMP2.SCLK
- net STAMP3_CS_SG1: now also STAMP1_ADC_SG9.!CS
- net STAMP3_CS_SG2: now also STAMP1_ADC_SG10.!CS
- net STAMP3_CS_TEMP: now also STAMP1_ADC_TEMP4.!CS
- net STAMP3_DRDY_SG1: now also STAMP1_ADC_SG9.!DRDY
- net STAMP3_DRDY_SG2: now also STAMP1_ADC_SG10.!DRDY
- net STAMP3_DRDY_TEMP: now also STAMP1_ADC_TEMP4.!DRDY
- net STAMP3_MISO: now also R121.1, R127.1, R131.1
- net STAMP3_MOSI: now also STAMP1_ADC_SG10.DIN, STAMP1_ADC_SG9.DIN, STAMP1_ADC_TEMP4.DIN
- net STAMP3_SCLK: now also STAMP1_ADC_SG10.SCLK, STAMP1_ADC_SG9.SCLK, STAMP1_ADC_TEMP4.SCLK
- net STAMP4_CS_SG1: now also STAMP1_ADC_SG11.!CS
- net STAMP4_CS_SG2: now also STAMP1_ADC_SG12.!CS
- net STAMP4_CS_TEMP: now also STAMP1_ADC_TEMP5.!CS
- net STAMP4_DRDY_SG1: now also STAMP1_ADC_SG11.!DRDY
- net STAMP4_DRDY_SG2: now also STAMP1_ADC_SG12.!DRDY
- net STAMP4_DRDY_TEMP: now also STAMP1_ADC_TEMP5.!DRDY
- net STAMP4_MISO: now also R140.1, R146.1, R150.1
- net STAMP4_MOSI: now also STAMP1_ADC_SG11.DIN, STAMP1_ADC_SG12.DIN, STAMP1_ADC_TEMP5.DIN
- net STAMP4_SCLK: now also STAMP1_ADC_SG11.SCLK, STAMP1_ADC_SG12.SCLK, STAMP1_ADC_TEMP5.SCLK
- net STAMP5_CS_SG1: now also STAMP1_ADC_SG7.!CS
- net STAMP5_CS_SG2: now also STAMP1_ADC_SG8.!CS
- net STAMP5_CS_TEMP: now also STAMP1_ADC_TEMP3.!CS
- net STAMP5_DRDY_SG1: now also STAMP1_ADC_SG7.!DRDY
- net STAMP5_DRDY_SG2: now also STAMP1_ADC_SG8.!DRDY
- net STAMP5_DRDY_TEMP: now also STAMP1_ADC_TEMP3.!DRDY
- net STAMP5_MISO: now also R102.1, R108.1, R112.1
- net STAMP5_MOSI: now also STAMP1_ADC_SG7.DIN, STAMP1_ADC_SG8.DIN, STAMP1_ADC_TEMP3.DIN
- net STAMP5_SCLK: now also STAMP1_ADC_SG7.SCLK, STAMP1_ADC_SG8.SCLK, STAMP1_ADC_TEMP3.SCLK
- net STAMP6_CS_SG1: now also STAMP1_ADC_SG15.!CS
- net STAMP6_CS_SG2: now also STAMP1_ADC_SG16.!CS
- net STAMP6_CS_TEMP: now also STAMP1_ADC_TEMP7.!CS
- net STAMP6_DRDY_SG1: now also STAMP1_ADC_SG15.!DRDY
- net STAMP6_DRDY_SG2: now also STAMP1_ADC_SG16.!DRDY
- net STAMP6_DRDY_TEMP: now also STAMP1_ADC_TEMP7.!DRDY
- net STAMP6_MISO: now also R178.1, R184.1, R188.1
- net STAMP6_MOSI: now also STAMP1_ADC_SG15.DIN, STAMP1_ADC_SG16.DIN, STAMP1_ADC_TEMP7.DIN
- net STAMP6_SCLK: now also STAMP1_ADC_SG15.SCLK, STAMP1_ADC_SG16.SCLK, STAMP1_ADC_TEMP7.SCLK
- net WP: now also S70FL.WP#/IO2; no longer U$4.WP#/IO2
Other:
- note added: "STAMP 1"
