File: SPU.sch (EAGLE design)
At the start: 396 parts, among them Q2 CSTCR6M00G53Z

Commit message: Adds suggestions
Other:
- note added: "STAMP 2"
- note added: "STAMP 3"
- note added: "STAMP 4"
- note added: "STAMP 5"
- note added: "STAMP 6"
Changed lines of the file:
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@@
 <description>STAMP 2</description>
 <plain>
+<text x="165.1" y="238.76" size="6.4516" layer="94">STAMP 2</text>
 </plain>
 <instances>
@@
 <description>STAMP 3</description>
 <plain>
+<text x="162.56" y="238.76" size="6.4516" layer="94">STAMP 3</text>
 </plain>
 <instances>
@@
 <description>STAMP 4</description>
 <plain>
+<text x="162.56" y="236.22" size="6.4516" layer="94">STAMP 4</text>
 </plain>
 <instances>
@@
 <description>STAMP 5</description>
 <plain>
+<text x="165.1" y="236.22" size="6.4516" layer="94">STAMP 5</text>
 </plain>
 <instances>
@@
 <description>STAMP 6</description>
 <plain>
+<text x="162.56" y="236.22" size="6.4516" layer="94">STAMP 6</text>
 </plain>
 <instances>

Commit message: Improves labelling
Parts:
- removed CON_STAMP8: IL-AG5-10P-S3T2, con-jae:IL-AG5-10P-S3T2
- added CON_STAMP2: IL-AG5-10P-S3T2, con-jae:IL-AG5-10P-S3T2
Connections:
- net GND: now also CON_STAMP2.P$7; no longer CON_STAMP8.P$7
- net STAMP2_SG1_AIN1: now also CON_STAMP2.P$1; no longer CON_STAMP3.P$1
- net STAMP2_SG1_AIN2: now also CON_STAMP2.P$2; no longer CON_STAMP3.P$2
- net STAMP2_SG1_AIN3: now also CON_STAMP2.P$3; no longer CON_STAMP3.P$3
- net STAMP2_SG2_AIN1: now also CON_STAMP2.P$10; no longer CON_STAMP3.P$10
- net STAMP2_SG2_AIN2: now also CON_STAMP2.P$9; no longer CON_STAMP3.P$9
- net STAMP2_SG2_AIN3: now also CON_STAMP2.P$8; no longer CON_STAMP3.P$8
- net STAMP2_TEMP_AIN1: now also CON_STAMP2.P$4; no longer CON_STAMP3.P$4
- net STAMP2_TEMP_AIN2: now also CON_STAMP2.P$5; no longer CON_STAMP3.P$5
- net STAMP2_TEMP_AIN3: now also CON_STAMP2.P$6; no longer CON_STAMP3.P$6
- net STAMP3_SG1_AIN1: now also CON_STAMP3.P$1; no longer CON_STAMP5.P$1
- net STAMP3_SG1_AIN2: now also CON_STAMP3.P$2; no longer CON_STAMP5.P$2
- net STAMP3_SG1_AIN3: now also CON_STAMP3.P$3; no longer CON_STAMP5.P$3
- net STAMP3_SG2_AIN1: now also CON_STAMP3.P$10; no longer CON_STAMP5.P$10
- net STAMP3_SG2_AIN2: now also CON_STAMP3.P$9; no longer CON_STAMP5.P$9
- net STAMP3_SG2_AIN3: now also CON_STAMP3.P$8; no longer CON_STAMP5.P$8
- net STAMP3_TEMP_AIN1: now also CON_STAMP3.P$4; no longer CON_STAMP5.P$4
- net STAMP3_TEMP_AIN2: now also CON_STAMP3.P$5; no longer CON_STAMP5.P$5
- net STAMP3_TEMP_AIN3: now also CON_STAMP3.P$6; no longer CON_STAMP5.P$6
- net STAMP4_SG1_AIN1: now also CON_STAMP4.P$1; no longer CON_STAMP6.P$1
- net STAMP4_SG1_AIN2: now also CON_STAMP4.P$2; no longer CON_STAMP6.P$2
- net STAMP4_SG1_AIN3: now also CON_STAMP4.P$3; no longer CON_STAMP6.P$3
- net STAMP4_SG2_AIN1: now also CON_STAMP4.P$10; no longer CON_STAMP6.P$10
- net STAMP4_SG2_AIN2: now also CON_STAMP4.P$9; no longer CON_STAMP6.P$9
- net STAMP4_SG2_AIN3: now also CON_STAMP4.P$8; no longer CON_STAMP6.P$8
- net STAMP4_TEMP_AIN1: now also CON_STAMP4.P$4; no longer CON_STAMP6.P$4
- net STAMP4_TEMP_AIN2: now also CON_STAMP4.P$5; no longer CON_STAMP6.P$5
- net STAMP4_TEMP_AIN3: now also CON_STAMP4.P$6; no longer CON_STAMP6.P$6
- net STAMP5_SG1_AIN1: now also CON_STAMP5.P$1; no longer CON_STAMP4.P$1
- net STAMP5_SG1_AIN2: now also CON_STAMP5.P$2; no longer CON_STAMP4.P$2
- net STAMP5_SG1_AIN3: now also CON_STAMP5.P$3; no longer CON_STAMP4.P$3
- net STAMP5_SG2_AIN1: now also CON_STAMP5.P$10; no longer CON_STAMP4.P$10
- net STAMP5_SG2_AIN2: now also CON_STAMP5.P$9; no longer CON_STAMP4.P$9
- net STAMP5_SG2_AIN3: now also CON_STAMP5.P$8; no longer CON_STAMP4.P$8
- net STAMP5_TEMP_AIN1: now also CON_STAMP5.P$4; no longer CON_STAMP4.P$4
- net STAMP5_TEMP_AIN2: now also CON_STAMP5.P$5; no longer CON_STAMP4.P$5
- net STAMP5_TEMP_AIN3: now also CON_STAMP5.P$6; no longer CON_STAMP4.P$6
- net STAMP6_SG1_AIN1: now also CON_STAMP6.P$1; no longer CON_STAMP8.P$1
- net STAMP6_SG1_AIN2: now also CON_STAMP6.P$2; no longer CON_STAMP8.P$2
- net STAMP6_SG1_AIN3: now also CON_STAMP6.P$3; no longer CON_STAMP8.P$3
- net STAMP6_SG2_AIN1: now also CON_STAMP6.P$10; no longer CON_STAMP8.P$10
- net STAMP6_SG2_AIN2: now also CON_STAMP6.P$9; no longer CON_STAMP8.P$9
- net STAMP6_SG2_AIN3: now also CON_STAMP6.P$8; no longer CON_STAMP8.P$8
- net STAMP6_TEMP_AIN1: now also CON_STAMP6.P$4; no longer CON_STAMP8.P$4
- net STAMP6_TEMP_AIN2: now also CON_STAMP6.P$5; no longer CON_STAMP8.P$5
- net STAMP6_TEMP_AIN3: now also CON_STAMP6.P$6; no longer CON_STAMP8.P$6

Commit message: Updates schematics
Parts:
- removed FTDI: FT2232D, smf2:FT2232D
- removed LED6, LED7, LED8: 1V9, adafruit:LEDCHIP-LED0805
- removed R5: 4k7, rcl:R-EU_R0805
- removed R6, R8: 27, rcl:R-EU_R0805
- removed R64, R65: inf, rcl:R-EU_R0805
- removed R66: inf, rcl:R-TRIMM3224X
- removed R7: 1k5, rcl:R-EU_R0805
- removed RN10: 330, resistor-dil:4R-NEXBS8V
- removed U_LT1: LT1528, aSparkFun:LT1528
- added C71, C72, C73: 100n, rcl:C-EUC0805
- added C74, C75: 22p, rcl:C-EUC0805
- added L1, L2: (no value), rcl:L-EUL1812
- added Q1, Q3, Q4, Q5, Q6: BSS123, transistor-small-signal:BSS123
- added R34, R43, R44, R53, R57: 1k, rcl:R-EU_R0805
- added R37, R38, R39, R42: 600, rcl:R-EU_R0805
- added R47, R48: 330, rcl:R-EU_R0805
- added R49, R52: 680, rcl:R-EU_R0805
- added R54: 3R65, rcl:R-EU_R0805
- added REF4V096: LM4030, selfmade:LM4030
- added SF2_M2S010TQ2: SF2_M2S010TQ144, smf2:SF2_M2S010TQ144
- added TPS78512QKVURQ1: TPS785, selfmade:TPS785
- added U$1, U$2, U$3: NXB0108PWJ, selfmade:NXB0108PWJ
- added USB: FT2232HL, smf2:FT2232HL
- added ZE05H-4P-2V: ZE05-4P-2V, con-hirose:ZE05-4P-2V
- C24, C26: value 100n -> 4u7
- C27: value 100n -> 150n
- C3, C5: value 4.7u -> 4u7
- C30, C31, C32: value 10u -> 100n; device rcl:CPOL-EUE/7260-38W -> rcl:C-EUC0805
- Q2: value CSTCR6M00G53Z -> 12MHz; device murata-filter:CSTCR6M00G53Z -> adafruit:CRYSTALHC49UP
- R19: value 330 -> 680
- R20: value 4k7 -> 680
- R21: value 470 -> 1k
- R22: value 2k -> 1k
- R4: value 10k -> 2
- R9: value 470 -> 12k
- X1: device con-subd:F15HP -> con-subd:M15H
Connections:
- removed net 5V-28V: C43.1, R16.1, R21.2, R25.2, U_7805.VOUT, U_MAX488P.VCC
- removed net HB_MSS: RN10C.1, SF2_M2S010TQ1G$6.MSIO76PB7
- removed net HB_STAMPS: RN10A.1, SF2_M2S010TQ1G$6.MSIO77PB7
- removed net HB_STORAGE: RN10B.1, SF2_M2S010TQ1G$6.MSIO77NB7
- removed net LED4: RN10D.1, SF2_M2S010TQ1G$6.MSIO76NB7
- removed net USB_N: CN1.D-, R8.2
- removed net USB_P: CN1.D+, R6.2
- removed net VCCINT: C10.1, C11.1, C12.1, C13.1, C14.1, C29.2, C31.+, C32.+, C7.1, C8.1, C9.1, SF2_M2S010TQ1G$7.VDD, U_LT1.OUT, U_LT1.SENSE
- new net 1V2: C10.1, C11.1, C12.1, C13.1, C14.1, C29.1, C7.1, C8.1, C9.1, R37.1, R38.1, R39.1, R42.1, SF2_M2S010TQ2G$7.VDD, SF2_M2S010TQ2G$7.VDDI0, SF2_M2S010TQ2G$7.VDDI6, TPS78512QKVURQ1.OUT, U$1.OE, U$1.VCCA, U$2.OE, U$2.VCCA, U$3.OE, U$3.VCCA
- new net 4V096: R105.2, R111.2, R124.2, R130.2, R143.2, R149.2, R181.2, R187.2, R33.2, R54.1, R74.2, R86.2, R92.2, REF4V096.C, U$10.5, U$11.5, U$12.5, U$13.5, U$14.5, U$15.5, U$16.5, U$19.5, U$20.5, U$6.5, U$7.5, U$9.5
- new net 5V-NONISO: C43.1, R16.1, R25.2, U_7805.VOUT, U_MAX488P.VCC
- new net ACD_START_1V2: U$3.A7
- new net ADC_START_1V2: SF2_M2S010TQ1G$1.DDRIO47NB0
- new net LED_FPGA_LOADED: Q3.G, R44.2, SF2_M2S010TQ1G$5.MSIOD84PB6/CCC_NE1_CLKI2
- new net LED_HB_MEMSYNC: Q6.G, R53.2, SF2_M2S010TQ1G$5.MSIOD90PB6
- new net LED_HB_MSS: Q5.G, R34.2, SF2_M2S010TQ1G$5.MSIOD85PB6/CCC_NE1_CLKI1
- new net LED_RECORDING: Q4.G, R21.2, SF2_M2S010TQ1G$5.MSIOD90NB6
- new net N$175: LED3.A, R49.2
- new net N$176: R47.2, ZE05H-4P-2V.P$4
- new net N$177: LED3.C, Q4.D
- new net N$178: R48.2, ZE05H-4P-2V.P$2
- new net N$179: C30.2, USB.VCORE@1, USB.VCORE@2, USB.VCORE@3, USB.VREGOUT
- new net N$180: C25.2, C26.2, L2.2, USB.VPLL
- new net N$28: R35.2, U$1.B2
- new net N$36: SF2_M2S010TQ1G$1.DDRIO37PB0, U$2.A2
- new net N$42: SF2_M2S010TQ1G$1.DDRIO43NB0, U$2.A1
- new net N$44: Q1.D, U_OPTO_4.C1
- new net N$53: SF2_M2S010TQ1G$1.DDRIO48PB0, U$1.A3
- new net N$54: SF2_M2S010TQ1G$1.DDRIO53NB0, U$1.A4
- new net N$57: SF2_M2S010TQ1G$1.DDRIO55PB0/CCC_NE0_CLKI3, U$1.A7
- new net N$58: SF2_M2S010TQ1G$1.DDRIO59NB0/GB4, U$1.A8
- new net N$59: SF2_M2S010TQ1G$5.MSIOD99NB6, U$3.A5
- new net N$60: SF2_M2S010TQ1G$1.DDRIO29PB0, U$2.A8
- new net N$61: SF2_M2S010TQ1G$1.DDRIO30PB0, U$2.A7
- new net N$62: SF2_M2S010TQ1G$1.DDRIO30NB0, U$2.A6
- new net N$63: SF2_M2S010TQ1G$1.DDRIO35NB0, U$2.A5
- new net N$66: SF2_M2S010TQ1G$1.DDRIO35PB0, U$2.A4
- new net N$67: SF2_M2S010TQ1G$1.DDRIO37NB0, U$2.A3
- new net N$68: SF2_M2S010TQ1G$5.MSIOD93PB6, U$3.A6
- new net N$71: R60.1, SF2_M2S010TQ1G$6.MSIO64NB7
- new net N$72: R61.1, SF2_M2S010TQ1G$6.MSIO64PB7
- new net N$73: R57.2, USB.NRESET
- new net N$76: C27.1, R4.1, SF2_M2S010TQ2G$7.XTLOSC_AUX_EXTAL
- new net N$77: LED5.A, R52.2
- new net STAMP1_CS_TEMP_1V2: SF2_M2S010TQ1G$1.DDRIO60NB0/CCC_NE1_CLKI3, U$3.A8
- net 28V: no longer R20.2
- net 28VGND: now also U_OPTO_4.EMT2; no longer LED7.C, LED8.C
- net 3V3: now also C28.2, C31.2, C32.2, C71.2, C72.2, C73.2, L1.1, L2.1, R22.2, R4.2, R57.1, SF2_M2S010TQ2G$7.VDDI2, SF2_M2S010TQ2G$7.VDDI3, SF2_M2S010TQ2G$7.VDDI4, SF2_M2S010TQ2G$7.VDDI7, SF2_M2S010TQ2G$7.VPP, SF2_M2S010TQ2G$7.VPPNVM, SF2_M2S010TQ2G$7.XTLOSC_AUX_XTAL, TPS78512QKVURQ1.EN, TPS78512QKVURQ1.IN, U$1.VCCB, U$2.VCCB, U$3.VCCB, USB.VCCIO@1, USB.VCCIO@2, USB.VCCIO@3, USB.VCCIO@4, USB.VREGIN; no longer C24.2, C25.2, C26.2, C27.2, FTDI.VCC, FTDI.VCC1, FTDI.VCCIOB, FTDI.VVCIOA, R105.2, R111.2, R124.2, R130.2, R143.2, R149.2, R181.2, R187.2, R19.2, R33.2, R74.2, R86.2, R9.1, R92.2, SF2_M2S010TQ1G$3.JTAG_TRSTB/M3_TRSTB, SF2_M2S010TQ1G$7.VDDI0, SF2_M2S010TQ1G$7.VDDI2, SF2_M2S010TQ1G$7.VDDI3, SF2_M2S010TQ1G$7.VDDI4, SF2_M2S010TQ1G$7.VDDI6, SF2_M2S010TQ1G$7.VDDI7, SF2_M2S010TQ1G$7.VPP, SF2_M2S010TQ1G$7.VPPNVM, U$10.5, U$11.5, U$12.5, U$13.5, U$14.5, U$15.5, U$16.5, U$19.5, U$20.5, U$6.5, U$7.5, U$9.5
- net 5V: now also R18.1, R19.1, R20.1, R47.1, R48.1, R49.1, R52.1, R54.2; no longer C28.2, C30.+, R18.2, R65.1, R66.E, U_LT1.IN, U_LT1.SHDN
- net ADC_START: now also U$3.B7; no longer SF2_M2S010TQ1G$1.DDRIO47NB0
- net DAPI_CTS: now also U$2.B6, USB.BDBUS2; no longer FTDI.BDBUS2, SF2_M2S010TQ1G$1.DDRIO30NB0
- net DAPI_DSR: now also U$2.B4, USB.BDBUS4; no longer FTDI.BDBUS4, SF2_M2S010TQ1G$1.DDRIO35PB0
- net DAPI_DTR: now also U$2.B3, USB.BDBUS5; no longer FTDI.BDBUS5, SF2_M2S010TQ1G$1.DDRIO37NB0
- net DAPI_RTS: now also U$2.B5, USB.BDBUS3; no longer FTDI.BDBUS3, SF2_M2S010TQ1G$1.DDRIO35NB0
- net DAPI_RXD: now also U$2.B8, USB.BDBUS0; no longer FTDI.BDBUS0, SF2_M2S010TQ1G$1.DDRIO29PB0
- net DAPI_TXD: now also U$2.B7, USB.BDBUS1; no longer FTDI.BDBUS1, SF2_M2S010TQ1G$1.DDRIO30PB0
- net EECLK: now also USB.EECLK; no longer FTDI.EESK
- net EECS: now also USB.EECS; no longer FTDI.EECS
- net EED: now also USB.EEDATA; no longer FTDI.EEDATA
- net GND: now also C22.2, C24.2, C27.2, C29.2, C30.1, C31.1, C32.1, C71.1, C72.1, C73.1, C74.2, C75.2, Q1.S, Q3.S, Q4.S, Q5.S, Q6.S, R21.1, R34.1, R43.2, R44.1, R53.1, R9.1, REF4V096.A, SF2_M2S010TQ2G$7.VSS, SF2_M2S010TQ2G$7.VSSNVM, TPS78512QKVURQ1.GND, U$1.GND, U$2.GND, U$3.GND, USB.AGND, USB.GND@1, USB.GND@2, USB.GND@3, USB.GND@4, USB.GND@5, USB.GND@6, USB.GND@7, USB.GND@8, USB.TEST, ZE05H-4P-2V.P$1, ZE05H-4P-2V.P$3, ZE05H-4P-2V.P$5; no longer C22.1, C24.1, C27.1, C29.1, C30.-, C31.-, C32.-, FTDI.AGND, FTDI.GND1, FTDI.GND2, FTDI.GND3, FTDI.GND4, FTDI.TEST, LED2.C, LED3.C, LED4.C, LED5.C, LED6.C, Q2.2, R22.2, R4.1, R64.1, R66.A, SF2_M2S010TQ1G$7.VSS, SF2_M2S010TQ1G$7.VSSNVM, U_LT1.GND, U_OPTO_4.EMT2
- net LO: now also R38.2, SF2_M2S010TQ1G$1.DDRIO44PB0; no longer SF2_M2S010TQ1G$1.DDRIO43PB0
- net N$11: now also C74.1, Q2.2, USB.OSCI; no longer FTDI.USBDM, R8.1
- net N$12: now also SF2_M2S010TQ1G$5.MSIOD96PB6, U$3.A1; no longer FTDI.XTIN, Q2.1
- net N$13: now also SF2_M2S010TQ1G$5.MSIOD96NB6, U$3.A2; no longer C21.2, FTDI.3V3OUT
- net N$14: now also SF2_M2S010TQ1G$5.MSIOD98NB6, U$3.A3; no longer C22.2, FTDI.AVCC, R9.2
- net N$15: now also C21.2, CN1.VBUS; no longer FTDI.RESET#, R4.2, R5.1
- net N$16: now also C22.1, C24.1, L1.2, USB.VPHY; no longer CN1.VBUS, R5.2
- net N$17: now also R36.2, U$1.B1; no longer R64.2, R65.2, R66.S, U_TRACODCDC.TRIM
- net N$18: now also USB.ADBUS0; no longer FTDI.ADBUS0
- net N$19: now also USB.ADBUS1; no longer FTDI.ADBUS1
- net N$2: now also SF2_M2S010TQ2G$7.DEVRST_N; no longer SF2_M2S010TQ1G$7.DEVRST_N
- net N$20: now also USB.ADBUS2; no longer FTDI.ADBUS2
- net N$21: now also USB.ADBUS3; no longer FTDI.ADBUS3
- net N$22: now also SF2_M2S010TQ1G$5.MSIOD99PB6, U$3.A4; no longer FTDI.XTOUT, Q2.3
- net N$27: now also U_OPTO_4.A1; no longer U_OPTO_4.C1
- net N$30: now also R18.2; no longer RN10A.2
- net N$31: now also LED5.C, Q6.D; no longer LED2.A, RN10B.2
- net N$32: now also LED4.C, Q5.D; no longer LED3.A, RN10C.2
- net N$33: now also LED2.C, Q3.D; no longer LED4.A, RN10D.2
- net N$4: now also SF2_M2S010TQ2G$7.CCC_NE1_PLL_VSSA; no longer SF2_M2S010TQ1G$7.CCC_NE1_PLL_VSSA
- net N$45: now also LED2.A, R19.2; no longer R35.2, SF2_M2S010TQ1G$1.DDRIO48NB0
- net N$46: now also R40.1, U$2.B2; no longer R40.2, SF2_M2S010TQ1G$1.DDRIO59PB0/GB0
- net N$47: now also U$1.A1; no longer R36.2
- net N$48: now also R41.1, U$2.B1; no longer R41.2, SF2_M2S010TQ1G$1.DDRIO63PB0
- net N$5: now also SF2_M2S010TQ2G$7.CCC_NE1_PLL_VDDA; no longer SF2_M2S010TQ1G$7.CCC_NE1_PLL_VDDA
- net N$51: now also LED4.A, R20.2; no longer LED5.A, R18.1
- net N$52: now also SF2_M2S010TQ1G$1.DDRIO48NB0, U$1.A2; no longer LED6.A, R19.1
- net N$55: now also SF2_M2S010TQ1G$1.DDRIO53PB0, U$1.A5; no longer LED7.A, R20.1
- net N$56: now also SF2_M2S010TQ1G$1.DDRIO55NB0, U$1.A6; no longer LED8.A, R21.1
- net N$6: now also SF2_M2S010TQ2G$7.CCC_NE0_PLL_VDDA; no longer SF2_M2S010TQ1G$7.CCC_NE0_PLL_VDDA
- net N$7: now also SF2_M2S010TQ2G$7.CCC_NE0_PLL_VSSA; no longer SF2_M2S010TQ1G$7.CCC_NE0_PLL_VSSA
- net N$74: now also R9.2, USB.REF; no longer R60.2, SF2_M2S010TQ1G$5.MSIOD96NB6
- net N$75: now also C75.1, Q2.1, USB.OSCO; no longer R61.2, SF2_M2S010TQ1G$5.MSIOD98NB6
- net N$8: now also CN1.D-, USB.DM; no longer FTDI.RSTOUT#, R7.1
- net N$9: now also CN1.D+, USB.DP; no longer FTDI.USBDP, R6.1, R7.2
- net SODS: now also R37.2
- net SOE: now also R39.2, SF2_M2S010TQ1G$1.DDRIO43PB0; no longer SF2_M2S010TQ1G$1.DDRIO44PB0
- net STAMP1_CS_SG1: now also U$1.B7; no longer SF2_M2S010TQ1G$1.DDRIO55PB0/CCC_NE0_CLKI3
- net STAMP1_CS_SG2: now also U$1.B8; no longer SF2_M2S010TQ1G$1.DDRIO59NB0/GB4
- net STAMP1_CS_TEMP: now also U$3.B8; no longer SF2_M2S010TQ1G$1.DDRIO60NB0/CCC_NE1_CLKI3
- net STAMP1_DRDY_SG1: now also U$1.B4; no longer SF2_M2S010TQ1G$1.DDRIO53NB0
- net STAMP1_DRDY_SG2: now also U$1.B5; no longer SF2_M2S010TQ1G$1.DDRIO53PB0
- net STAMP1_DRDY_TEMP: now also U$1.B6; no longer SF2_M2S010TQ1G$1.DDRIO55NB0
- net STAMP1_MISO: now also U$1.B3; no longer SF2_M2S010TQ1G$1.DDRIO48PB0
- net STAMP2_MOSI: now also R41.2; no longer R41.1
- net STAMP2_SCLK: now also R40.2; no longer R40.1
- net STAMP5_CS_SG1: now also U$3.B5; no longer SF2_M2S010TQ1G$5.MSIOD93NB6
- net STAMP5_CS_SG2: now also SF2_M2S010TQ1G$6.MSIO76NB7; no longer SF2_M2S010TQ1G$5.MSIOD93PB6
- net STAMP5_CS_TEMP: now also SF2_M2S010TQ1G$6.MSIO76PB7; no longer SF2_M2S010TQ1G$5.MSIOD96PB6
- net STAMP5_DRDY_SG1: now also U$3.B2; no longer SF2_M2S010TQ1G$5.MSIOD85PB6/CCC_NE1_CLKI1
- net STAMP5_DRDY_SG2: now also U$3.B3; no longer SF2_M2S010TQ1G$5.MSIOD90NB6
- net STAMP5_DRDY_TEMP: now also U$3.B4; no longer SF2_M2S010TQ1G$5.MSIOD90PB6
- net STAMP5_MISO: now also U$3.B1; no longer SF2_M2S010TQ1G$5.MSIOD84PB6/CCC_NE1_CLKI2
- net STAMP6_CS_SG1: now also SF2_M2S010TQ1G$6.MSIO72NB7; no longer SF2_M2S010TQ1G$6.MSIO67NB7
- net STAMP6_CS_SG2: now also SF2_M2S010TQ1G$6.MSIO73NB7; no longer SF2_M2S010TQ1G$6.MSIO67PB7
- net STAMP6_CS_TEMP: now also SF2_M2S010TQ1G$6.MSIO81PB7; no longer SF2_M2S010TQ1G$6.MSIO71NB7
- net STAMP6_DRDY_SG1: now also SF2_M2S010TQ1G$6.MSIO67PB7; no longer SF2_M2S010TQ1G$5.MSIOD99NB6
- net STAMP6_DRDY_SG2: now also SF2_M2S010TQ1G$6.MSIO71NB7; no longer SF2_M2S010TQ1G$6.MSIO64NB7
- net STAMP6_DRDY_TEMP: now also SF2_M2S010TQ1G$6.MSIO71PB7; no longer SF2_M2S010TQ1G$6.MSIO64PB7
- net STAMP6_MISO: now also SF2_M2S010TQ1G$6.MSIO67NB7; no longer SF2_M2S010TQ1G$5.MSIOD99PB6
- net STAMP6_MOSI: now also R61.2; no longer R61.1
- net STAMP6_SCLK: now also R60.2; no longer R60.1
- net TM_RX: now also R42.2, SF2_M2S010TQ1G$1.DDRIO63PB0; no longer SF2_M2S010TQ1G$1.DDRIO37PB0
- net TM_TX: now also Q1.G, R43.1, SF2_M2S010TQ1G$1.DDRIO59PB0/GB0; no longer SF2_M2S010TQ1G$1.DDRIO43NB0, U_OPTO_4.A1
- net WP: now also U$3.B6; no longer SF2_M2S010TQ1G$6.MSIO71PB7
Other:
- note added: "External LEDs: Dialight 559-2301-003F (Red) Dialight 559-2501-007F (Orange)"
- note added: "RC Network Oscillator: 3,333...MHz = 1 / (2Ohm x 150nF)"
- note added: "ZE05 matching parts: Plug ZE05-4S-HU/R Crimp ZE05-2022SCF"
- moved on the sheet: C21, C22, C23, C24, C25, C26, C28, C29, C42, C43, C44, CN1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

Commit message: Fixes LEDs
Connections:
- removed net N$33: LED2.C, Q3.D
- new net N$181: LED2.C, Q3.D, ZE05H-4P-2V.P$3
- net GND: no longer ZE05H-4P-2V.P$1, ZE05H-4P-2V.P$3
- net N$177: now also ZE05H-4P-2V.P$1

Commit message: Finished Placement
Parts:
- removed C30, C32, C72: 100n, rcl:C-EUC0805
- removed R37, R38, R39: 600, rcl:R-EU_R0805
- removed SF2_M2S010TQ2: SF2_M2S010TQ144, smf2:SF2_M2S010TQ144
- added C76, C77, C78: 100n, rcl:C-EUC0805
- added C79: 4u7, rcl:C-EUC0805
Connections:
- net N$8 renamed USB_N
- net N$9 renamed USB_P
- removed net ACD_START_1V2: U$3.A7
- removed net N$76: C27.1, R4.1, SF2_M2S010TQ2G$7.XTLOSC_AUX_EXTAL
- new net N$33: C27.1, R4.1, SF2_M2S010TQ1G$7.XTLOSC_AUX_EXTAL
- net 1V2: now also SF2_M2S010TQ1G$7.VDD, SF2_M2S010TQ1G$7.VDDI0, SF2_M2S010TQ1G$7.VDDI6; no longer R37.1, R38.1, R39.1, SF2_M2S010TQ2G$7.VDD, SF2_M2S010TQ2G$7.VDDI0, SF2_M2S010TQ2G$7.VDDI6
- net 3V3: now also SF2_M2S010TQ1G$7.VDDI2, SF2_M2S010TQ1G$7.VDDI3, SF2_M2S010TQ1G$7.VDDI4, SF2_M2S010TQ1G$7.VDDI7, SF2_M2S010TQ1G$7.VPP, SF2_M2S010TQ1G$7.VPPNVM, SF2_M2S010TQ1G$7.XTLOSC_AUX_XTAL; no longer C32.2, C72.2, SF2_M2S010TQ2G$7.VDDI2, SF2_M2S010TQ2G$7.VDDI3, SF2_M2S010TQ2G$7.VDDI4, SF2_M2S010TQ2G$7.VDDI7, SF2_M2S010TQ2G$7.VPP, SF2_M2S010TQ2G$7.VPPNVM, SF2_M2S010TQ2G$7.XTLOSC_AUX_XTAL
- net ADC_START_1V2: now also U$3.A7
- net GND: now also C76.1, C77.1, C78.1, C79.1, SF2_M2S010TQ1G$7.VSS, SF2_M2S010TQ1G$7.VSSNVM; no longer C30.1, C32.1, C72.1, SF2_M2S010TQ2G$7.VSS, SF2_M2S010TQ2G$7.VSSNVM
- net LO: no longer R38.2
- net N$179: now also C76.2, C77.2, C78.2, C79.2; no longer C30.2
- net N$2: now also SF2_M2S010TQ1G$7.DEVRST_N; no longer SF2_M2S010TQ2G$7.DEVRST_N
- net N$4: now also SF2_M2S010TQ1G$7.CCC_NE1_PLL_VSSA; no longer SF2_M2S010TQ2G$7.CCC_NE1_PLL_VSSA
- net N$5: now also SF2_M2S010TQ1G$7.CCC_NE1_PLL_VDDA; no longer SF2_M2S010TQ2G$7.CCC_NE1_PLL_VDDA
- net N$6: now also SF2_M2S010TQ1G$7.CCC_NE0_PLL_VDDA; no longer SF2_M2S010TQ2G$7.CCC_NE0_PLL_VDDA
- net N$7: now also SF2_M2S010TQ1G$7.CCC_NE0_PLL_VSSA; no longer SF2_M2S010TQ2G$7.CCC_NE0_PLL_VSSA
- net SODS: no longer R37.2
- net SOE: no longer R39.2
Other:
- note added: "RC Network: 3,33...MHz = 1 / (2Ohm * 150nF)"
- note removed: "RC Network Oscillator: 3,333...MHz = 1 / (2Ohm x 150nF)"
- moved on the sheet: C71

Commit message: During work commit
Parts:
- renumbered CN1 to USB_CONN
Changed lines of the file:
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@@
 <part name="R61" library="rcl" library_urn="urn:adsk.eagle:library:334" deviceset="R-EU_" device="R0805" package3d_urn="urn:adsk.eagle:package:23553/2" value="47"/>
 <part name="FRAME2" library="frames" library_urn="urn:adsk.eagle:library:229" deviceset="A3L-LOC" device=""/>
-<part name="CN1" library="adafruit" library_urn="urn:adsk.eagle:library:420" deviceset="USB" device="MINIB" package3d_urn="urn:adsk.eagle:package:6240633/1"/>
+<part name="USB_CONN" library="adafruit" library_urn="urn:adsk.eagle:library:420" deviceset="USB" device="MINIB" package3d_urn="urn:adsk.eagle:package:6240633/1"/>
 <part name="R24" library="rcl" library_urn="urn:adsk.eagle:library:334" deviceset="R-EU_" device="R0805" package3d_urn="urn:adsk.eagle:package:23553/2" value="2k2"/>
 <part name="STAMP1_ADC_SG1" library="ads11xx" deviceset="ADS1148QPWRQ1" device="" package3d_urn="urn:adsk.eagle:package:17526348/1"/>
@@
 <attribute name="VALUE" x="57.912" y="33.528" size="1.778" layer="96" rot="MR0"/>
 </instance>
-<instance part="CN1" gate="G$1" x="210.82" y="111.76" smashed="yes" grouprefs="DAPI">
+<instance part="USB_CONN" gate="G$1" x="210.82" y="111.76" smashed="yes" grouprefs="DAPI">
 <attribute name="NAME" x="200.66" y="120.396" size="1.27" layer="95"/>
 <attribute name="VALUE" x="200.66" y="101.6" size="1.27" layer="96"/>
@@
 </segment>
 <segment>
-<pinref part="CN1" gate="G$1" pin="GND"/>
+<pinref part="USB_CONN" gate="G$1" pin="GND"/>
 <wire x1="220.98" y1="106.68" x2="223.52" y2="106.68" width="0.1524" layer="91" grouprefs="DAPI"/>
 <label x="223.52" y="106.68" size="1.27" layer="95" xref="yes" grouprefs="DAPI"/>
@@
 <net name="USB_N" class="0">
 <segment>
-<pinref part="CN1" gate="G$1" pin="D-"/>
+<pinref part="USB_CONN" gate="G$1" pin="D-"/>
 <wire x1="220.98" y1="111.76" x2="236.22" y2="111.76" width="0.1524" layer="91" grouprefs="DAPI"/>
 <wire x1="236.22" y1="111.76" x2="236.22" y2="114.3" width="0.1524" layer="91" grouprefs="DAPI"/>
@@
 <net name="USB_P" class="0">
 <segment>
-<pinref part="CN1" gate="G$1" pin="D+"/>
+<pinref part="USB_CONN" gate="G$1" pin="D+"/>
 <wire x1="220.98" y1="114.3" x2="233.68" y2="114.3" width="0.1524" layer="91" grouprefs="DAPI"/>
 <wire x1="233.68" y1="114.3" x2="233.68" y2="109.22" width="0.1524" layer="91" grouprefs="DAPI"/>
@@
 <net name="N$15" class="0">
 <segment>
-<pinref part="CN1" gate="G$1" pin="VBUS"/>
+<pinref part="USB_CONN" gate="G$1" pin="VBUS"/>
 <pinref part="C21" gate="G$1" pin="2"/>
 <wire x1="220.98" y1="116.84" x2="223.52" y2="116.84" width="0.1524" layer="91" grouprefs="DAPI"/>

Commit message: Schematic: changed names from STAMP2 - STMAP6 to STAMPN_ADC_SG/TEMP Bord: Adding names for more readabilty.
Parts:
- renumbered STAMP1_ADC_SG10 to STAMP3_ADC_SG2, STAMP1_ADC_SG11 to STAMP4_ADC_SG1, STAMP1_ADC_SG12 to STAMP4_ADC_SG2, STAMP1_ADC_SG15 to STAMP6_ADC_SG1, STAMP1_ADC_SG16 to STAMP6_ADC_SG2, STAMP1_ADC_SG5 to STAMP2_ADC_SG1, STAMP1_ADC_SG6 to STAMP2_ADC_SG2, STAMP1_ADC_SG7 to STAMP5_ADC_SG1, STAMP1_ADC_SG8 to STAMP5_ADC_SG2, STAMP1_ADC_SG9 to STAMP3_ADC_SG1, STAMP1_ADC_TEMP2 to STAMP2_ADC_TEMP, STAMP1_ADC_TEMP3 to STAMP5_ADC_TEMP, STAMP1_ADC_TEMP4 to STAMP3_ADC_TEMP, STAMP1_ADC_TEMP5 to STAMP4_ADC_TEMP, STAMP1_ADC_TEMP7 to STAMP6_ADC_TEMP
Connections:
- net STAMP2_TEMP_AIN1 renamed SMASHALL
