File: SPU.brd (EAGLE design)
At the start: 127.6 x 101.6 mm, 261 parts, among them Q1 12MHz

Commit message: Almost final sch
Parts:
- removed C28, C29, C30, C31, C32, C33, C75: 100n, rcl:C0805
- removed C45, C46, C47, C48, C50, C51, C53, C54, C55, C57, C58, C59, C_AVDD_PT1, C_AVDD_PT2, C_AVDD_PT3, C_DVDD_PT1, C_DVDD_PT2, C_DVDD_PT3, C_RDIFF_PT3: 100n, rcl:C0603
- removed C49, C56: 1u, rcl:C1206
- removed C52, C74: 10n, rcl:C0805
- removed C68, C69, C70, C71, C72, C73: 10u, rcl:E/7260-38W
- removed C76: 100n, aSparkFun:0603-CAP
- removed C77, C78: 100n, rcl:C1206
- removed C_ICM1_PT1, C_ICM1_PT2, C_ICM2_PT1, C_ICM2_PT2, C_IDIFF_PT1, C_IDIFF_PT2, C_RCM1_PT1, C_RCM1_PT2, C_RCM1_PT3, C_RCM2_PT1, C_RCM2_PT2, C_RCM2_PT3, C_RDIFF_PT1, C_RDIFF_PT2: (no value), rcl:C0603
- removed C_ICM1_PT3, C_ICM2_PT3: 4n7, rcl:C0603
- removed C_IDIFF_PT3: 47n, rcl:C0603
- removed C_VREF_PT1, C_VREF_PT2, C_VREF_PT3: 1u, rcl:C0603
- removed D10, D11, D12, D3, D4, D7, D8, D9: 3V6, diodes:DMELF
- removed D2, D6: 5V6, diodes:DMELF
- removed JP1: JUMPER-SMT_2_NC_PASTE_SILK, SparkFun-Jumpers:SMT-JUMPER_2_NC_PASTE_SILK
- removed JP_MS: x, aSparkFun:1X02
- removed Q1: 12MHz, adafruit:SM49
- removed R24: ?, rcl:R0805
- removed R28: 99M, rcl:R0805
- removed R29: 10k, rcl:R0805
- removed R30: 4k7, ++Bedrahtet:R0603
- removed R31: 47, ++Bedrahtet:R0603
- removed R32, R33: 40 1%, ++Bedrahtet:R0805
- removed RN11: 3k, resistor-dil:EXBS8V
- removed RN12: 1k, resistor-dil:EXBS8V
- removed RN_A_PT1, RN_A_PT2, RN_A_PT3, RN_B_PT1, RN_B_PT2, RN_B_PT3, RN_DMS1, RN_DMS2, RN_DMS3, RN_DMS4, RN_DMS5, RN_DMS6: 47, resistor-dil:0603-ARC
- removed R_I1_PT1, R_I1_PT2, R_I2_PT1, R_I2_PT2, R_R1_PT1, R_R1_PT2, R_R2_PT1, R_R2_PT2, R_REF_PT1, R_REF_PT2: (no value), ++Bedrahtet:R0603
- removed R_I1_PT3, R_I2_PT3: 5k, ++Bedrahtet:R0603
- removed R_R1_PT3: 3k16, ++Bedrahtet:R0603
- removed R_R2_PT3: inf, ++Bedrahtet:R0603
- removed R_REF_PT3: 1k62, ++Bedrahtet:R0603
- removed SJ_MS: (no value), aSparkFun:SJ_2S-NO
- removed U$6: COMMON_MODE_CHOKE, selfmade:COMMON_MODE_CHOKE
- removed U$7: MICROSD, adafruit:MICROSD
- removed U$8: PLT131PLT131-T1, everlight-fiber-optics-spdif:PLT131-T1
- removed U$9: PLR135, everlight-fiber-optics-spdif:PLR135-T1
- removed U_ADC_DMS1, U_ADC_DMS2, U_ADC_DMS3, U_ADC_DMS4, U_ADC_DMS5, U_ADC_DMS6, U_ADC_PT1, U_ADC_PT2, U_ADC_PT3: ADS1147TSSOP20, ads11xx:TSSOP20
- removed U_ADR366_3: ADR366WAUJZ, ADR360:SOT23-5
- removed U_CH340G: CH340G, ch340g:SOIC16
- removed U_FLASH1, U_FLASH2: S70FL01GS, S70FL01GS:SO16
- removed U_OPTO_1, U_OPTO_2: MOCD207MSOIC-8, Opto-Electronic:SOIC127P594X363-8N
- removed U_STM32F779: STM32F77XXXLQFP208, stm32f:QFP50P3060X3060X385-208
- removed X_DMS, X_GPIO, X_RXSM-DAPI: 403-5X020-5X, con-ept-One27:403-5X020-5X
- removed X_MIRROR, X_MIRROR1: 403-5X026-5X, con-ept-One27:403-5X026-5X
- removed X_PROG: x, con-lstb:MA10-2
- removed X_PT: 403-5X012-5X, con-ept-One27:403-5X012-5X
- added PROBES: (no value), selfmade:PSS254_G3
- added Q2: CSTCR6M00G53Z, murata-filter:CSTCR6M
- added R67, STAMP1:R28, STAMP1:R31, STAMP1:R70, STAMP1:R71, STAMP1:R75, STAMP1:R76, STAMP2:R28, STAMP2:R31, STAMP2:R70, STAMP2:R71, STAMP2:R75, STAMP2:R76, STAMP3:R28, STAMP3:R31, STAMP3:R70, STAMP3:R71, STAMP3:R75, STAMP3:R76, STAMP4:R28, STAMP4:R31, STAMP4:R70, STAMP4:R71, STAMP4:R75, STAMP4:R76, STAMP5:R28, STAMP5:R31, STAMP5:R70, STAMP5:R71, STAMP5:R75, STAMP5:R76, STAMP6:R28, STAMP6:R31, STAMP6:R70, STAMP6:R71, STAMP6:R75, STAMP6:R76: 47, rcl:R0805
- added SF2_M2S010TQ1: SF2_M2S010TQ144, smf2:TQFP144
- added ST1, ST2, ST3, ST4, ST5, STAMP1:ST, STAMP2:ST, STAMP3:ST, STAMP4:ST, STAMP5:ST, STAMP6:ST: LY20-10P-DT1, con-jae-ly:10P-T
- added STAMP1:ADC_SG1, STAMP1:ADC_SG2, STAMP1:ADC_TEMP, STAMP2:ADC_SG1, STAMP2:ADC_SG2, STAMP2:ADC_TEMP, STAMP3:ADC_SG1, STAMP3:ADC_SG2, STAMP3:ADC_TEMP, STAMP4:ADC_SG1, STAMP4:ADC_SG2, STAMP4:ADC_TEMP, STAMP5:ADC_SG1, STAMP5:ADC_SG2, STAMP5:ADC_TEMP, STAMP6:ADC_SG1, STAMP6:ADC_SG2, STAMP6:ADC_TEMP: ADS1148QPWRQ1, ads11xx:TSSOP28
- added STAMP1:C28, STAMP1:C30, STAMP1:C31, STAMP1:C32, STAMP1:C33, STAMP1:C45, STAMP1:C47, STAMP1:C48, STAMP1:C49, STAMP1:C50, STAMP1:C51, STAMP1:C52, STAMP2:C28, STAMP2:C30, STAMP2:C31, STAMP2:C32, STAMP2:C33, STAMP2:C45, STAMP2:C47, STAMP2:C48, STAMP2:C49, STAMP2:C50, STAMP2:C51, STAMP2:C52, STAMP3:C28, STAMP3:C30, STAMP3:C31, STAMP3:C32, STAMP3:C33, STAMP3:C45, STAMP3:C47, STAMP3:C48, STAMP3:C49, STAMP3:C50, STAMP3:C51, STAMP3:C52, STAMP4:C28, STAMP4:C30, STAMP4:C31, STAMP4:C32, STAMP4:C33, STAMP4:C45, STAMP4:C47, STAMP4:C48, STAMP4:C49, STAMP4:C50, STAMP4:C51, STAMP4:C52, STAMP5:C28, STAMP5:C30, STAMP5:C31, STAMP5:C32, STAMP5:C33, STAMP5:C45, STAMP5:C47, STAMP5:C48, STAMP5:C49, STAMP5:C50, STAMP5:C51, STAMP5:C52, STAMP6:C28, STAMP6:C30, STAMP6:C31, STAMP6:C32, STAMP6:C33, STAMP6:C45, STAMP6:C47, STAMP6:C48, STAMP6:C49, STAMP6:C50, STAMP6:C51, STAMP6:C52: 100n, rcl:C0805
- added STAMP1:C29, STAMP1:C46, STAMP1:C56, STAMP2:C29, STAMP2:C46, STAMP2:C56, STAMP3:C29, STAMP3:C46, STAMP3:C56, STAMP4:C29, STAMP4:C46, STAMP4:C56, STAMP5:C29, STAMP5:C46, STAMP5:C56, STAMP6:C29, STAMP6:C46, STAMP6:C56: 1u, rcl:C0805
- added STAMP1:C53, STAMP1:C55, STAMP2:C53, STAMP2:C55, STAMP3:C53, STAMP3:C55, STAMP4:C53, STAMP4:C55, STAMP5:C53, STAMP5:C55, STAMP6:C53, STAMP6:C55: 6n8, rcl:C0805
- added STAMP1:C54, STAMP2:C54, STAMP3:C54, STAMP4:C54, STAMP5:C54, STAMP6:C54: 68n, rcl:C0805
- added STAMP1:C57, STAMP2:C57, STAMP3:C57, STAMP4:C57, STAMP5:C57, STAMP6:C57: 33n, rcl:C0805
- added STAMP1:C58, STAMP1:C59, STAMP2:C58, STAMP2:C59, STAMP3:C58, STAMP3:C59, STAMP4:C58, STAMP4:C59, STAMP5:C58, STAMP5:C59, STAMP6:C58, STAMP6:C59: 3n3, rcl:C0805
- added STAMP1:R24, STAMP1:R68, STAMP1:R77, STAMP2:R24, STAMP2:R68, STAMP2:R77, STAMP3:R24, STAMP3:R68, STAMP3:R77, STAMP4:R24, STAMP4:R68, STAMP4:R77, STAMP5:R24, STAMP5:R68, STAMP5:R77, STAMP6:R24, STAMP6:R68, STAMP6:R77: 4k7, rcl:R0805
- added STAMP1:R29, STAMP1:R32, STAMP1:R72, STAMP1:R73, STAMP2:R29, STAMP2:R32, STAMP2:R72, STAMP2:R73, STAMP3:R29, STAMP3:R32, STAMP3:R72, STAMP3:R73, STAMP4:R29, STAMP4:R32, STAMP4:R72, STAMP4:R73, STAMP5:R29, STAMP5:R32, STAMP5:R72, STAMP5:R73, STAMP6:R29, STAMP6:R32, STAMP6:R72, STAMP6:R73: 40 1%, rcl:R0805
- added STAMP1:R30, STAMP1:R33, STAMP1:R69, STAMP1:R74, STAMP2:R30, STAMP2:R33, STAMP2:R69, STAMP2:R74, STAMP3:R30, STAMP3:R33, STAMP3:R69, STAMP3:R74, STAMP4:R30, STAMP4:R33, STAMP4:R69, STAMP4:R74, STAMP5:R30, STAMP5:R33, STAMP5:R69, STAMP5:R74, STAMP6:R30, STAMP6:R33, STAMP6:R69, STAMP6:R74: 1k 0.1%, rcl:R0805
- added STAMP1:R78, STAMP1:R79, STAMP2:R78, STAMP2:R79, STAMP3:R78, STAMP3:R79, STAMP4:R78, STAMP4:R79, STAMP5:R78, STAMP5:R79, STAMP6:R78, STAMP6:R79: 4k7 1%, rcl:R0805
- added STAMP1:R80, STAMP1:R81, STAMP2:R80, STAMP2:R81, STAMP3:R80, STAMP3:R81, STAMP4:R80, STAMP4:R81, STAMP5:R80, STAMP5:R81, STAMP6:R80, STAMP6:R81: 9k09 1%, rcl:R0805
- added STAMP1:R82, STAMP2:R82, STAMP3:R82, STAMP4:R82, STAMP5:R82, STAMP6:R82: 820 0.1%, rcl:R0805
- added STAMP1:U$6, STAMP1:U$7, STAMP2:U$6, STAMP2:U$7, STAMP3:U$6, STAMP3:U$7, STAMP4:U$6, STAMP4:U$7, STAMP5:U$6, STAMP5:U$7, STAMP6:U$6, STAMP6:U$7: COMMON_MODE_CHOKE, selfmade:COMMON_MODE_CHOKE
- added U_OPTO_4, U_OPTO_5: MOCD207M, Opto-Electronic:SOIC127P594X363-8N
- added WP: (no value), selfmade:PSS254_G2
- C1: value 22p -> 100n; device rcl:C0603 -> rcl:C0805
- C10, C12, C13, C14, C15, C19, C21, C22, C23, C24, C25, C27, C7, C8, C9: device rcl:C0603 -> rcl:C0805
- C11, C20, C26: value 1u -> 100n; device rcl:C1206 -> rcl:C0805
- C16, C17: value 2.2u -> 100n; device rcl:C1206 -> rcl:C0805
- C18: device aSparkFun:0603-CAP -> rcl:C0805
- C2: value 22p -> 10n; device rcl:C0603 -> rcl:C0805
- C3, C5: value 100n -> 4.7u; device rcl:C0603 -> rcl:C0805
- C4: value 1u -> 470n; device rcl:C1206 -> rcl:C0805
- C6: value 100n -> 470n; device rcl:C0603 -> rcl:C0805
- R1: value 4k7 -> 10k; device ++Bedrahtet:R0603 -> rcl:R0805
- R12: value 2k -> 3k
- R13: value 4k7 -> 3k
- R14: value 7k5 -> 47
- R2: value 4k7 -> 2; device ++Bedrahtet:R0603 -> rcl:R0805
- R22: value 100k -> 2k
- R23: value 1k -> 3k
- R25: value ? -> 7k5
- R3: value 47 -> 2; device ++Bedrahtet:R0603 -> rcl:R0805
- R34, R35, R41, R42, R48, R49, R55, R56, R62, R63: value 1k 0.1% -> 47; device ++Bedrahtet:R0805 -> rcl:R0805
- R36, R37, R43, R44, R50, R51, R57, R58: value 4k7 -> 47; device ++Bedrahtet:R0603 -> rcl:R0805
- R38, R45, R52, R59: device ++Bedrahtet:R0603 -> rcl:R0805
- R39, R40, R46, R47, R53, R54, R60, R61: value 40 1% -> 47; device ++Bedrahtet:R0805 -> rcl:R0805
- R4: value 40 1% -> 10k; device ++Bedrahtet:R0805 -> rcl:R0805
- R5: value 40 1% -> 4k7; device ++Bedrahtet:R0805 -> rcl:R0805
- R6: value 1k 0.1% -> 27; device ++Bedrahtet:R0805 -> rcl:R0805
- R7: value 1k 0.1% -> 1k5; device ++Bedrahtet:R0805 -> rcl:R0805
- R8: value 4k7 -> 27; device ++Bedrahtet:R0603 -> rcl:R0805
- R9: value 10k -> 470
- U$1: value COMMON_MODE_CHOKE -> FT2232D; device selfmade:COMMON_MODE_CHOKE -> smf2:FTDI2232D
- U$2: value COMMON_MODE_CHOKE -> USB_B_STANDING; device selfmade:COMMON_MODE_CHOKE -> selfmade:USB_B_STANDING
- U$3: value COMMON_MODE_CHOKE -> M93C46-WDW6TP; device selfmade:COMMON_MODE_CHOKE -> smf2:TSSOP-8
- U$4: value COMMON_MODE_CHOKE -> S70FL01GSAGM; device selfmade:COMMON_MODE_CHOKE -> smf2:SOIC16
- U$5: value COMMON_MODE_CHOKE -> DSC1001CI1-004.0960T; device selfmade:COMMON_MODE_CHOKE -> selfmade:CDFN3225
- U_OPTO_3: value MOCD207MSOIC-8 -> MOCD207M
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Connections:
- removed net !CS!_DMS1: R3.2, U_STM32F779.74
- removed net !CS!_DMS2: R31.2, U_STM32F779.75
- removed net !CS!_DMS3: R38.2, U_STM32F779.76
- removed net !CS!_DMS4: R45.2, U_STM32F779.77
- removed net !CS!_DMS5: R52.2, U_STM32F779.78
- removed net !CS!_DMS6: R59.2, U_STM32F779.79
- removed net !CS!_PT1: RN_B_PT1.7, U_STM32F779.117
- removed net !CS!_PT2: RN_B_PT2.7, U_STM32F779.116
- removed net !CS!_PT3: RN_B_PT3.7, U_STM32F779.108
- removed net !DRDY!_DMS1: RN_DMS1.5, U_STM32F779.131
- removed net !DRDY!_DMS2: RN_DMS2.5, U_STM32F779.142
- removed net !DRDY!_DMS3: RN_DMS3.5, U_STM32F779.143
- removed net !DRDY!_DMS4: RN_DMS4.5, U_STM32F779.144
- removed net !DRDY!_DMS5: RN_DMS5.5, U_STM32F779.145
- removed net !DRDY!_DMS6: RN_DMS6.5, U_STM32F779.146
- removed net !DRDY!_PT1: RN_B_PT1.8, U_STM32F779.177
- removed net !DRDY!_PT2: RN_B_PT2.8, U_STM32F779.176
- removed net !DRDY!_PT3: RN_B_PT3.8, U_STM32F779.175
- removed net 3V3CAP: U_STM32F779.6
- removed net 3V3REF: C74.2, C75.2, R24.2, U_ADR366_3.4, U_STM32F779.41
- removed net DAPI_N: D1.C, U_CH340G.6, X_RXSM-DAPI.P$B9
- removed net DAPI_P: D2.C, U_CH340G.5, X_RXSM-DAPI.P$B10
- removed net DAPI_RX: D4.C, U_CH340G.2, U_STM32F779.11
- removed net DAPI_TX: D3.C, U_CH340G.3, U_STM32F779.43
- removed net DMS11: U$2.P$1, X_DMS.P$B3
- removed net DMS12: U$2.P$3, X_DMS.P$B2
- removed net DMS13: U$2.P$5, X_DMS.P$B1
- removed net DMS21: U$1.P$1, X_DMS.P$B6
- removed net DMS22: U$1.P$3, X_DMS.P$B5
- removed net DMS23: U$1.P$5, X_DMS.P$B4
- removed net DMS31: U$3.P$1, X_DMS.P$B9
- removed net DMS32: U$3.P$3, X_DMS.P$B8
- removed net DMS33: U$3.P$5, X_DMS.P$B7
- removed net DMS41: U$4.P$1, X_DMS.P$A1
- removed net DMS42: U$4.P$3, X_DMS.P$A2
- removed net DMS43: U$4.P$5, X_DMS.P$A3
- removed net DMS51: U$5.P$1, X_DMS.P$A4
- removed net DMS52: U$5.P$3, X_DMS.P$A5
- removed net DMS53: U$5.P$5, X_DMS.P$A6
- removed net DMS61: U$6.P$1, X_DMS.P$A7
- removed net DMS62: U$6.P$3, X_DMS.P$A8
- removed net DMS63: U$6.P$5, X_DMS.P$A9
- removed net EXP_IN_OPT: D10.C, R13.1, U_OPTO_3.8, U_STM32F779.200
- removed net EXP_OUT_OPT: U_OPTO_3.3, U_STM32F779.201
- removed net FL_1_CS1: U_FLASH1.7, U_STM32F779.104
- removed net FL_1_CS2: U_FLASH1.6, U_STM32F779.102
- removed net FL_1_HLD: U_FLASH1.1, U_STM32F779.99
- removed net FL_1_RES: U_FLASH1.3, U_STM32F779.101
- removed net FL_1_WP: U_FLASH1.9, U_STM32F779.100
- removed net FL_2_CS1: U_FLASH2.7, U_STM32F779.112
- removed net FL_2_CS2: U_FLASH2.6, U_STM32F779.111
- removed net FL_2_HLD: U_FLASH2.1, U_STM32F779.109
- removed net FL_2_RES: U_FLASH2.3, U_STM32F779.110
- removed net FL_2_WP: U_FLASH2.9, U_STM32F779.113
- removed net INTERSPU_RX: D11.C, U_STM32F779.166, X_MIRROR.P$A9, X_MIRROR1.P$A4
- removed net INTERSPU_TX: D12.C, U_STM32F779.163, X_MIRROR.P$A10, X_MIRROR1.P$A5
- removed net IO1: U_STM32F779.50, X_GPIO.P$A10
- removed net IO2: U_STM32F779.49, X_GPIO.P$A9
- removed net IO3: U_STM32F779.48, X_GPIO.P$A8
- removed net IO4: U_STM32F779.47, X_GPIO.P$A7
- removed net IO5: U_STM32F779.38, X_GPIO.P$A6
- removed net IO6: U_STM32F779.37, X_GPIO.P$A5
- removed net IO7: U_STM32F779.36, X_GPIO.P$A4
- removed net IO8: U_STM32F779.35, X_GPIO.P$A3
- removed net LO_OPT: D7.C, RN12.6, U_OPTO_2.8, U_STM32F779.208
- removed net LWL_IN: U$9.VOUT, U_STM32F779.7
- removed net LWL_OUT: U$8.VIN, U_STM32F779.157
- removed net MS_SEL: JP_MS.2, R29.1, SJ_MS.2, U_STM32F779.129
- removed net N$1 (its old number): C2.1, Q1.2, U_CH340G.8
- removed net N$114: C50.2, C51.1, R53.1, U_ADC_DMS5.9
- removed net N$115: C51.2, C53.1, R54.1, U_ADC_DMS5.10
- removed net N$116: R54.2, R55.1, R56.1
- removed net N$117: C49.1, U_ADC_DMS5.7
- removed net N$118: R53.2, U$5.P$4
- removed net N$119: R50.2, U_ADC_DMS5.4
- removed net N$120: R51.1, U_ADC_DMS5.15
- removed net N$121: RN_DMS5.1, U_ADC_DMS5.20
- removed net N$122: RN_DMS5.2, U_ADC_DMS5.19
- removed net N$123: RN_DMS5.3, U_ADC_DMS5.18
- removed net N$124: RN_DMS5.4, U_ADC_DMS5.17
- removed net N$125: R52.1, U_ADC_DMS5.16
- removed net N$128: C57.2, C58.1, R60.1, U_ADC_DMS6.9
- removed net N$129: C58.2, C59.1, R61.1, U_ADC_DMS6.10
- removed net N$130: R61.2, R62.1, R63.1
- removed net N$131: C56.1, U_ADC_DMS6.7
- removed net N$132: R60.2, U$6.P$4
- removed net N$133: R57.2, U_ADC_DMS6.4
- removed net N$134: R58.1, U_ADC_DMS6.15
- removed net N$135: RN_DMS6.1, U_ADC_DMS6.20
- removed net N$136: RN_DMS6.2, U_ADC_DMS6.19
- removed net N$137: RN_DMS6.3, U_ADC_DMS6.18
- removed net N$138: RN_DMS6.4, U_ADC_DMS6.17
- removed net N$139: R59.1, U_ADC_DMS6.16
- removed net NRST: C18.1, JP1.1, R26.1, U_STM32F779.34, X_PROG.15
- removed net PDR_ON: R9.1, U_STM32F779.203
- removed net PT11: R_I1_PT1.2, U_ADC_PT1.9, X_PT.P$B3
- removed net PT12: R_I2_PT1.2, U_ADC_PT1.12, X_PT.P$B2
- removed net PT13: R_R1_PT1.2, R_REF_PT1.2, X_PT.P$B1
- removed net PT21: R_I1_PT2.2, U_ADC_PT2.9, X_PT.P$B5
- removed net PT22: R_I2_PT2.2, U_ADC_PT2.12, X_PT.P$B4
- removed net PT23: R_R1_PT2.2, R_REF_PT2.2, X_PT.P$B6
- removed net PT31: R_I1_PT3.2, U_ADC_PT3.9, X_PT.P$A1
- removed net PT32: R_I2_PT3.2, U_ADC_PT3.12, X_PT.P$A2
- removed net PT33: R_R1_PT3.2, R_REF_PT3.2, X_PT.P$A3
- removed net SD_CS: U$7.2, U_STM32F779.31
- removed net SODS_OPT: D8.C, RN12.8, U_OPTO_1.8, U_STM32F779.206
- removed net SOE_OPT: D9.C, RN12.7, U_OPTO_1.6, U_STM32F779.207
- removed net SPI2_MISO: U_FLASH2.8, U_STM32F779.106
- removed net SPI2_MOSI: U_FLASH2.15, U_STM32F779.107
- removed net SPI2_SCK: U_FLASH2.16, U_STM32F779.105
- removed net SPI3_MISO: RN_A_PT1.5, RN_A_PT2.5, RN_A_PT3.5, U_STM32F779.162
- removed net SPI3_MOSI: RN_A_PT1.6, RN_A_PT2.6, RN_A_PT3.6, U_STM32F779.63
- removed net SPI3_SCK: RN_A_PT1.7, RN_A_PT2.7, RN_A_PT3.7, U_STM32F779.161
- removed net SPI4_MISO: RN_DMS1.6, RN_DMS2.6, RN_DMS3.6, RN_DMS4.6, RN_DMS5.6, RN_DMS6.6, U_STM32F779.4
- removed net SPI4_MOSI: RN_DMS1.7, RN_DMS2.7, RN_DMS3.7, RN_DMS4.7, RN_DMS5.7, RN_DMS6.7, U_STM32F779.5
- removed net SPI4_SCK: RN_DMS1.8, RN_DMS2.8, RN_DMS3.8, RN_DMS4.8, RN_DMS5.8, RN_DMS6.8, U_STM32F779.1
- removed net SPI5_MISO: U$7.7, U_STM32F779.29
- removed net SPI5_MOSI: U$7.3, U_STM32F779.30
- removed net SPI5_SCK: U$7.5, U_STM32F779.28
- removed net SPI6_MISO: U_FLASH1.8, U_STM32F779.55
- removed net SPI6_MOSI: U_FLASH1.15, U_STM32F779.56
- removed net SPI6_SCK: U_FLASH1.16, U_STM32F779.54
- removed net TCK: U_STM32F779.159, X_PROG.9
- removed net TDI: U_STM32F779.160, X_PROG.5
- removed net TDO: U_STM32F779.192, X_PROG.13
- removed net TMS: U_STM32F779.147, X_PROG.7
- removed net TRST: JP1.2, U_STM32F779.193, X_PROG.3
- new net ADC_START: R34.2, STAMP1:ADC_SG1.23, STAMP1:ADC_SG2.23, STAMP1:ADC_TEMP.23, STAMP2:ADC_SG1.23, STAMP2:ADC_SG2.23, STAMP2:ADC_TEMP.23, STAMP3:ADC_SG1.23, STAMP3:ADC_SG2.23, STAMP3:ADC_TEMP.23, STAMP4:ADC_SG1.23, STAMP4:ADC_SG2.23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
- new net DAPI_CTS: SF2_M2S010TQ1.112, U$1.38
- new net DAPI_DSR: SF2_M2S010TQ1.116, U$1.36
- new net DAPI_DTR: SF2_M2S010TQ1.117, U$1.35
- new net DAPI_RTS: SF2_M2S010TQ1.115, U$1.37
- new net DAPI_RXD: SF2_M2S010TQ1.110, U$1.40
- new net DAPI_TXD: SF2_M2S010TQ1.111, U$1.39
- new net EECLK: U$1.1, U$3.2
- new net EECS: U$1.48, U$3.1
- new net EED: R27.2, U$1.2, U$3.3
- new net F_CLK: SF2_M2S010TQ1.100, U$4.16
- new net F_CS1: SF2_M2S010TQ1.103, U$4.7
- new net F_CS2: SF2_M2S010TQ1.94, U$4.6
- new net F_MISO: SF2_M2S010TQ1.101, U$4.8
- new net F_MOSI: SF2_M2S010TQ1.102, U$4.15
- new net N$18: SF2_M2S010TQ1.75, U$1.24
- new net N$19: SF2_M2S010TQ1.79, U$1.23
- new net N$50: R45.2, SF2_M2S010TQ1.91
- new net PROBE_A: PROBES.1, SF2_M2S010TQ1.47
- new net PROBE_B: PROBES.3, SF2_M2S010TQ1.46
- new net RXSM_LO: U_OPTO_5.2
- new net RXSM_SODS: U_OPTO_5.4
- new net RXSM_SOE: U_OPTO_3.2
- new net SG_CLK: R14.2, STAMP1:ADC_SG1.3, STAMP1:ADC_SG2.3, STAMP2:ADC_SG1.3, STAMP2:ADC_SG2.3, STAMP3:ADC_SG1.3, STAMP3:ADC_SG2.3, STAMP4:ADC_SG1.3, STAMP4:ADC_SG2.3, STAMP5:ADC_SG1.3, STAMP5:ADC_SG2.3, STAMP6:ADC_SG1.3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
- new net STAMP1:N$34: STAMP1:ADC_SG1.9, STAMP1:C29.1
- new net STAMP1:N$35: STAMP1:ADC_SG2.4, STAMP1:R68.1
- new net STAMP1:N$36: STAMP1:ADC_SG1.25, STAMP1:R28.2
- new net STAMP1:N$37: STAMP1:ADC_SG1.4, STAMP1:R24.1
- new net STAMP1:N$38: STAMP1:ADC_SG1.26, STAMP1:R31.2
- new net STAMP1:N$39: STAMP1:ADC_SG1.11, STAMP1:C31.2, STAMP1:C32.1, STAMP1:R29.1
- new net STAMP1:N$40: STAMP1:ADC_SG1.12, STAMP1:C32.2, STAMP1:C33.1, STAMP1:R32.1
- new net STAMP1:N$41: STAMP1:ADC_SG2.9, STAMP1:C46.1
- new net STAMP1:N$42: STAMP1:ADC_SG2.25, STAMP1:R71.2
- new net STAMP1:N$43: STAMP1:ADC_SG2.26, STAMP1:R70.2
- new net STAMP1:N$79: STAMP1:ADC_SG2.11, STAMP1:C48.2, STAMP1:C49.1, STAMP1:R72.1
- new net STAMP1:N$80: STAMP1:ADC_SG2.12, STAMP1:C49.2, STAMP1:C50.1, STAMP1:R73.1
- new net STAMP1:N$81: STAMP1:R30.1, STAMP1:R32.2, STAMP1:R33.1
- new net STAMP1:N$82: STAMP1:R69.1, STAMP1:R73.2, STAMP1:R74.1
- new net STAMP1:N$83: STAMP1:R29.2, STAMP1:U$6.P$3
- new net STAMP1:N$84: STAMP1:R72.2, STAMP1:U$7.P$3
- new net STAMP1:N$85: STAMP1:ADC_TEMP.25, STAMP1:R76.2
- new net STAMP1:N$86: STAMP1:ADC_TEMP.26, STAMP1:R75.2
- new net STAMP1:N$87: STAMP1:ADC_TEMP.4, STAMP1:R77.1
- new net STAMP1:N$88: STAMP1:ADC_TEMP.12, STAMP1:C53.2, STAMP1:C54.1, STAMP1:R78.1
- new net STAMP1:N$89: STAMP1:ADC_TEMP.17, STAMP1:C54.2, STAMP1:C55.1, STAMP1:R79.1
- new net STAMP1:N$90: STAMP1:ADC_TEMP.9, STAMP1:C56.1
- new net STAMP1:N$91: STAMP1:ADC_TEMP.6, STAMP1:C57.2, STAMP1:C58.1, STAMP1:R81.1
- new net STAMP1:N$92: STAMP1:ADC_TEMP.5, STAMP1:C57.1, STAMP1:C59.2, STAMP1:R80.1
- new net STAMP1_CS_SG1: R37.1, STAMP1:ADC_SG1.24
- new net STAMP1_CS_SG2: R38.1, STAMP1:ADC_SG2.24
- new net STAMP1_CS_TEMP: R39.1, STAMP1:ADC_TEMP.24
- new net STAMP1_DRDY_SG1: SF2_M2S010TQ1.134, STAMP1:R28.1
- new net STAMP1_DRDY_SG2: SF2_M2S010TQ1.135, STAMP1:R71.1
- new net STAMP1_DRDY_TEMP: SF2_M2S010TQ1.136, STAMP1:R76.1
- new net STAMP1_MISO: SF2_M2S010TQ1.131, STAMP1:R31.1, STAMP1:R70.1, STAMP1:R75.1
- new net STAMP1_MOSI: R35.1, STAMP1:ADC_SG1.27, STAMP1:ADC_SG2.27, STAMP1:ADC_TEMP.27
- new net STAMP1_SCLK: R36.1, STAMP1:ADC_SG1.28, STAMP1:ADC_SG2.28, STAMP1:ADC_TEMP.28
- new net STAMP2:N$34: STAMP2:ADC_SG1.9, STAMP2:C29.1
- new net STAMP2:N$35: STAMP2:ADC_SG2.4, STAMP2:R68.1
- new net STAMP2:N$36: STAMP2:ADC_SG1.25, STAMP2:R28.2
- new net STAMP2:N$37: STAMP2:ADC_SG1.4, STAMP2:R24.1
- new net STAMP2:N$38: STAMP2:ADC_SG1.26, STAMP2:R31.2
- new net STAMP2:N$39: STAMP2:ADC_SG1.11, STAMP2:C31.2, STAMP2:C32.1, STAMP2:R29.1
- new net STAMP2:N$40: STAMP2:ADC_SG1.12, STAMP2:C32.2, STAMP2:C33.1, STAMP2:R32.1
- new net STAMP2:N$41: STAMP2:ADC_SG2.9, STAMP2:C46.1
- new net STAMP2:N$42: STAMP2:ADC_SG2.25, STAMP2:R71.2
- new net STAMP2:N$43: STAMP2:ADC_SG2.26, STAMP2:R70.2
- new net STAMP2:N$79: STAMP2:ADC_SG2.11, STAMP2:C48.2, STAMP2:C49.1, STAMP2:R72.1
- new net STAMP2:N$80: STAMP2:ADC_SG2.12, STAMP2:C49.2, STAMP2:C50.1, STAMP2:R73.1
- new net STAMP2:N$81: STAMP2:R30.1, STAMP2:R32.2, STAMP2:R33.1
- new net STAMP2:N$82: STAMP2:R69.1, STAMP2:R73.2, STAMP2:R74.1
- new net STAMP2:N$83: STAMP2:R29.2, STAMP2:U$6.P$3
- new net STAMP2:N$84: STAMP2:R72.2, STAMP2:U$7.P$3
- new net STAMP2:N$85: STAMP2:ADC_TEMP.25, STAMP2:R76.2
- new net STAMP2:N$86: STAMP2:ADC_TEMP.26, STAMP2:R75.2
- new net STAMP2:N$87: STAMP2:ADC_TEMP.4, STAMP2:R77.1
- new net STAMP2:N$88: STAMP2:ADC_TEMP.12, STAMP2:C53.2, STAMP2:C54.1, STAMP2:R78.1
- new net STAMP2:N$89: STAMP2:ADC_TEMP.17, STAMP2:C54.2, STAMP2:C55.1, STAMP2:R79.1
- new net STAMP2:N$90: STAMP2:ADC_TEMP.9, STAMP2:C56.1
- new net STAMP2:N$91: STAMP2:ADC_TEMP.6, STAMP2:C57.2, STAMP2:C58.1, STAMP2:R81.1
- new net STAMP2:N$92: STAMP2:ADC_TEMP.5, STAMP2:C57.1, STAMP2:C59.2, STAMP2:R80.1
- new net STAMP2_CS_SG1: R42.2, STAMP2:ADC_SG1.24
- new net STAMP2_CS_SG2: R43.2, STAMP2:ADC_SG2.24
- new net STAMP2_CS_TEMP: R44.2, STAMP2:ADC_TEMP.24
- new net STAMP2_DRDY_SG1: SF2_M2S010TQ1.82, STAMP2:R28.1
- new net STAMP2_DRDY_SG2: SF2_M2S010TQ1.83, STAMP2:R71.1
- new net STAMP2_DRDY_TEMP: SF2_M2S010TQ1.85, STAMP2:R76.1
- new net STAMP2_MISO: SF2_M2S010TQ1.81, STAMP2:R31.1, STAMP2:R70.1, STAMP2:R75.1
- new net STAMP2_MOSI: R41.1, STAMP2:ADC_SG1.27, STAMP2:ADC_SG2.27, STAMP2:ADC_TEMP.27
- new net STAMP2_SCLK: R40.1, STAMP2:ADC_SG1.28, STAMP2:ADC_SG2.28, STAMP2:ADC_TEMP.28
- new net STAMP3:N$34: STAMP3:ADC_SG1.9, STAMP3:C29.1
- new net STAMP3:N$35: STAMP3:ADC_SG2.4, STAMP3:R68.1
- new net STAMP3:N$36: STAMP3:ADC_SG1.25, STAMP3:R28.2
- new net STAMP3:N$37: STAMP3:ADC_SG1.4, STAMP3:R24.1
- new net STAMP3:N$38: STAMP3:ADC_SG1.26, STAMP3:R31.2
- new net STAMP3:N$39: STAMP3:ADC_SG1.11, STAMP3:C31.2, STAMP3:C32.1, STAMP3:R29.1
- new net STAMP3:N$40: STAMP3:ADC_SG1.12, STAMP3:C32.2, STAMP3:C33.1, STAMP3:R32.1
- new net STAMP3:N$41: STAMP3:ADC_SG2.9, STAMP3:C46.1
- new net STAMP3:N$42: STAMP3:ADC_SG2.25, STAMP3:R71.2
- new net STAMP3:N$43: STAMP3:ADC_SG2.26, STAMP3:R70.2
- new net STAMP3:N$79: STAMP3:ADC_SG2.11, STAMP3:C48.2, STAMP3:C49.1, STAMP3:R72.1
- new net STAMP3:N$80: STAMP3:ADC_SG2.12, STAMP3:C49.2, STAMP3:C50.1, STAMP3:R73.1
- new net STAMP3:N$81: STAMP3:R30.1, STAMP3:R32.2, STAMP3:R33.1
- new net STAMP3:N$82: STAMP3:R69.1, STAMP3:R73.2, STAMP3:R74.1
- new net STAMP3:N$83: STAMP3:R29.2, STAMP3:U$6.P$3
- new net STAMP3:N$84: STAMP3:R72.2, STAMP3:U$7.P$3
- new net STAMP3:N$85: STAMP3:ADC_TEMP.25, STAMP3:R76.2
- new net STAMP3:N$86: STAMP3:ADC_TEMP.26, STAMP3:R75.2
- new net STAMP3:N$87: STAMP3:ADC_TEMP.4, STAMP3:R77.1
- new net STAMP3:N$88: STAMP3:ADC_TEMP.12, STAMP3:C53.2, STAMP3:C54.1, STAMP3:R78.1
- new net STAMP3:N$89: STAMP3:ADC_TEMP.17, STAMP3:C54.2, STAMP3:C55.1, STAMP3:R79.1
- new net STAMP3:N$90: STAMP3:ADC_TEMP.9, STAMP3:C56.1
- new net STAMP3:N$91: STAMP3:ADC_TEMP.6, STAMP3:C57.2, STAMP3:C58.1, STAMP3:R81.1
- new net STAMP3:N$92: STAMP3:ADC_TEMP.5, STAMP3:C57.1, STAMP3:C59.2, STAMP3:R80.1
- new net STAMP3_CS_SG1: R47.2, STAMP3:ADC_SG1.24
- new net STAMP3_CS_SG2: R48.2, STAMP3:ADC_SG2.24
- new net STAMP3_CS_TEMP: R49.2, STAMP3:ADC_TEMP.24
- new net STAMP3_DRDY_SG1: SF2_M2S010TQ1.93, STAMP3:R28.1
- new net STAMP3_DRDY_SG2: SF2_M2S010TQ1.43, STAMP3:R71.1
- new net STAMP3_DRDY_TEMP: SF2_M2S010TQ1.44, STAMP3:R76.1
- new net STAMP3_MISO: SF2_M2S010TQ1.92, STAMP3:R31.1, STAMP3:R70.1, STAMP3:R75.1
- new net STAMP3_MOSI: R45.1, STAMP3:ADC_SG1.27, STAMP3:ADC_SG2.27, STAMP3:ADC_TEMP.27
- new net STAMP3_SCLK: R46.2, STAMP3:ADC_SG1.28, STAMP3:ADC_SG2.28, STAMP3:ADC_TEMP.28
- new net STAMP4:N$34: STAMP4:ADC_SG1.9, STAMP4:C29.1
- new net STAMP4:N$35: STAMP4:ADC_SG2.4, STAMP4:R68.1
- new net STAMP4:N$36: STAMP4:ADC_SG1.25, STAMP4:R28.2
- new net STAMP4:N$37: STAMP4:ADC_SG1.4, STAMP4:R24.1
- new net STAMP4:N$38: STAMP4:ADC_SG1.26, STAMP4:R31.2
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Routing:
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- removed copper zone on layer 1, net 28VGND
- removed copper zone on layer 15, net 28VGND
- removed copper zone on layer 16, net 28VGND
- removed copper zone on layer 2, net 28VGND
- removed copper zone on layer 1, net 3V3
- removed copper zone on layer 15, net 3V3
- removed copper zone on layer 16, net 3V3
- removed copper zone on layer 2, net 3V3
- removed copper zone on layer 1, net 5V
- removed copper zone on layer 15, net 5V
- removed copper zone on layer 16, net 5V
- removed copper zone on layer 2, net 5V
- removed copper zone on layer 1, net GND
- removed copper zone on layer 15, net GND
- removed copper zone on layer 16, net GND
- removed copper zone on layer 2, net GND
- removed copper zone on layer 1, net STRUCT
- removed copper zone on layer 15, net STRUCT
- removed copper zone on layer 16, net STRUCT
- removed copper zone on layer 2, net STRUCT
Other:
- board size 127.6 x 101.6 mm -> 160 x 100 mm
- board text removed: "28V"
- board text removed: "3V3"
- board text removed: "5V"
- board text removed: "5V-28V"
- board text removed: "HERMESS"
- board text removed: "LED1"
- board text removed: "LED2"
- board text removed: "LED3"
- board text removed: "LED4"
- board text removed: "SPU Rev 2.3"
- board text removed: "VIN: 9 - 35 V DC CIN: <2.35 A"
- board text removed: "h = 9.9 mm"

Commit message: Adds changes as of Grimsmann
Parts:
- removed ST1, ST2, ST3, ST4, ST5, STAMP1:ST, STAMP2:ST, STAMP3:ST, STAMP4:ST, STAMP5:ST, STAMP6:ST: LY20-10P-DT1, con-jae-ly:10P-T
- removed U$2: USB_B_STANDING, selfmade:USB_B_STANDING
- added C28, C29: 100n, rcl:C0805
- added C30, C31, C32: 10u, rcl:E/7260-38W
- added CN1: (no value), adafruit:USB-MINIB
- added R24: 2k2, rcl:R0805
- added STAMP1:CON, STAMP2:CON, STAMP3:CON, STAMP4:CON, STAMP5:CON, STAMP6:CON: IL-AG5-10P-S3T2, con-jae:IL-AG5-10P-S3T2
- added U_LT1: LT1528, aSparkFun:Q5-DD
- added X1: (no value), con-subd:F15HP
- moved R11 195.6 mm to (-212.1, 275.6)
- moved C21 193.2 mm to (-209.6, 260.4)
- moved C22 193.2 mm to (-215.9, 260.4)
- moved STAMP1:R68 183.5 mm to (-24.1, 19.1)
- moved STAMP2:R68 183.5 mm to (-24.1, 54.6)
- moved STAMP3:R68 183.5 mm to (-24.1, 90.2)
- moved STAMP4:R68 183.5 mm to (-24.1, 125.7)
- moved STAMP5:R68 183.5 mm to (-24.1, 161.3)
- moved STAMP6:R68 183.5 mm to (-24.1, 196.8)
- moved STAMP1:R82 181.7 mm to (-24.1, 25.4)
- moved STAMP2:R82 181.7 mm to (-24.1, 61.0)
- moved STAMP3:R82 181.7 mm to (-24.1, 96.5)
- moved STAMP4:R82 181.7 mm to (-24.1, 132.1)
- moved STAMP5:R82 181.7 mm to (-24.1, 167.6)
- moved STAMP6:R82 181.7 mm to (-24.1, 203.2)
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Connections:
- removed net LED_1: RN10.1
- removed net LED_2: RN10.2
- removed net LED_3: RN10.3
- removed net LED_4: RN10.4
- removed net N$100: ST4.P$9, STAMP4:ST.P$9, STAMP4:U$7.P$4
- removed net N$101: ST4.P$8, STAMP4:ST.P$8, STAMP4:U$7.P$2
- removed net N$102: ST4.P$7, STAMP4:ADC_TEMP.11, STAMP4:R78.2, STAMP4:ST.P$4
- removed net N$103: ST4.P$6, STAMP4:ADC_TEMP.18, STAMP4:R79.2, STAMP4:ST.P$7
- removed net N$104: ST4.P$5, STAMP4:R80.2, STAMP4:R82.2, STAMP4:ST.P$6
- removed net N$105: ST5.P$1
- removed net N$106: ST5.P$2
- removed net N$107: ST5.P$3
- removed net N$108: ST5.P$10
- removed net N$109: ST5.P$9
- removed net N$110: ST5.P$8
- removed net N$111: ST5.P$7
- removed net N$112: ST5.P$6
- removed net N$113: ST5.P$5
- removed net N$28: U$4.9, WP.2
- removed net N$34: ST1.P$3, STAMP1:ST.P$1, STAMP1:U$6.P$6
- removed net N$35: ST1.P$2, STAMP1:ST.P$2, STAMP1:U$6.P$4
- removed net N$36: ST1.P$1, STAMP1:ST.P$3, STAMP1:U$6.P$2
- removed net N$37: ST1.P$10, STAMP1:ST.P$10, STAMP1:U$7.P$6
- removed net N$38: ST1.P$9, STAMP1:ST.P$9, STAMP1:U$7.P$4
- removed net N$39: ST1.P$8, STAMP1:ST.P$8, STAMP1:U$7.P$2
- removed net N$40: ST1.P$7, STAMP1:ADC_TEMP.11, STAMP1:R78.2, STAMP1:ST.P$4
- removed net N$41: ST1.P$6, STAMP1:ADC_TEMP.18, STAMP1:R79.2, STAMP1:ST.P$7
- removed net N$42: ST1.P$5, STAMP1:R80.2, STAMP1:R82.2, STAMP1:ST.P$6
- removed net N$43: ST2.P$1, STAMP2:ST.P$3, STAMP2:U$6.P$2
- removed net N$79: ST2.P$2, STAMP2:ST.P$2, STAMP2:U$6.P$4
- removed net N$80: ST2.P$3, STAMP2:ST.P$1, STAMP2:U$6.P$6
- removed net N$81: ST2.P$10, STAMP2:ST.P$10, STAMP2:U$7.P$6
- removed net N$82: ST2.P$9, STAMP2:ST.P$9, STAMP2:U$7.P$4
- removed net N$83: ST2.P$8, STAMP2:ST.P$8, STAMP2:U$7.P$2
- removed net N$84: ST2.P$7, STAMP2:ADC_TEMP.11, STAMP2:R78.2, STAMP2:ST.P$4
- removed net N$85: ST2.P$6, STAMP2:ADC_TEMP.18, STAMP2:R79.2, STAMP2:ST.P$7
- removed net N$86: ST2.P$5, STAMP2:R80.2, STAMP2:R82.2, STAMP2:ST.P$6
- removed net N$87: ST3.P$1, STAMP3:ST.P$3, STAMP3:U$6.P$2
- removed net N$88: ST3.P$2, STAMP3:ST.P$2, STAMP3:U$6.P$4
- removed net N$89: ST3.P$3, STAMP3:ST.P$1, STAMP3:U$6.P$6
- removed net N$90: ST3.P$10, STAMP3:ST.P$10, STAMP3:U$7.P$6
- removed net N$91: ST3.P$9, STAMP3:ST.P$9, STAMP3:U$7.P$4
- removed net N$92: ST3.P$8, STAMP3:ST.P$8, STAMP3:U$7.P$2
- removed net N$93: ST3.P$7, STAMP3:ADC_TEMP.11, STAMP3:R78.2, STAMP3:ST.P$4
- removed net N$94: ST3.P$6, STAMP3:ADC_TEMP.18, STAMP3:R79.2, STAMP3:ST.P$7
- removed net N$95: ST3.P$5, STAMP3:R80.2, STAMP3:R82.2, STAMP3:ST.P$6
- removed net N$96: ST4.P$1, STAMP4:ST.P$3, STAMP4:U$6.P$2
- removed net N$97: ST4.P$2, STAMP4:ST.P$2, STAMP4:U$6.P$4
- removed net N$98: ST4.P$3, STAMP4:ST.P$1, STAMP4:U$6.P$6
- removed net N$99: ST4.P$10, STAMP4:ST.P$10, STAMP4:U$7.P$6
- new net HB_MSS: RN10.3, SF2_M2S010TQ1.15
- new net HB_STAMPS: RN10.1, SF2_M2S010TQ1.13
- new net HB_STORAGE: RN10.2, SF2_M2S010TQ1.14
- new net LED4: RN10.4, SF2_M2S010TQ1.16
- new net STAMP1:SG1_AIN1: STAMP1:CON.P$1, STAMP1:U$6.P$6
- new net STAMP1:SG1_AIN2: STAMP1:CON.P$2, STAMP1:U$6.P$4
- new net STAMP1:SG1_AIN3: STAMP1:CON.P$3, STAMP1:U$6.P$2
- new net STAMP1:SG2_AIN1: STAMP1:CON.P$10, STAMP1:U$7.P$6
- new net STAMP1:SG2_AIN2: STAMP1:CON.P$9, STAMP1:U$7.P$4
- new net STAMP1:SG2_AIN3: STAMP1:CON.P$8, STAMP1:U$7.P$2
- new net STAMP1:TEMP_AIN1: STAMP1:ADC_TEMP.11, STAMP1:CON.P$4, STAMP1:R78.2
- new net STAMP1:TEMP_AIN2: STAMP1:ADC_TEMP.18, STAMP1:CON.P$5, STAMP1:R79.2
- new net STAMP1:TEMP_AIN3: STAMP1:CON.P$7, STAMP1:R80.2, STAMP1:R82.2
- new net STAMP2:SG1_AIN1: STAMP2:CON.P$1, STAMP2:U$6.P$6
- new net STAMP2:SG1_AIN2: STAMP2:CON.P$2, STAMP2:U$6.P$4
- new net STAMP2:SG1_AIN3: STAMP2:CON.P$3, STAMP2:U$6.P$2
- new net STAMP2:SG2_AIN1: STAMP2:CON.P$10, STAMP2:U$7.P$6
- new net STAMP2:SG2_AIN2: STAMP2:CON.P$9, STAMP2:U$7.P$4
- new net STAMP2:SG2_AIN3: STAMP2:CON.P$8, STAMP2:U$7.P$2
- new net STAMP2:TEMP_AIN1: STAMP2:ADC_TEMP.11, STAMP2:CON.P$4, STAMP2:R78.2
- new net STAMP2:TEMP_AIN2: STAMP2:ADC_TEMP.18, STAMP2:CON.P$5, STAMP2:R79.2
- new net STAMP2:TEMP_AIN3: STAMP2:CON.P$7, STAMP2:R80.2, STAMP2:R82.2
- new net STAMP3:SG1_AIN1: STAMP3:CON.P$1, STAMP3:U$6.P$6
- new net STAMP3:SG1_AIN2: STAMP3:CON.P$2, STAMP3:U$6.P$4
- new net STAMP3:SG1_AIN3: STAMP3:CON.P$3, STAMP3:U$6.P$2
- new net STAMP3:SG2_AIN1: STAMP3:CON.P$10, STAMP3:U$7.P$6
- new net STAMP3:SG2_AIN2: STAMP3:CON.P$9, STAMP3:U$7.P$4
- new net STAMP3:SG2_AIN3: STAMP3:CON.P$8, STAMP3:U$7.P$2
- new net STAMP3:TEMP_AIN1: STAMP3:ADC_TEMP.11, STAMP3:CON.P$4, STAMP3:R78.2
- new net STAMP3:TEMP_AIN2: STAMP3:ADC_TEMP.18, STAMP3:CON.P$5, STAMP3:R79.2
- new net STAMP3:TEMP_AIN3: STAMP3:CON.P$7, STAMP3:R80.2, STAMP3:R82.2
- new net STAMP4:SG1_AIN1: STAMP4:CON.P$1, STAMP4:U$6.P$6
- new net STAMP4:SG1_AIN2: STAMP4:CON.P$2, STAMP4:U$6.P$4
- new net STAMP4:SG1_AIN3: STAMP4:CON.P$3, STAMP4:U$6.P$2
- new net STAMP4:SG2_AIN1: STAMP4:CON.P$10, STAMP4:U$7.P$6
- new net STAMP4:SG2_AIN2: STAMP4:CON.P$9, STAMP4:U$7.P$4
- new net STAMP4:SG2_AIN3: STAMP4:CON.P$8, STAMP4:U$7.P$2
- new net STAMP4:TEMP_AIN1: STAMP4:ADC_TEMP.11, STAMP4:CON.P$4, STAMP4:R78.2
- new net STAMP4:TEMP_AIN2: STAMP4:ADC_TEMP.18, STAMP4:CON.P$5, STAMP4:R79.2
- new net STAMP4:TEMP_AIN3: STAMP4:CON.P$7, STAMP4:R80.2, STAMP4:R82.2
- new net WP: SF2_M2S010TQ1.8, U$4.9, WP.2
- net 28V: now also X1.1, X1.9
- net 28VGND: now also X1.15, X1.8
- net 3V3: now also R27.2, U$5.P1
- net 5V: now also C28.2, C30.+, U_LT1.4, U_LT1.5
- net EED: now also R24.2; no longer R27.2
- net EXP_IN_N: now also X1.14
- net EXP_IN_P: now also X1.13
- net EXP_OUT_N: now also X1.7
- net EXP_OUT_P: now also X1.6
- net GND: now also C28.1, C29.1, C30.-, C31.-, C32.-, CN1.GND, STAMP1:CON.P$6, STAMP2:CON.P$6, STAMP3:CON.P$6, STAMP4:CON.P$6, STAMP5:CON.P$6, STAMP6:CON.P$6, U_LT1.3, U_LT1.6; no longer ST1.P$4, ST2.P$4, ST3.P$4, ST4.P$4, ST5.P$4, STAMP1:ST.P$5, STAMP2:ST.P$5, STAMP3:ST.P$5, STAMP4:ST.P$5, STAMP5:ST.P$5, STAMP6:ST.P$5, U$2.P$4, U$2.P$5, U$2.P$6
- net N$16: now also CN1.VBUS; no longer U$2.P$1
- net N$23: now also R24.1
- net RXSM_LO: now also X1.5
- net RXSM_SODS: now also X1.3
- net RXSM_SOE: now also X1.4
- net STAMP5:SG1_AIN1: now also STAMP5:CON.P$1; no longer STAMP5:ST.P$1
- net STAMP5:SG1_AIN2: now also STAMP5:CON.P$2; no longer STAMP5:ST.P$2
- net STAMP5:SG1_AIN3: now also STAMP5:CON.P$3; no longer STAMP5:ST.P$3
- net STAMP5:SG2_AIN1: now also STAMP5:CON.P$10; no longer STAMP5:ST.P$10
- net STAMP5:SG2_AIN2: now also STAMP5:CON.P$9; no longer STAMP5:ST.P$9
- net STAMP5:SG2_AIN3: now also STAMP5:CON.P$8; no longer STAMP5:ST.P$8
- net STAMP5:TEMP_AIN1: now also STAMP5:CON.P$4; no longer STAMP5:ST.P$4
- net STAMP5:TEMP_AIN2: now also STAMP5:CON.P$5; no longer STAMP5:ST.P$7
- net STAMP5:TEMP_AIN3: now also STAMP5:CON.P$7; no longer STAMP5:ST.P$6
- net STAMP6:SG1_AIN1: now also STAMP6:CON.P$1; no longer STAMP6:ST.P$1
- net STAMP6:SG1_AIN2: now also STAMP6:CON.P$2; no longer STAMP6:ST.P$2
- net STAMP6:SG1_AIN3: now also STAMP6:CON.P$3; no longer STAMP6:ST.P$3
- net STAMP6:SG2_AIN1: now also STAMP6:CON.P$10; no longer STAMP6:ST.P$10
- net STAMP6:SG2_AIN2: now also STAMP6:CON.P$9; no longer STAMP6:ST.P$9
- net STAMP6:SG2_AIN3: now also STAMP6:CON.P$8; no longer STAMP6:ST.P$8
- net STAMP6:TEMP_AIN1: now also STAMP6:CON.P$4; no longer STAMP6:ST.P$4
- net STAMP6:TEMP_AIN2: now also STAMP6:CON.P$5; no longer STAMP6:ST.P$7
- net STAMP6:TEMP_AIN3: now also STAMP6:CON.P$7; no longer STAMP6:ST.P$6
- net USB_N: now also CN1.D-; no longer U$2.P$2
- net USB_P: now also CN1.D+; no longer U$2.P$3
- net VCCINT: now also C29.2, C31.+, C32.+, U_LT1.1, U_LT1.2
Other:
- board size 160 x 100 mm -> 160 x 130 mm

Commit message: First STAMP layout
Parts:
- removed C34: 100n, rcl:C0805
- removed R34, R37, R38, R39, R42, R43, R44, R47, R48, R49, R52, R53, R54, R57, R58, R59, R62, R63, R67, STAMP1:R28, STAMP1:R71, STAMP1:R76, STAMP2:R28, STAMP2:R71, STAMP2:R76, STAMP3:R28, STAMP3:R71, STAMP3:R76, STAMP4:R28, STAMP4:R71, STAMP4:R76, STAMP5:R28, STAMP5:R71, STAMP5:R76, STAMP6:R28, STAMP6:R71, STAMP6:R76: 47, rcl:R0805
- C42: device rcl:C0805 -> rcl:C1206
- moved R65 408.9 mm to (125.7, 29.3), flipped to the bottom
- moved RN10 408.6 mm to (152.4, 55.9), turned to 270 degrees
- moved R64 405.3 mm to (125.7, 26.9), flipped to the bottom
- moved R66 395.0 mm to (114.3, 11.4), turned to 180 degrees
- moved R11 392.6 mm to (143.5, 109.2), turned to 270 degrees
- moved R25 389.6 mm to (139.7, 58.4), turned to 180 degrees
- moved R21 387.4 mm to (151.1, 41.9), turned to 180 degrees
- moved R23 382.9 mm to (141.0, 53.3), turned to 90 degrees
- moved R20 380.8 mm to (151.1, 44.5), turned to 180 degrees
- moved C20 380.3 mm to (129.5, 76.2)
- moved R22 378.3 mm to (137.2, 47.0), turned to 270 degrees
- moved C19 376.6 mm to (129.5, 72.4)
- moved R19 374.2 mm to (151.1, 47.0), turned to 180 degrees
- moved C66 370.3 mm to (139.7, 39.4), flipped to the bottom, turned to 270 degrees
- moved R18 367.5 mm to (151.1, 49.5), turned to 180 degrees
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Connections:
- removed net N$44: R34.1, SF2_M2S010TQ1.128
- removed net N$53: R37.2, SF2_M2S010TQ1.137
- removed net N$54: R38.2, SF2_M2S010TQ1.141
- removed net N$57: R39.2, SF2_M2S010TQ1.142
- removed net N$58: R42.1, SF2_M2S010TQ1.87
- removed net N$59: R43.1, SF2_M2S010TQ1.88
- removed net N$60: R44.1, SF2_M2S010TQ1.89
- removed net N$61: R47.1, SF2_M2S010TQ1.48
- removed net N$62: R48.1, SF2_M2S010TQ1.49
- removed net N$63: R49.1, SF2_M2S010TQ1.52
- removed net N$66: R54.2, SF2_M2S010TQ1.61
- removed net N$67: R53.2, SF2_M2S010TQ1.60
- removed net N$68: R52.2, SF2_M2S010TQ1.58
- removed net N$71: R57.1, SF2_M2S010TQ1.29
- removed net N$72: R58.1, SF2_M2S010TQ1.30
- removed net N$73: R59.2, SF2_M2S010TQ1.32
- removed net N$76: R62.1, SF2_M2S010TQ1.3
- removed net N$77: R63.1, SF2_M2S010TQ1.4
- removed net N$78: R67.1, SF2_M2S010TQ1.7
- removed net STAMP1:N$36: STAMP1:ADC_SG1.25, STAMP1:R28.2
- removed net STAMP1:N$42: STAMP1:ADC_SG2.25, STAMP1:R71.2
- removed net STAMP1:N$85: STAMP1:ADC_TEMP.25, STAMP1:R76.2
- removed net STAMP2:N$36: STAMP2:ADC_SG1.25, STAMP2:R28.2
- removed net STAMP2:N$42: STAMP2:ADC_SG2.25, STAMP2:R71.2
- removed net STAMP2:N$85: STAMP2:ADC_TEMP.25, STAMP2:R76.2
- removed net STAMP3:N$36: STAMP3:ADC_SG1.25, STAMP3:R28.2
- removed net STAMP3:N$42: STAMP3:ADC_SG2.25, STAMP3:R71.2
- removed net STAMP3:N$85: STAMP3:ADC_TEMP.25, STAMP3:R76.2
- removed net STAMP4:N$36: STAMP4:ADC_SG1.25, STAMP4:R28.2
- removed net STAMP4:N$42: STAMP4:ADC_SG2.25, STAMP4:R71.2
- removed net STAMP4:N$85: STAMP4:ADC_TEMP.25, STAMP4:R76.2
- removed net STAMP5:N$36: STAMP5:ADC_SG1.25, STAMP5:R28.2
- removed net STAMP5:N$42: STAMP5:ADC_SG2.25, STAMP5:R71.2
- removed net STAMP5:N$85: STAMP5:ADC_TEMP.25, STAMP5:R76.2
- removed net STAMP6:N$36: STAMP6:ADC_SG1.25, STAMP6:R28.2
- removed net STAMP6:N$42: STAMP6:ADC_SG2.25, STAMP6:R71.2
- removed net STAMP6:N$85: STAMP6:ADC_TEMP.25, STAMP6:R76.2
- net 28V: no longer C34.2
- net 28VGND: no longer C34.1
- net ADC_START: now also SF2_M2S010TQ1.128; no longer R34.2
- net HB_MSS: now also SF2_M2S010TQ1.14; no longer SF2_M2S010TQ1.15
- net HB_STAMPS: now also SF2_M2S010TQ1.16; no longer SF2_M2S010TQ1.13
- net HB_STORAGE: now also SF2_M2S010TQ1.15; no longer SF2_M2S010TQ1.14
- net LED4: now also SF2_M2S010TQ1.13; no longer SF2_M2S010TQ1.16
- net STAMP1_CS_SG1: now also SF2_M2S010TQ1.137; no longer R37.1
- net STAMP1_CS_SG2: now also SF2_M2S010TQ1.141; no longer R38.1
- net STAMP1_CS_TEMP: now also SF2_M2S010TQ1.142; no longer R39.1
- net STAMP1_DRDY_SG1: now also STAMP1:ADC_SG1.25; no longer STAMP1:R28.1
- net STAMP1_DRDY_SG2: now also STAMP1:ADC_SG2.25; no longer STAMP1:R71.1
- net STAMP1_DRDY_TEMP: now also STAMP1:ADC_TEMP.25; no longer STAMP1:R76.1
- net STAMP2_CS_SG1: now also SF2_M2S010TQ1.87; no longer R42.2
- net STAMP2_CS_SG2: now also SF2_M2S010TQ1.88; no longer R43.2
- net STAMP2_CS_TEMP: now also SF2_M2S010TQ1.89; no longer R44.2
- net STAMP2_DRDY_SG1: now also STAMP2:ADC_SG1.25; no longer STAMP2:R28.1
- net STAMP2_DRDY_SG2: now also STAMP2:ADC_SG2.25; no longer STAMP2:R71.1
- net STAMP2_DRDY_TEMP: now also STAMP2:ADC_TEMP.25; no longer STAMP2:R76.1
- net STAMP3_CS_SG1: now also SF2_M2S010TQ1.48; no longer R47.2
- net STAMP3_CS_SG2: now also SF2_M2S010TQ1.49; no longer R48.2
- net STAMP3_CS_TEMP: now also SF2_M2S010TQ1.52; no longer R49.2
- net STAMP3_DRDY_SG1: now also STAMP3:ADC_SG1.25; no longer STAMP3:R28.1
- net STAMP3_DRDY_SG2: now also STAMP3:ADC_SG2.25; no longer STAMP3:R71.1
- net STAMP3_DRDY_TEMP: now also STAMP3:ADC_TEMP.25; no longer STAMP3:R76.1
- net STAMP4_CS_SG1: now also SF2_M2S010TQ1.61; no longer R54.1
- net STAMP4_CS_SG2: now also SF2_M2S010TQ1.60; no longer R53.1
- net STAMP4_CS_TEMP: now also SF2_M2S010TQ1.58; no longer R52.1
- net STAMP4_DRDY_SG1: now also STAMP4:ADC_SG1.25; no longer STAMP4:R28.1
- net STAMP4_DRDY_SG2: now also STAMP4:ADC_SG2.25; no longer STAMP4:R71.1
- net STAMP4_DRDY_TEMP: now also STAMP4:ADC_TEMP.25; no longer STAMP4:R76.1
- net STAMP5_CS_SG1: now also SF2_M2S010TQ1.29; no longer R57.2
- net STAMP5_CS_SG2: now also SF2_M2S010TQ1.30; no longer R58.2
- net STAMP5_CS_TEMP: now also SF2_M2S010TQ1.32; no longer R59.1
- net STAMP5_DRDY_SG1: now also STAMP5:ADC_SG1.25; no longer STAMP5:R28.1
- net STAMP5_DRDY_SG2: now also STAMP5:ADC_SG2.25; no longer STAMP5:R71.1
- net STAMP5_DRDY_TEMP: now also STAMP5:ADC_TEMP.25; no longer STAMP5:R76.1
- net STAMP6_CS_SG1: now also SF2_M2S010TQ1.3; no longer R62.2
- net STAMP6_CS_SG2: now also SF2_M2S010TQ1.4; no longer R63.2
- net STAMP6_CS_TEMP: now also SF2_M2S010TQ1.7; no longer R67.2
- net STAMP6_DRDY_SG1: now also STAMP6:ADC_SG1.25; no longer STAMP6:R28.1
- net STAMP6_DRDY_SG2: now also STAMP6:ADC_SG2.25; no longer STAMP6:R71.1
- net STAMP6_DRDY_TEMP: now also STAMP6:ADC_TEMP.25; no longer STAMP6:R76.1
Routing:
- net 28V: track 0.00 -> 209.9 mm, vias 0 -> 4
- net 28VGND: track 0.00 -> 172.5 mm, vias 0 -> 2
- net 3V3: track 0.00 -> 155.1 mm, vias 0 -> 5
- net 5V: track 0.00 -> 128.6 mm
- net GND: track 0.00 -> 116.1 mm, vias 0 -> 1
- net 5V-28V: track 0.00 -> 63.7 mm, vias 0 -> 7
- net SODS: track 0.00 -> 54.0 mm
- net SOE: track 0.00 -> 52.0 mm, vias 0 -> 1
- net LO: track 0.00 -> 50.7 mm
- net STAMP1:SG1_AIN1: track 0.00 -> 45.8 mm
- net EXP_IN_N: track 0.00 -> 43.2 mm
- net VCCINT: track 0.00 -> 41.3 mm
- net STAMP1:TEMP_AIN3: track 0.00 -> 41.1 mm
- net EXP_IN_P: track 0.00 -> 40.2 mm, vias 0 -> 1
- net EXP_OUT_P: track 0.00 -> 40.1 mm
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