File: SPU.brd (EAGLE design)
At the start: 160 x 130 mm, 414 parts, among them Q1 BSS123, Q2 12MHz, Q3 BSS123, Q4 BSS123, Q5 BSS123, Q6 BSS123

Commit message: During work commit Reorderd RXSM interface
Parts:
- moved C21 51.8 mm to (145.0, 116.7), flipped to the top
- moved R9 48.3 mm to (130.3, 109.6)
- moved C42 21.4 mm to (147.1, 73.8), flipped to the top, turned to 270 degrees
- moved R23 16.1 mm to (127.3, 83.8), turned to 270 degrees
- moved U_7805 15.2 mm to (141.1, 73.8), flipped to the top, turned to 180 degrees
- moved R16 13.7 mm to (145.8, 97.5), flipped to the top, turned to 0 degrees
- moved R43 13.7 mm to (122.6, 84.3)
- moved Q1 13.7 mm to (122.6, 87.9)
- moved R57 11.5 mm to (140.0, 117.2), turned to 0 degrees
- moved R22 11.3 mm to (122.6, 90.9), turned to 180 degrees
- moved U_OPTO_3 10.6 mm to (130.2, 74.7), flipped to the top
- moved D5 10.4 mm to (141.4, 86.4), turned to 0 degrees
- moved R12 10.2 mm to (141.4, 83.7), turned to 180 degrees
- moved C43 9.82 mm to (145.7, 80.4), flipped to the top, turned to 0 degrees
- moved L1 9.79 mm to (147.8, 67.1)
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Routing:
- net DAPI_RTS: track 0.00 -> 69.2 mm, vias 0 -> 2
- net DAPI_CTS: track 0.00 -> 68.3 mm, vias 0 -> 2
- net DAPI_TXD: track 0.00 -> 67.8 mm, vias 0 -> 2
- net DAPI_RXD: track 0.00 -> 65.1 mm, vias 0 -> 2
- net SG_CLK: track 348.4 -> 396.5 mm
- net N$180: track 0.00 -> 15.8 mm
- net EED: track 0.00 -> 10.0 mm
- net N$179: track 0.00 -> 9.85 mm, vias 0 -> 1
- net 1V2: track 53.3 -> 60.7 mm
- net N$23: track 0.00 -> 6.33 mm
- net EECS: track 0.00 -> 5.31 mm
- net EECLK: track 0.00 -> 5.24 mm
- net 28VGND: track 3.11 -> 0.00 mm
- net F_CS2: track 33.7 -> 36.2 mm
- net N$11: track 10.5 -> 12.6 mm
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